Commit message: feat: Integrate nerf launcher into gubot_one robot and refine launcher URDF and simulation launch files.

File: src/nerf_standalone/description/urdf/launcher.urdf.xacro (robot description, xacro)
@@ -1,14 +1,23 @@
 <?xml version="1.0"?>
 <robot xmlns:xacro="http://www.ros.org/wiki/xacro" name="nerf_standalone">
+    <!-- Colors -->
+    <material name="white">
+        <color rgba="1 1 1 1" />
+    </material>
+    <material name="orange">
+        <color rgba="1 0.3 0.1 1"/>
+    </material>
+    <material name="blue">
+        <color rgba="0.2 0.2 1 1"/>
+    </material>
+    <material name="black">
+        <color rgba="0 0 0 1"/>
+    </material>
+    <material name="red">
+        <color rgba="1 0 0 1"/>
+    </material>
     <!-- World Link -->
     <link name="world"/>
-    <!-- Joint: Montageplatte -> Motor_und_Magazinplatte (Fixed for now to build base) -->
-    <!-- NOTE: In original URDF, Motor_und_Magazinplatte was PARENT of Montageplatte.
-         But here we attached Montageplatte to world.
-         Let's stick to the physical reality: Motor_und_Magazinplatte is the big base plate.
-         So let's attach Motor_und_Magazinplatte to World, and Montageplatte to IT.
-         RE-STRUCTURING to match original hierarchy:
-         World -> Motor_und_Magazinplatte (Base) -> Montageplatte (Trigger)
-    -->
+    <!-- 1. Montageplatte (BASE, connected to world for testing) -->
     <joint name="world_to_montage_joint" type="fixed">
         <parent link="world"/>
@@ -16,5 +25,4 @@
         <origin xyz="0 0 0.5" rpy="0 -1.5708 0"/>
     </joint>
-    <!-- Refined Montageplatte (Visual update to match relative position) -->
     <link name="Montageplatte">
         <visual>
@@ -37,3 +45,31 @@
         </inertial>
     </link>
+    <!-- 2. Motor_und_Magazinplatte (Attached to Montageplatte) -->
+    <joint name="trigger_joint" type="fixed">
+        <!-- User specified rotation: X=180, Y=-90. Position: 0.1m forward (Z-axis locally) -->
+        <origin xyz="0 0.0975 -0.013768" rpy="3.14159 -1.5708 0"/>
+        <parent link="Montageplatte"/>
+        <child link="Motor_und_Magazinplatte"/>
+    </joint>
+    <link name="Motor_und_Magazinplatte">
+        <visual>
+             <origin xyz="0 0 0" rpy="0 0 0"/>
+            <geometry>
+                <mesh filename="file://$(find nerf_standalone)/description/meshes/Motor_und_Magazinplatte.stl" scale="0.001 0.001 0.001"/>
+            </geometry>
+            <material name="grey">
+                <color rgba="0.5 0.5 0.5 1.0"/>
+            </material>
+        </visual>
+        <collision>
+            <origin xyz="0 0 0" rpy="0 0 0"/>
+            <geometry>
+                <box size="0.06 0.08 0.02"/>
+            </geometry>
+        </collision>
+        <inertial>
+            <mass value="0.25"/>
+            <inertia ixx="0.00036" ixy="0" ixz="0" iyy="0.00014" iyz="0" izz="0.00048"/>
+        </inertial>
+    </link>
 </robot>

Commit message: feat: Integrate the nerf launcher into gubot_one with ROS2 control, enabling a revolute trigger joint and cleaning up configurations.

File: src/nerf_standalone/description/urdf/launcher.urdf.xacro (robot description, xacro)
@@ -1,23 +1,11 @@
 <?xml version="1.0"?>
 <robot xmlns:xacro="http://www.ros.org/wiki/xacro" name="nerf_standalone">
-    <!-- Colors -->
-    <material name="white">
-        <color rgba="1 1 1 1" />
-    </material>
     <material name="orange">
         <color rgba="1 0.3 0.1 1"/>
     </material>
-    <material name="blue">
-        <color rgba="0.2 0.2 1 1"/>
+    <material name="grey">
+        <color rgba="0.5 0.5 0.5 1.0"/>
     </material>
-    <material name="black">
-        <color rgba="0 0 0 1"/>
-    </material>
-    <material name="red">
-        <color rgba="1 0 0 1"/>
-    </material>
-    <!-- World Link -->
     <link name="world"/>
-    <!-- 1. Montageplatte (BASE, connected to world for testing) -->
     <joint name="world_to_montage_joint" type="fixed">
         <parent link="world"/>
@@ -31,7 +19,5 @@
                 <mesh filename="file://$(find nerf_standalone)/description/meshes/Montageplatte.stl" scale="0.001 0.001 0.001"/>
             </geometry>
-            <material name="orange">
-                <color rgba="1.0 0.5 0.0 1.0"/>
-            </material>
+            <material name="orange"/>
         </visual>
         <collision>
@@ -45,10 +31,11 @@
         </inertial>
     </link>
-    <!-- 2. Motor_und_Magazinplatte (Attached to Montageplatte) -->
-    <joint name="trigger_joint" type="fixed">
-        <!-- User specified rotation: X=180, Y=-90. Position: 0.1m forward (Z-axis locally) -->
+    <joint name="trigger_joint" type="revolute">
         <origin xyz="0 0.0975 -0.013768" rpy="3.14159 -1.5708 0"/>
         <parent link="Montageplatte"/>
         <child link="Motor_und_Magazinplatte"/>
+        <axis xyz="1 0 0"/>
+        <limit lower="0.0" upper="1.5708" effort="10.0" velocity="1.0"/>
+        <dynamics damping="0.1" friction="0.1"/>
     </joint>
     <link name="Motor_und_Magazinplatte">
@@ -73,3 +60,5 @@
         </inertial>
     </link>
+    <xacro:include filename="ros2_control.xacro" />
+    <xacro:nerf_ros2_control />
 </robot>

File: src/nerf_standalone/description/urdf/ros2_control.xacro (robot description, xacro)
@@ -6,20 +6,5 @@
                 <plugin>gazebo_ros2_control/GazeboSystem</plugin>
             </hardware>
-            <joint name="flywheel_left_joint">
-                <command_interface name="velocity"/>
-                <state_interface name="velocity"/>
-                <state_interface name="position"/>
-            </joint>
-            <joint name="flywheel_right_joint">
-                <command_interface name="velocity"/>
-                <state_interface name="velocity"/>
-                <state_interface name="position"/>
-            </joint>
             <joint name="trigger_joint">
-                <command_interface name="position"/>
-                <state_interface name="velocity"/>
-                <state_interface name="position"/>
-            </joint>
-            <joint name="dart_pusher_joint">
                 <command_interface name="position"/>
                 <state_interface name="velocity"/>

Commit message: feat: Add new meshes for launcher components and update URDF configuration for motors and materials

File: src/nerf_standalone/description/urdf/launcher.urdf.xacro (robot description, xacro)
@@ -6,4 +6,13 @@
     <material name="grey">
         <color rgba="0.5 0.5 0.5 1.0"/>
+    </material>
+    <material name="blue">
+        <color rgba="0.2 0.2 1 1"/>
+    </material>
+    <!-- <material name="black">
+        <color rgba="0 0 0 1"/>
+    </material> -->
+    <material name="red">
+        <color rgba="1 0 0 1"/>
     </material>
     <link name="world"/>
@@ -32,15 +41,17 @@
     </link>
     <joint name="trigger_joint" type="revolute">
-        <origin xyz="0 0.0975 -0.013768" rpy="3.14159 -1.5708 0"/>
+        <!-- <origin xyz="0 0.0975 -0.013768" rpy="3.14159 -1.5708 0"/> -->
+        <origin xyz="0 0 0" rpy="3.14159 -1.5708 0"/>
         <parent link="Montageplatte"/>
         <child link="Motor_und_Magazinplatte"/>
-        <axis xyz="1 0 0"/>
-        <limit lower="0.0" upper="1.5708" effort="10.0" velocity="1.0"/>
+        <axis xyz="-1 0 0"/>
+        <limit lower="0.0" upper="2.1" effort="10.0" velocity="1.0"/>
         <dynamics damping="0.1" friction="0.1"/>
     </joint>
     <link name="Motor_und_Magazinplatte">
         <visual>
-             <origin xyz="0 0 0" rpy="0 0 0"/>
-            <geometry>
+             <origin xyz="-0.013735 -0.0982192 0.0" rpy="0 0 0"/>
+             <!-- <origin xyz="-0.013735 -0.0991 0.0005" rpy="0 0 0"/> -->
+             <geometry>
                 <mesh filename="file://$(find nerf_standalone)/description/meshes/Motor_und_Magazinplatte.stl" scale="0.001 0.001 0.001"/>
             </geometry>
@@ -60,4 +71,43 @@
         </inertial>
     </link>
+    <!-- Motor Left (Fixed to Magazinplatte) -->
+    <!-- Rotated -90 degrees around X (Counter-Clockwise if looking from front? Or standard?) -->
+    <joint name="motor_left_joint" type="fixed">
+        <origin xyz="0.055 0.035 0.02" rpy="-1.5708 3.1416 0"/>
+        <parent link="Motor_und_Magazinplatte"/>
+        <child link="motor_left"/>
+    </joint>
+    <link name="motor_left">
+        <visual>
+            <geometry>
+                <mesh filename="file://$(find nerf_standalone)/description/meshes/motor_left.stl" scale="0.001 0.001 0.001"/>
+            </geometry>
+            <material name="red"/>
+        </visual>
+        <collision>
+            <geometry>
+                <cylinder length="0.03" radius="0.015"/>
+            </geometry>
+        </collision>
+    </link>
+    <!-- Motor Right (Fixed to Magazinplatte) -->
+    <joint name="motor_right_joint" type="fixed">
+        <origin xyz="0.055 0.035 -0.02" rpy="-1.5708 3.1416 0"/>
+        <parent link="Motor_und_Magazinplatte"/>
+        <child link="motor_right"/>
+    </joint>
+    <link name="motor_right">
+        <visual>
+            <geometry>
+                <mesh filename="file://$(find nerf_standalone)/description/meshes/motor_right.stl" scale="0.001 0.001 0.001"/>
+            </geometry>
+            <material name="blue"/>
+        </visual>
+        <collision>
+            <geometry>
+                <cylinder length="0.03" radius="0.015"/>
+            </geometry>
+        </collision>
+    </link>
     <xacro:include filename="ros2_control.xacro" />
     <xacro:nerf_ros2_control />

Commit message: fix: Adjust motor joint origins for left and right motors in URDF

File: src/nerf_standalone/description/urdf/launcher.urdf.xacro (robot description, xacro)
@@ -74,5 +74,5 @@
     <!-- Rotated -90 degrees around X (Counter-Clockwise if looking from front? Or standard?) -->
     <joint name="motor_left_joint" type="fixed">
-        <origin xyz="0.055 0.035 0.02" rpy="-1.5708 3.1416 0"/>
+        <origin xyz="0.01 -0.09600 0" rpy="-1.5708 3.1416 0"/>
         <parent link="Motor_und_Magazinplatte"/>
         <child link="motor_left"/>
@@ -93,5 +93,5 @@
     <!-- Motor Right (Fixed to Magazinplatte) -->
     <joint name="motor_right_joint" type="fixed">
-        <origin xyz="0.055 0.035 -0.02" rpy="-1.5708 3.1416 0"/>
+        <origin xyz="-0.035 -0.0960 0" rpy="-1.5708 3.1416 0"/>
         <parent link="Motor_und_Magazinplatte"/>
         <child link="motor_right"/>

Commit message: feat: Integrate nerf dart launcher into the gubot_one robot model, updating its URDF, simulation launch, and RViz configurations.

File: src/nerf_standalone/description/urdf/launcher.urdf.xacro (robot description, xacro)
@@ -90,4 +90,8 @@
             </geometry>
         </collision>
+        <inertial>
+            <mass value="0.05"/>
+            <inertia ixx="0.00001" ixy="0" ixz="0" iyy="0.00001" iyz="0" izz="0.00001"/>
+        </inertial>
     </link>
     <!-- Motor Right (Fixed to Magazinplatte) -->
@@ -109,4 +113,62 @@
             </geometry>
         </collision>
+        <inertial>
+            <mass value="0.05"/>
+            <inertia ixx="0.00001" ixy="0" ixz="0" iyy="0.00001" iyz="0" izz="0.00001"/>
+        </inertial>
+    </link>
+    <!-- Flywheel Left -->
+    <joint name="flywheel_left_joint" type="continuous">
+        <origin xyz="0 0 0.0" rpy="0 0 0"/>
+        <parent link="motor_left"/>
+        <child link="flywheel_left"/>
+        <axis xyz="0 0 1"/>
+        <limit effort="5.0" velocity="100.0"/>
+        <dynamics damping="0.01" friction="0.01"/>
+    </joint>
+    <link name="flywheel_left">
+        <visual>
+            <origin xyz="0.08928 0.002734 0" rpy="-1.5708 0 0"/>
+            <geometry>
+                <mesh filename="file://$(find nerf_standalone)/description/meshes/Launcher_wheel_left.stl" scale="0.001 0.001 0.001"/>
+            </geometry>
+            <material name="red"/>
+        </visual>
+        <collision>
+            <geometry>
+                <cylinder length="0.02" radius="0.02"/>
+            </geometry>
+        </collision>
+        <inertial>
+            <mass value="0.05"/>
+            <inertia ixx="0.00001" ixy="0" ixz="0" iyy="0.00001" iyz="0" izz="0.00002"/>
+        </inertial>
+    </link>
+    <!-- Flywheel Right -->
+    <joint name="flywheel_right_joint" type="continuous">
+        <origin xyz="0 0 0.005" rpy="0 0 0"/>
+        <parent link="motor_right"/>
+        <child link="flywheel_right"/>
+        <axis xyz="0 0 1"/>
+        <limit effort="5.0" velocity="100.0"/>
+        <dynamics damping="0.01" friction="0.01"/>
+    </joint>
+    <link name="flywheel_right">
+        <visual>
+            <origin xyz="0.08928 0.002734 0" rpy="-1.5708 0 0"/>
+            <geometry>
+                <mesh filename="file://$(find nerf_standalone)/description/meshes/Launcher_wheel_right.stl" scale="0.001 0.001 0.001"/>
+            </geometry>
+            <material name="blue"/>
+        </visual>
+        <collision>
+            <geometry>
+                <cylinder length="0.02" radius="0.02"/>
+            </geometry>
+        </collision>
+        <inertial>
+            <mass value="0.05"/>
+            <inertia ixx="0.00001" ixy="0" ixz="0" iyy="0.00001" iyz="0" izz="0.00002"/>
+        </inertial>
     </link>
     <xacro:include filename="ros2_control.xacro" />

File: src/nerf_standalone/description/urdf/ros2_control.xacro (robot description, xacro)
@@ -8,4 +8,14 @@
             <joint name="trigger_joint">
                 <command_interface name="position"/>
+                <state_interface name="velocity"/>
+                <state_interface name="position"/>
+            </joint>
+            <joint name="flywheel_left_joint">
+                <command_interface name="velocity"/>
+                <state_interface name="velocity"/>
+                <state_interface name="position"/>
+            </joint>
+            <joint name="flywheel_right_joint">
+                <command_interface name="velocity"/>
                 <state_interface name="velocity"/>
                 <state_interface name="position"/>

Commit message: feat: Add Nerf Dart Launcher model, control configuration, firmware, and integrate it into the gubot_one robot.

File: src/nerf_standalone/description/urdf/launcher.urdf.xacro (robot description, xacro)
@@ -91,11 +91,11 @@
         </collision>
         <inertial>
-            <mass value="0.05"/>
-            <inertia ixx="0.00001" ixy="0" ixz="0" iyy="0.00001" iyz="0" izz="0.00001"/>
+            <mass value="0.1"/>
+            <inertia ixx="0.0001" ixy="0" ixz="0" iyy="0.0001" iyz="0" izz="0.0001"/>
         </inertial>
     </link>
     <!-- Motor Right (Fixed to Magazinplatte) -->
     <joint name="motor_right_joint" type="fixed">
-        <origin xyz="-0.035 -0.0960 0" rpy="-1.5708 3.1416 0"/>
+        <origin xyz="-0.030 -0.0960 0" rpy="-1.5708 3.1416 0"/>
         <parent link="Motor_und_Magazinplatte"/>
         <child link="motor_right"/>
@@ -114,6 +114,6 @@
         </collision>
         <inertial>
-            <mass value="0.05"/>
-            <inertia ixx="0.00001" ixy="0" ixz="0" iyy="0.00001" iyz="0" izz="0.00001"/>
+            <mass value="0.1"/>
+            <inertia ixx="0.0001" ixy="0" ixz="0" iyy="0.0001" iyz="0" izz="0.0001"/>
         </inertial>
     </link>
@@ -123,5 +123,5 @@
         <parent link="motor_left"/>
         <child link="flywheel_left"/>
-        <axis xyz="0 0 1"/>
+        <axis xyz="0 1 0"/>
         <limit effort="5.0" velocity="100.0"/>
         <dynamics damping="0.01" friction="0.01"/>
@@ -136,4 +136,5 @@
         </visual>
         <collision>
+            <origin xyz="0.08928 0.002734 0" rpy="-1.5708 0 0"/>
             <geometry>
                 <cylinder length="0.02" radius="0.02"/>
@@ -141,6 +142,6 @@
         </collision>
         <inertial>
-            <mass value="0.05"/>
-            <inertia ixx="0.00001" ixy="0" ixz="0" iyy="0.00001" iyz="0" izz="0.00002"/>
+            <mass value="0.1"/>
+            <inertia ixx="0.0001" ixy="0" ixz="0" iyy="0.0001" iyz="0" izz="0.0001"/>
         </inertial>
     </link>
@@ -150,5 +151,5 @@
         <parent link="motor_right"/>
         <child link="flywheel_right"/>
-        <axis xyz="0 0 1"/>
+        <axis xyz="0 1 0"/>
         <limit effort="5.0" velocity="100.0"/>
         <dynamics damping="0.01" friction="0.01"/>
@@ -156,5 +157,5 @@
     <link name="flywheel_right">
         <visual>
-            <origin xyz="0.08928 0.002734 0" rpy="-1.5708 0 0"/>
+            <origin xyz="0.08928 0.002734 -0.005" rpy="-1.5708 0 0"/>
             <geometry>
                 <mesh filename="file://$(find nerf_standalone)/description/meshes/Launcher_wheel_right.stl" scale="0.001 0.001 0.001"/>
@@ -163,4 +164,5 @@
         </visual>
         <collision>
+            <origin xyz="0.08928 0.002734 -0.005" rpy="-1.5708 0 0"/>
             <geometry>
                 <cylinder length="0.02" radius="0.02"/>
@@ -168,6 +170,32 @@
         </collision>
         <inertial>
-            <mass value="0.05"/>
-            <inertia ixx="0.00001" ixy="0" ixz="0" iyy="0.00001" iyz="0" izz="0.00002"/>
+            <mass value="0.1"/>
+            <inertia ixx="0.0001" ixy="0" ixz="0" iyy="0.0001" iyz="0" izz="0.0001"/>
+        </inertial>
+    </link>
+    <!-- Dart Pusher -->
+    <joint name="dart_pusher_joint" type="continuous">
+        <origin xyz="-0.05 0 0.025" rpy="0 0 0"/>
+        <parent link="Motor_und_Magazinplatte"/>
+        <child link="dart_pusher"/>
+        <axis xyz="0 0 1"/>
+        <limit effort="10.0" velocity="10.0"/>
+        <dynamics damping="0.0" friction="0.0"/>
+    </joint>
+    <link name="dart_pusher">
+        <visual>
+            <geometry>
+                <mesh filename="file://$(find nerf_standalone)/description/meshes/Dart_Pusher.stl" scale="0.001 0.001 0.001"/>
+            </geometry>
+            <material name="orange"/>
+        </visual>
+        <!-- <collision>
+            <geometry>
+                <box size="0.03 0.03 0.01"/>
+            </geometry>
+        </collision> -->
+        <inertial>
+            <mass value="0.1"/>
+            <inertia ixx="0.0002" ixy="0" ixz="0" iyy="0.0002" iyz="0" izz="0.0002"/>
         </inertial>
     </link>

File: src/nerf_standalone/description/urdf/ros2_control.xacro (robot description, xacro)
@@ -21,4 +21,9 @@
                 <state_interface name="position"/>
             </joint>
+            <joint name="dart_pusher_joint">
+                <command_interface name="velocity"/>
+                <state_interface name="velocity"/>
+                <state_interface name="position"/>
+            </joint>
         </ros2_control>
         <gazebo>
@@ -27,4 +32,5 @@
                 <robot_param_node>robot_state_publisher</robot_param_node>
                 <parameters>$(find nerf_standalone)/config/controllers.yaml</parameters>
+                <parameters>$(find nerf_standalone)/config/gains.yaml</parameters>
             </plugin>
         </gazebo>
