Commit message: feat: add `nerf_standalone` package with URDF, meshes, control configuration, and firmware, alongside updates to `gubot_one` launch and control settings.

File: src/nerf_standalone/description/urdf/launcher.urdf.xacro (robot description, xacro)
@@ -1,203 +1,309 @@
-<?xml version="1.0"?>
+<?xml version='1.0' encoding='utf-8'?>
 <robot xmlns:xacro="http://www.ros.org/wiki/xacro" name="nerf_standalone">
-    <material name="orange">
-        <color rgba="1 0.3 0.1 1"/>
-    </material>
-    <material name="grey">
-        <color rgba="0.5 0.5 0.5 1.0"/>
-    </material>
-    <material name="blue">
-        <color rgba="0.2 0.2 1 1"/>
-    </material>
-    <!-- <material name="black">
-        <color rgba="0 0 0 1"/>
-    </material> -->
-    <material name="red">
-        <color rgba="1 0 0 1"/>
-    </material>
-    <link name="world"/>
-    <joint name="world_to_montage_joint" type="fixed">
-        <parent link="world"/>
-        <child link="Montageplatte"/>
-        <origin xyz="0 0 0.5" rpy="0 -1.5708 0"/>
-    </joint>
-    <link name="Montageplatte">
-        <visual>
-            <origin xyz="0.0012 0.1035 -0.0889" rpy="-3.1416 -1.5708 0"/>
-            <geometry>
-                <mesh filename="file://$(find nerf_standalone)/description/meshes/Montageplatte.stl" scale="0.001 0.001 0.001"/>
-            </geometry>
-            <material name="orange"/>
-        </visual>
-        <collision>
-            <geometry>
-                <box size="0.05 0.1 0.02"/>
-            </geometry>
-        </collision>
-        <inertial>
-            <mass value="0.2"/>
-            <inertia ixx="0.0004" ixy="0" ixz="0" iyy="0.00005" iyz="0" izz="0.00037"/>
-        </inertial>
+    <link name="bottom_plate">
+        <inertial>
+            <origin xyz="0.07506008367977571 0.06788755296524361 -0.015949194976296238" rpy="0.0 0.0 0.0" />
+            <mass value="0.2021986172178209" />
+            <inertia ixx="0.00037557930532003186" iyy="5.362127850969058e-05" izz="0.00041640489807794057" ixy="-1.2945646322185759e-06" iyz="-1.5574886339585816e-05" ixz="9.440243990688213e-08" />
+        </inertial>
+        <visual name="bottom_plate_visual">
+            <origin xyz="0.0 0.0 0.0" rpy="0.0 0.0 0.0" />
+            <geometry>
+                <mesh filename="file://$(find nerf_standalone)/description/meshes/bottom_plate.stl" scale="0.001 0.001 0.001" />
+            </geometry>
+        </visual>
+        <collision name="bottom_plate_collision">
+            <origin xyz="0.0 0.0 0.0" rpy="0.0 0.0 0.0" />
+            <geometry>
+                <mesh filename="file://$(find nerf_standalone)/description/meshes/bottom_plate.stl" scale="0.001 0.001 0.001" />
+            </geometry>
+        </collision>
+    </link>
+    <link name="motor_bracket">
+        <inertial>
+            <origin xyz="0.06445114377692326 -0.001293871011977803 -0.01805979631895027" rpy="0.0 -7.504780922022523e-26 6.462348535570529e-27" />
+            <mass value="0.24458145922412514" />
+            <inertia ixx="0.00013685810139727812" iyy="0.0004819875327694177" izz="0.0003647641226204775" ixy="-1.2856327940143035e-05" iyz="-1.071289298066829e-05" ixz="-2.0865729712333423e-05" />
+        </inertial>
+        <visual name="motor_bracket_visual">
+            <origin xyz="0.09803428669398517 -4.3732793080548534e-05 -0.013700000763976723" rpy="1.5703501879750486 -1.5707963267948937 0" />
+            <geometry>
+                <mesh filename="file://$(find nerf_standalone)/description/meshes/motor_bracket.stl" scale="0.001 0.001 0.001" />
+            </geometry>
+        </visual>
+        <collision name="motor_bracket_collision">
+            <origin xyz="0.09803428669398517 -4.3732793080548534e-05 -0.013700000763976723" rpy="1.5703501879750486 -1.5707963267948937 0" />
+            <geometry>
+                <!-- box size="0.1 0.1 0.1" / --> <!-- Disabled to avoid jitter -->
+                <mesh filename="file://$(find nerf_standalone)/description/meshes/motor_bracket.stl" scale="0.001 0.001 0.001" />
+            </geometry>
+        </collision>
+    </link>
+    <link name="magazin">
+        <inertial>
+            <origin xyz="-0.0001099393864912468 -0.026417511497997506 0.050134930638840614" rpy="0.0 -0.0 1.3345868986244463e-43" />
+            <mass value="0.3738306581420113" />
+            <inertia ixx="0.0007705630831377967" iyy="0.0005270994299410312" izz="0.00029276667724726724" ixy="-1.4455536319398637e-06" iyz="-3.697688012621039e-06" ixz="-3.532708772950154e-07" />
+        </inertial>
+        <visual name="magazin_visual">
+            <origin xyz="0.009991696360929777 -0.1260585761325394 0.08876880466816899" rpy="-3.141146514736195 1.079162159671481e-15 3.1415267664655997" />
+            <geometry>
+                <mesh filename="file://$(find nerf_standalone)/description/meshes/magazin.stl" scale="0.001 0.001 0.001" />
+            </geometry>
+        </visual>
+        <collision name="magazin_collision">
+            <origin xyz="0.009991696360929777 -0.1260585761325394 0.08876880466816899" rpy="-3.141146514736195 1.079162159671481e-15 3.1415267664655997" />
+            <geometry>
+                <!-- mesh filename="file://$(find nerf_standalone)/description/meshes/magazin.stl" scale="0.001 0.001 0.001" / -->
+            </geometry>
+        </collision>
+    </link>
+    <link name="motor_right">
+        <inertial>
+            <origin xyz="-9.623629244821963e-05 6.345649512652485e-05 -0.00884165710596623" rpy="0.0 -0.0 -1.3345868986244463e-43" />
+            <mass value="0.062400101460318526" />
+            <inertia ixx="4.550449109527322e-06" iyy="4.535524044740256e-06" izz="5.8345867583526245e-06" ixy="-4.341977289852876e-08" iyz="-2.5667746773632163e-08" ixz="3.7561048949347344e-08" />
+        </inertial>
+        <visual name="motor_right_visual">
+            <origin xyz="-1.73567760164417e-09 3.029328534687181e-09 -1.3556827271887785e-09" rpy="-1.5707188555909968 0.00043936100150414944 1.7453951561374372" />
+            <geometry>
+                <mesh filename="file://$(find nerf_standalone)/description/meshes/motor_right.stl" scale="0.001 0.001 0.001" />
+            </geometry>
+        </visual>
+        <collision name="motor_right_collision">
+            <origin xyz="-1.73567760164417e-09 3.029328534687181e-09 -1.3556827271887785e-09" rpy="-1.5707188555909968 0.00043936100150414944 1.7453951561374372" />
+            <geometry>
+                <!-- mesh filename="file://$(find nerf_standalone)/description/meshes/motor_right.stl" scale="0.001 0.001 0.001" / -->
+            </geometry>
+        </collision>
+    </link>
+    <link name="motor_left">
+        <inertial>
+            <origin xyz="9.666486349146908e-09 0.00011354223425985799 -0.008841679450598963" rpy="0.0 -0.0 -1.3345868986244463e-43" />
+            <mass value="0.062400101460318526" />
+            <inertia ixx="4.499632799239714e-06" iyy="4.586322894256146e-06" izz="5.8346042191241955e-06" ixy="7.854576773205486e-09" iyz="-4.5250312344966005e-08" ixz="2.89703028683334e-11" />
+        </inertial>
+        <visual name="motor_left_visual">
+            <origin xyz="-1.8333526696778791e-09 -2.050084864091417e-09 -1.355682762715915e-09" rpy="-1.5711117946140916 0.00031546780349864484 0.7854640007616747" />
+            <geometry>
+                <mesh filename="file://$(find nerf_standalone)/description/meshes/motor_left.stl" scale="0.001 0.001 0.001" />
+            </geometry>
+        </visual>
+        <collision name="motor_left_collision">
+            <origin xyz="-1.8333526696778791e-09 -2.050084864091417e-09 -1.355682762715915e-09" rpy="-1.5711117946140916 0.00031546780349864484 0.7854640007616747" />
+            <geometry>
+                <!-- mesh filename="file://$(find nerf_standalone)/description/meshes/motor_left.stl" scale="0.001 0.001 0.001" / -->
+            </geometry>
+        </collision>
+    </link>
+    <link name="Servo_dart_pusher">
+        <inertial>
+            <origin xyz="0.0049984051741846615 0.024184885243938005 -0.011122220106766214" rpy="0.0 -0.0 1.433307898574046e-40" />
+            <mass value="0.26161409234448435" />
+            <inertia ixx="7.109172214710591e-05" iyy="4.2470781982637245e-05" izz="4.684557684163089e-05" ixy="1.8857294033572383e-09" iyz="-3.575365028985137e-07" ixz="2.3544253511525473e-11" />
+        </inertial>
+        <visual name="Servo_dart_pusher_visual">
+            <origin xyz="0.004998394584003245 0.024345667304006825 -0.010460860261822842" rpy="1.570796326794895 -0.0004461388535984491 -1.5707304396707022" />
+            <geometry>
+                <mesh filename="file://$(find nerf_standalone)/description/meshes/Servo_dart_pusher.stl" scale="0.001 0.001 0.001" />
+            </geometry>
+        </visual>
+        <collision name="Servo_dart_pusher_collision">
+            <origin xyz="0.004998394584003245 0.024345667304006825 -0.010460860261822842" rpy="1.570796326794895 -0.0004461388535984491 -1.5707304396707022" />
+            <geometry>
+                <!-- mesh filename="file://$(find nerf_standalone)/description/meshes/Servo_dart_pusher.stl" scale="0.001 0.001 0.001" / -->
+            </geometry>
+        </collision>
+    </link>
+    <link name="flywheel_left">
+        <inertial>
+            <origin xyz="-3.30024772132731e-08 0.00282389849043422 -1.2643906853559983e-06" rpy="0.0 -0.0 -1.232595164407831e-32" />
+            <mass value="0.05069354299067629" />
+            <inertia ixx="7.100606071477003e-06" iyy="1.1926848369973058e-05" izz="7.100622864546298e-06" ixy="3.0631255872513805e-12" iyz="-2.1531701364196465e-09" ixz="-1.1835077383908058e-08" />
+        </inertial>
+        <visual name="flywheel_left_visual">
+            <origin xyz="-0.0631325544432252 0.01313155884148008 -0.0631300993428637" rpy="-1.570165432787083 0.7853321767598774 -3.1411465441724866" />
+            <geometry>
+                <mesh filename="file://$(find nerf_standalone)/description/meshes/flywheel_left.stl" scale="0.001 0.001 0.001" />
+            </geometry>
+        </visual>
+        <collision name="flywheel_left_collision">
+            <origin xyz="-0.0631325544432252 0.01313155884148008 -0.0631300993428637" rpy="-1.570165432787083 0.7853321767598774 -3.1411465441724866" />
+            <geometry>
+                <!-- mesh filename="file://$(find nerf_standalone)/description/meshes/flywheel_left.stl" scale="0.001 0.001 0.001" / -->
+            </geometry>
+        </collision>
+    </link>
+    <link name="flywheel_right">
+        <inertial>
+            <origin xyz="-2.4884313427619988e-08 0.0028238984826724667 -1.2768684615038773e-06" rpy="0.0 -0.0 0.0" />
+            <mass value="0.05069354299067629" />
+            <inertia ixx="7.1117326126882305e-06" iyy="1.1926848372101947e-05" izz="7.089496321206277e-06" ixy="5.0012536903661526e-12" iyz="-2.15326659632331e-09" ixz="-4.055275447632519e-09" />
+        </inertial>
+        <visual name="flywheel_right_visual">
+            <origin xyz="-0.01550858803514851 0.013120498025483157 -0.08792554788989197" rpy="-1.568228080674074 1.3961969502773832 -3.139063424976714" />
+            <geometry>
+                <mesh filename="file://$(find nerf_standalone)/description/meshes/flywheel_right.stl" scale="0.001 0.001 0.001" />
+            </geometry>
+        </visual>
+        <collision name="flywheel_right_collision">
+            <origin xyz="-0.01550858803514851 0.013120498025483157 -0.08792554788989197" rpy="-1.568228080674074 1.3961969502773832 -3.139063424976714" />
+            <geometry>
+                <!-- mesh filename="file://$(find nerf_standalone)/description/meshes/flywheel_right.stl" scale="0.001 0.001 0.001" / -->
+            </geometry>
+        </collision>
+    </link>
+    <link name="pusher_servo_part">
+        <inertial>
+            <origin xyz="-0.0018390436822625488 -0.0015007596499086952 -3.0219289553024e-06" rpy="0.0 -0.0 0.0" />
+            <mass value="0.01733330859445771" />
+            <inertia ixx="1.2212390623549346e-06" iyy="2.0101597437367823e-06" izz="8.345079203264568e-07" ixy="-6.814032579605754e-09" iyz="-5.46330659846676e-10" ixz="8.808170918442501e-10" />
+        </inertial>
+        <visual name="pusher_servo_part_visual">
+            <origin xyz="5.0358234648939514e-09 -0.0031999983978120905 1.4265863324780527e-06" rpy="-1.5712424656484945 6.588712419531712e-05 9.66531786022265e-16" />
+            <geometry>
+                <mesh filename="file://$(find nerf_standalone)/description/meshes/pusher_servo_part.stl" scale="0.001 0.001 0.001" />
+            </geometry>
+        </visual>
+        <collision name="pusher_servo_part_collision">
+            <origin xyz="5.0358234648939514e-09 -0.0031999983978120905 1.4265863324780527e-06" rpy="-1.5712424656484945 6.588712419531712e-05 9.66531786022265e-16" />
+            <geometry>
+                <!-- mesh filename="file://$(find nerf_standalone)/description/meshes/pusher_servo_part.stl" scale="0.001 0.001 0.001" / -->
+            </geometry>
+        </collision>
+    </link>
+    <link name="Turret">
+        <inertial>
+            <origin xyz="2.3473630047377016e-05 -0.023337529138468247 0.010950166293641102" rpy="0.0 -0.0 1.3345868986244463e-43" />
+            <mass value="0.0611488221940506" />
+            <inertia ixx="2.777243622344256e-05" iyy="4.173856834856703e-06" izz="2.7265059862146765e-05" ixy="-5.4011863057096135e-08" iyz="8.577691363897659e-07" ixz="-1.6482918924949652e-09" />
+        </inertial>
+        <visual name="Turret_visual">
+            <origin xyz="0.0089380699537615 -0.0803571481976858 -0.002142981347950717" rpy="-0.000446138853596889 -1.0791087584284575e-15 -6.58871241935617e-05" />
+            <geometry>
+                <mesh filename="file://$(find nerf_standalone)/description/meshes/Turret.stl" scale="0.001 0.001 0.001" />
+            </geometry>
+        </visual>
+        <collision name="Turret_collision">
+            <origin xyz="0.0089380699537615 -0.0803571481976858 -0.002142981347950717" rpy="-0.000446138853596889 -1.0791087584284575e-15 -6.58871241935617e-05" />
+            <geometry>
+                <!-- mesh filename="file://$(find nerf_standalone)/description/meshes/Turret.stl" scale="0.001 0.001 0.001" / -->
+            </geometry>
+        </collision>
+    </link>
+    <link name="Servoarm-v1">
+        <inertial>
+            <origin xyz="0.0026217000068642538 0.004143996186734538 -0.000121866399240258" rpy="0.0 -0.0 0.0" />
+            <mass value="0.0018742003163414853" />
+            <inertia ixx="6.432185064591283e-08" iyy="8.097740948868152e-09" izz="5.977319996496844e-08" ixy="-2.9381687092850316e-09" iyz="1.5210177440573648e-09" ixz="8.640739219842197e-11" />
+        </inertial>
+        <visual name="Servoarm-v1_visual">
+            <origin xyz="0.004000004389203955 -0.08928319312789187 0.01647600710867764" rpy="0.029400113955168578 -8.659366307345483e-14 -3.141592653583827" />
+            <geometry>
+                <mesh filename="file://$(find nerf_standalone)/description/meshes/Servoarm-v1.stl" scale="0.001 0.001 0.001" />
+            </geometry>
+        </visual>
+        <collision name="Servoarm-v1_collision">
+            <origin xyz="0.004000004389203955 -0.08928319312789187 0.01647600710867764" rpy="0.029400113955168578 -8.659366307345483e-14 -3.141592653583827" />
+            <geometry>
+                <!-- mesh filename="file://$(find nerf_standalone)/description/meshes/Servoarm-v1.stl" scale="0.001 0.001 0.001" / -->
+                <!-- Disabled to isolate collision jitter -->
+            </geometry>
+        </collision>
+    </link>
+    <link name="Nerf-Dart-Launcher_Servo-MG-v1">
+        <inertial>
+            <origin xyz="0.013667304718322098 2.2982730654663718e-06 -0.010985884494499025" rpy="0.0 -7.033867778682351e-39 0.0" />
+            <mass value="0.06129281941203147" />
+            <inertia ixx="4.553097622798822e-06" iyy="6.766608690911323e-06" izz="3.7522386670510236e-06" ixy="6.67505294805216e-10" iyz="-1.8244332424663443e-09" ixz="4.1145466064687034e-07" />
+        </inertial>
+        <visual name="Nerf-Dart-Launcher_Servo-MG-v1_visual">
+            <origin xyz="0.032232880187464355 0.10890697936911703 -0.024499995611303272" rpy="-8.077935669498046e-28 7.226432496549954e-26 1.570796326794921" />
+            <geometry>
+                <mesh filename="file://$(find nerf_standalone)/description/meshes/Nerf-Dart-Launcher_Servo-MG-v1.stl" scale="0.001 0.001 0.001" />
+            </geometry>
+        </visual>
+        <collision name="Nerf-Dart-Launcher_Servo-MG-v1_collision">
+            <origin xyz="0.032232880187464355 0.10890697936911703 -0.024499995611303272" rpy="-8.077935669498046e-28 7.226432496549954e-26 1.570796326794921" />
+            <geometry>
+                <!-- mesh filename="file://$(find nerf_standalone)/description/meshes/Nerf-Dart-Launcher_Servo-MG-v1.stl" scale="0.001 0.001 0.001" / -->
+                <!-- Disabled to isolate collision jitter -->
+            </geometry>
+        </collision>
     </link>
     <joint name="trigger_joint" type="revolute">
-        <!-- <origin xyz="0 0.0975 -0.013768" rpy="3.14159 -1.5708 0"/> -->
-        <origin xyz="0 0 0" rpy="3.14159 -1.5708 0"/>
-        <parent link="Montageplatte"/>
-        <child link="Motor_und_Magazinplatte"/>
-        <axis xyz="-1 0 0"/>
-        <limit lower="0.0" upper="2.1" effort="10.0" velocity="1.0"/>
-        <dynamics damping="0.1" friction="0.1"/>
-    </joint>
-    <link name="Motor_und_Magazinplatte">
-        <visual>
-             <origin xyz="-0.013735 -0.0982192 0.0" rpy="0 0 0"/>
-             <!-- <origin xyz="-0.013735 -0.0991 0.0005" rpy="0 0 0"/> -->
-             <geometry>
-                <mesh filename="file://$(find nerf_standalone)/description/meshes/Motor_und_Magazinplatte.stl" scale="0.001 0.001 0.001"/>
-            </geometry>
-            <material name="grey">
-                <color rgba="0.5 0.5 0.5 1.0"/>
-            </material>
-        </visual>
-        <collision>
-            <origin xyz="0 0 0" rpy="0 0 0"/>
-            <geometry>
-                <box size="0.06 0.08 0.02"/>
-            </geometry>
-        </collision>
-        <inertial>
-            <mass value="0.25"/>
-            <inertia ixx="0.00036" ixy="0" ixz="0" iyy="0.00014" iyz="0" izz="0.00048"/>
-        </inertial>
-    </link>
-    <!-- Motor Left (Fixed to Magazinplatte) -->
-    <!-- Rotated -90 degrees around X (Counter-Clockwise if looking from front? Or standard?) -->
-    <joint name="motor_left_joint" type="fixed">
-        <origin xyz="0.01 -0.09600 0" rpy="-1.5708 3.1416 0"/>
-        <parent link="Motor_und_Magazinplatte"/>
-        <child link="motor_left"/>
-    </joint>
-    <link name="motor_left">
-        <visual>
-            <geometry>
-                <mesh filename="file://$(find nerf_standalone)/description/meshes/motor_left.stl" scale="0.001 0.001 0.001"/>
-            </geometry>
-            <material name="red"/>
-        </visual>
-        <collision>
-            <geometry>
-                <cylinder length="0.03" radius="0.015"/>
-            </geometry>
-        </collision>
-        <inertial>
-            <mass value="0.1"/>
-            <inertia ixx="0.0001" ixy="0" ixz="0" iyy="0.0001" iyz="0" izz="0.0001"/>
-        </inertial>
-    </link>
-    <!-- Motor Right (Fixed to Magazinplatte) -->
-    <joint name="motor_right_joint" type="fixed">
-        <origin xyz="-0.030 -0.0960 0" rpy="-1.5708 3.1416 0"/>
-        <parent link="Motor_und_Magazinplatte"/>
-        <child link="motor_right"/>
-    </joint>
-    <link name="motor_right">
-        <visual>
-            <geometry>
-                <mesh filename="file://$(find nerf_standalone)/description/meshes/motor_right.stl" scale="0.001 0.001 0.001"/>
-            </geometry>
-            <material name="blue"/>
-        </visual>
-        <collision>
-            <geometry>
-                <cylinder length="0.03" radius="0.015"/>
-            </geometry>
-        </collision>
-        <inertial>
-            <mass value="0.1"/>
-            <inertia ixx="0.0001" ixy="0" ixz="0" iyy="0.0001" iyz="0" izz="0.0001"/>
-        </inertial>
-    </link>
-    <!-- Flywheel Left -->
+        <origin xyz="0.08882309 0.10354221000000001 -0.00119223" rpy="-1.5707963267948943 -3.374960801568061e-11 -1.570862213919093" />
+        <parent link="bottom_plate" />
+        <child link="motor_bracket" />
+        <axis xyz="1.1287570791617654e-07 2.227474133869779e-15 1.0000000021779938" />
+        <limit lower="5.235988" upper="6.283185" effort="100.0" velocity="5.0" />
+        <dynamics damping="10.0" friction="5.0"/>
+    </joint>
+    <joint name="motor_bracket_motor_left_fix_motor_bracket" type="fixed">
+        <origin xyz="0.09699999040378247 -4.326999672626883e-05 0.008800001069511083" rpy="1.5707963268286462 -1.5707304396707 3.141592653589793" />
+        <parent link="motor_bracket" />
+        <child link="motor_left" />
+    </joint>
+    <joint name="motor_bracket_motor_right_fix_motor_bracket" type="fixed">
+        <origin xyz="0.09699998532437559 -4.3269996726369024e-05 -0.036199999028498644" rpy="1.5707963268286462 -1.5707304396707 3.141592653589793" />
+        <parent link="motor_bracket" />
+        <child link="motor_right" />
+    </joint>
+    <joint name="flywheel_right_joint" type="continuous">
+        <origin xyz="0.0 -7.800000000000029e-06 -0.0175" rpy="1.5707963267948966 -7.224685652388453e-18 -2.3543024464062444e-21" />
+        <parent link="motor_right" />
+        <child link="flywheel_right" />
+        <axis xyz="-7.22468811426675e-18 -1.0 0.0004460000000000001" />
+        <limit effort="10.0" velocity="100.0"/>
+        <dynamics damping="0.0" friction="0.0"/>
+    </joint>
     <joint name="flywheel_left_joint" type="continuous">
-        <origin xyz="0 0 0.0" rpy="0 0 0"/>
-        <parent link="motor_left"/>
-        <child link="flywheel_left"/>
-        <axis xyz="0 1 0"/>
-        <limit effort="5.0" velocity="100.0"/>
-        <dynamics damping="0.01" friction="0.01"/>
-    </joint>
-    <link name="flywheel_left">
-        <visual>
-            <origin xyz="0.08928 0.002734 0" rpy="-1.5708 0 0"/>
-            <geometry>
-                <mesh filename="file://$(find nerf_standalone)/description/meshes/Launcher_wheel_left.stl" scale="0.001 0.001 0.001"/>
-            </geometry>
-            <material name="red"/>
-        </visual>
-        <collision>
-            <origin xyz="0.08928 0.002734 0" rpy="-1.5708 0 0"/>
-            <geometry>
-                <cylinder length="0.02" radius="0.02"/>
-            </geometry>
-        </collision>
-        <inertial>
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