Commit message: feat: add `nerf_standalone` package with URDF, meshes, control configuration, and firmware, alongside updates to `gubot_one` launch and control settings.

File: src/nerf_standalone/description/urdf/ros2_control.xacro (robot description, xacro)
@@ -2,4 +2,12 @@
 <robot xmlns:xacro="http://www.ros.org/wiki/xacro">
     <xacro:macro name="nerf_ros2_control">
+        <gazebo>
+            <plugin name="gazebo_ros2_control" filename="libgazebo_ros2_control.so">
+                <robot_param>robot_description</robot_param>
+                <robot_param_node>robot_state_publisher</robot_param_node>
+                <parameters>$(find nerf_standalone)/config/controllers.yaml</parameters>
+                <parameters>$(find nerf_standalone)/config/gains.yaml</parameters>
+            </plugin>
+        </gazebo>
         <ros2_control name="GazeboSystem" type="system">
             <hardware>
@@ -9,6 +17,15 @@
                 <command_interface name="position"/>
                 <state_interface name="velocity"/>
+                <state_interface name="position">
+                  <param name="initial_value">5.75</param>
+                </state_interface>
+            </joint>
+            <!-- Pusher Joint (Velocity Control) -->
+            <joint name="dart_pusher_joint">
+                <command_interface name="velocity"/>
+                <state_interface name="velocity"/>
                 <state_interface name="position"/>
             </joint>
+            <!-- Flywheel Left -->
             <joint name="flywheel_left_joint">
                 <command_interface name="velocity"/>
@@ -16,4 +33,5 @@
                 <state_interface name="position"/>
             </joint>
+            <!-- Flywheel Right -->
             <joint name="flywheel_right_joint">
                 <command_interface name="velocity"/>
@@ -21,18 +39,5 @@
                 <state_interface name="position"/>
             </joint>
-            <joint name="dart_pusher_joint">
-                <command_interface name="velocity"/>
-                <state_interface name="velocity"/>
-                <state_interface name="position"/>
-            </joint>
         </ros2_control>
-        <gazebo>
-            <plugin filename="libgazebo_ros2_control.so" name="gazebo_ros2_control">
-                <robot_param>robot_description</robot_param>
-                <robot_param_node>robot_state_publisher</robot_param_node>
-                <parameters>$(find nerf_standalone)/config/controllers.yaml</parameters>
-                <parameters>$(find nerf_standalone)/config/gains.yaml</parameters>
-            </plugin>
-        </gazebo>
     </xacro:macro>
 </robot>

Commit message: feat: Introduce STL analysis tool, simplify URDF collisions and inertias, and add initial position setup for the nerf launcher.

File: src/nerf_standalone/description/urdf/launcher.urdf.xacro (robot description, xacro)
@@ -14,7 +14,7 @@
         </visual>
         <collision name="bottom_plate_collision">
-            <origin xyz="0.0 0.0 0.0" rpy="0.0 0.0 0.0" />
-            <geometry>
-                <mesh filename="file://$(find nerf_standalone)/description/meshes/bottom_plate.stl" scale="0.001 0.001 0.001" />
+            <origin xyz="0.08 0.05 -0.01" rpy="0.0 0.0 0.0" />
+            <geometry>
+                 <box size="0.2 0.15 0.02"/>
             </geometry>
         </collision>
@@ -22,7 +22,7 @@
     <link name="motor_bracket">
         <inertial>
-            <origin xyz="0.06445114377692326 -0.001293871011977803 -0.01805979631895027" rpy="0.0 -7.504780922022523e-26 6.462348535570529e-27" />
-            <mass value="0.24458145922412514" />
-            <inertia ixx="0.00013685810139727812" iyy="0.0004819875327694177" izz="0.0003647641226204775" ixy="-1.2856327940143035e-05" iyz="-1.071289298066829e-05" ixz="-2.0865729712333423e-05" />
+            <origin xyz="0.06 0 0" rpy="0 0 0" />
+            <mass value="0.25" />
+            <inertia ixx="0.001" iyy="0.001" izz="0.001" ixy="0" iyz="0" ixz="0" />
         </inertial>
         <visual name="motor_bracket_visual">
@@ -33,8 +33,8 @@
         </visual>
         <collision name="motor_bracket_collision">
-            <origin xyz="0.09803428669398517 -4.3732793080548534e-05 -0.013700000763976723" rpy="1.5703501879750486 -1.5707963267948937 0" />
-            <geometry>
-                <!-- box size="0.1 0.1 0.1" / --> <!-- Disabled to avoid jitter -->
-                <mesh filename="file://$(find nerf_standalone)/description/meshes/motor_bracket.stl" scale="0.001 0.001 0.001" />
+            <!-- Simplified Box Collision for Tilt Head -->
+            <origin xyz="0.05 0.08 -0.02" rpy="0 0 0" />
+            <geometry>
+                <box size="0.15 0.12 0.08" />
             </geometry>
         </collision>
@@ -42,7 +42,7 @@
     <link name="magazin">
         <inertial>
-            <origin xyz="-0.0001099393864912468 -0.026417511497997506 0.050134930638840614" rpy="0.0 -0.0 1.3345868986244463e-43" />
-            <mass value="0.3738306581420113" />
-            <inertia ixx="0.0007705630831377967" iyy="0.0005270994299410312" izz="0.00029276667724726724" ixy="-1.4455536319398637e-06" iyz="-3.697688012621039e-06" ixz="-3.532708772950154e-07" />
+            <origin xyz="0 -0.02 0.05" rpy="0 0 0" />
+            <mass value="0.4" />
+            <inertia ixx="0.001" iyy="0.001" izz="0.001" ixy="0" iyz="0" ixz="0" />
         </inertial>
         <visual name="magazin_visual">
@@ -52,16 +52,13 @@
             </geometry>
         </visual>
-        <collision name="magazin_collision">
-            <origin xyz="0.009991696360929777 -0.1260585761325394 0.08876880466816899" rpy="-3.141146514736195 1.079162159671481e-15 3.1415267664655997" />
-            <geometry>
-                <!-- mesh filename="file://$(find nerf_standalone)/description/meshes/magazin.stl" scale="0.001 0.001 0.001" / -->
-            </geometry>
-        </collision>
+        <!-- collision name="magazin_collision">
+           Collision disabled
+        </collision -->
     </link>
     <link name="motor_right">
         <inertial>
-            <origin xyz="-9.623629244821963e-05 6.345649512652485e-05 -0.00884165710596623" rpy="0.0 -0.0 -1.3345868986244463e-43" />
-            <mass value="0.062400101460318526" />
-            <inertia ixx="4.550449109527322e-06" iyy="4.535524044740256e-06" izz="5.8345867583526245e-06" ixy="-4.341977289852876e-08" iyz="-2.5667746773632163e-08" ixz="3.7561048949347344e-08" />
+            <origin xyz="0 0 0" rpy="0 0 0" />
+            <mass value="0.1" />
+            <inertia ixx="0.0001" iyy="0.0001" izz="0.0001" ixy="0" iyz="0" ixz="0" />
         </inertial>
         <visual name="motor_right_visual">
@@ -71,16 +68,13 @@
             </geometry>
         </visual>
-        <collision name="motor_right_collision">
-            <origin xyz="-1.73567760164417e-09 3.029328534687181e-09 -1.3556827271887785e-09" rpy="-1.5707188555909968 0.00043936100150414944 1.7453951561374372" />
-            <geometry>
-                <!-- mesh filename="file://$(find nerf_standalone)/description/meshes/motor_right.stl" scale="0.001 0.001 0.001" / -->
-            </geometry>
-        </collision>
+        <!-- collision name="motor_right_collision">
+           Collision disabled
+        </collision -->
     </link>
     <link name="motor_left">
         <inertial>
-            <origin xyz="9.666486349146908e-09 0.00011354223425985799 -0.008841679450598963" rpy="0.0 -0.0 -1.3345868986244463e-43" />
-            <mass value="0.062400101460318526" />
-            <inertia ixx="4.499632799239714e-06" iyy="4.586322894256146e-06" izz="5.8346042191241955e-06" ixy="7.854576773205486e-09" iyz="-4.5250312344966005e-08" ixz="2.89703028683334e-11" />
+            <origin xyz="0 0 0" rpy="0 0 0" />
+            <mass value="0.1" />
+            <inertia ixx="0.0001" iyy="0.0001" izz="0.0001" ixy="0" iyz="0" ixz="0" />
         </inertial>
         <visual name="motor_left_visual">
@@ -90,16 +84,13 @@
             </geometry>
         </visual>
-        <collision name="motor_left_collision">
-            <origin xyz="-1.8333526696778791e-09 -2.050084864091417e-09 -1.355682762715915e-09" rpy="-1.5711117946140916 0.00031546780349864484 0.7854640007616747" />
-            <geometry>
-                <!-- mesh filename="file://$(find nerf_standalone)/description/meshes/motor_left.stl" scale="0.001 0.001 0.001" / -->
-            </geometry>
-        </collision>
+        <!-- collision name="motor_left_collision">
+           Collision disabled
+        </collision -->
     </link>
     <link name="Servo_dart_pusher">
         <inertial>
-            <origin xyz="0.0049984051741846615 0.024184885243938005 -0.011122220106766214" rpy="0.0 -0.0 1.433307898574046e-40" />
-            <mass value="0.26161409234448435" />
-            <inertia ixx="7.109172214710591e-05" iyy="4.2470781982637245e-05" izz="4.684557684163089e-05" ixy="1.8857294033572383e-09" iyz="-3.575365028985137e-07" ixz="2.3544253511525473e-11" />
+            <origin xyz="0 0.02 -0.01" rpy="0 0 0" />
+            <mass value="0.25" />
+            <inertia ixx="0.001" iyy="0.001" izz="0.001" ixy="0" iyz="0" ixz="0" />
         </inertial>
         <visual name="Servo_dart_pusher_visual">
@@ -109,16 +100,13 @@
             </geometry>
         </visual>
-        <collision name="Servo_dart_pusher_collision">
-            <origin xyz="0.004998394584003245 0.024345667304006825 -0.010460860261822842" rpy="1.570796326794895 -0.0004461388535984491 -1.5707304396707022" />
-            <geometry>
-                <!-- mesh filename="file://$(find nerf_standalone)/description/meshes/Servo_dart_pusher.stl" scale="0.001 0.001 0.001" / -->
-            </geometry>
-        </collision>
+        <!-- collision name="Servo_dart_pusher_collision">
+           Collision disabled
+        </collision -->
     </link>
     <link name="flywheel_left">
         <inertial>
-            <origin xyz="-3.30024772132731e-08 0.00282389849043422 -1.2643906853559983e-06" rpy="0.0 -0.0 -1.232595164407831e-32" />
-            <mass value="0.05069354299067629" />
-            <inertia ixx="7.100606071477003e-06" iyy="1.1926848369973058e-05" izz="7.100622864546298e-06" ixy="3.0631255872513805e-12" iyz="-2.1531701364196465e-09" ixz="-1.1835077383908058e-08" />
+            <origin xyz="0 0.003 0" rpy="0 0 0" />
+            <mass value="0.1" />
+            <inertia ixx="0.0001" iyy="0.0001" izz="0.0001" ixy="0" iyz="0" ixz="0" />
         </inertial>
         <visual name="flywheel_left_visual">
@@ -128,16 +116,13 @@
             </geometry>
         </visual>
-        <collision name="flywheel_left_collision">
-            <origin xyz="-0.0631325544432252 0.01313155884148008 -0.0631300993428637" rpy="-1.570165432787083 0.7853321767598774 -3.1411465441724866" />
-            <geometry>
-                <!-- mesh filename="file://$(find nerf_standalone)/description/meshes/flywheel_left.stl" scale="0.001 0.001 0.001" / -->
-            </geometry>
-        </collision>
+        <!-- collision name="flywheel_left_collision">
+           Collision disabled
+        </collision -->
     </link>
     <link name="flywheel_right">
         <inertial>
-            <origin xyz="-2.4884313427619988e-08 0.0028238984826724667 -1.2768684615038773e-06" rpy="0.0 -0.0 0.0" />
-            <mass value="0.05069354299067629" />
-            <inertia ixx="7.1117326126882305e-06" iyy="1.1926848372101947e-05" izz="7.089496321206277e-06" ixy="5.0012536903661526e-12" iyz="-2.15326659632331e-09" ixz="-4.055275447632519e-09" />
+            <origin xyz="0 0.003 0" rpy="0 0 0" />
+            <mass value="0.1" />
+            <inertia ixx="0.0001" iyy="0.0001" izz="0.0001" ixy="0" iyz="0" ixz="0" />
         </inertial>
         <visual name="flywheel_right_visual">
@@ -147,16 +132,13 @@
             </geometry>
         </visual>
-        <collision name="flywheel_right_collision">
-            <origin xyz="-0.01550858803514851 0.013120498025483157 -0.08792554788989197" rpy="-1.568228080674074 1.3961969502773832 -3.139063424976714" />
-            <geometry>
-                <!-- mesh filename="file://$(find nerf_standalone)/description/meshes/flywheel_right.stl" scale="0.001 0.001 0.001" / -->
-            </geometry>
-        </collision>
+        <!-- collision name="flywheel_right_collision">
+           Collision disabled
+        </collision -->
     </link>
     <link name="pusher_servo_part">
         <inertial>
-            <origin xyz="-0.0018390436822625488 -0.0015007596499086952 -3.0219289553024e-06" rpy="0.0 -0.0 0.0" />
-            <mass value="0.01733330859445771" />
-            <inertia ixx="1.2212390623549346e-06" iyy="2.0101597437367823e-06" izz="8.345079203264568e-07" ixy="-6.814032579605754e-09" iyz="-5.46330659846676e-10" ixz="8.808170918442501e-10" />
+            <origin xyz="-0.002 -0.002 0" rpy="0 0 0" />
+            <mass value="0.05" />
+            <inertia ixx="0.0001" iyy="0.0001" izz="0.0001" ixy="0" iyz="0" ixz="0" />
         </inertial>
         <visual name="pusher_servo_part_visual">
@@ -166,16 +148,13 @@
             </geometry>
         </visual>
-        <collision name="pusher_servo_part_collision">
-            <origin xyz="5.0358234648939514e-09 -0.0031999983978120905 1.4265863324780527e-06" rpy="-1.5712424656484945 6.588712419531712e-05 9.66531786022265e-16" />
-            <geometry>
-                <!-- mesh filename="file://$(find nerf_standalone)/description/meshes/pusher_servo_part.stl" scale="0.001 0.001 0.001" / -->
-            </geometry>
-        </collision>
+        <!-- collision name="pusher_servo_part_collision">
+           Collision disabled
+        </collision -->
     </link>
     <link name="Turret">
         <inertial>
-            <origin xyz="2.3473630047377016e-05 -0.023337529138468247 0.010950166293641102" rpy="0.0 -0.0 1.3345868986244463e-43" />
-            <mass value="0.0611488221940506" />
-            <inertia ixx="2.777243622344256e-05" iyy="4.173856834856703e-06" izz="2.7265059862146765e-05" ixy="-5.4011863057096135e-08" iyz="8.577691363897659e-07" ixz="-1.6482918924949652e-09" />
+            <origin xyz="0 -0.02 0.01" rpy="0 0 0" />
+            <mass value="0.1" />
+            <inertia ixx="0.0001" iyy="0.0001" izz="0.0001" ixy="0" iyz="0" ixz="0" />
         </inertial>
         <visual name="Turret_visual">
@@ -185,16 +164,13 @@
             </geometry>
         </visual>
-        <collision name="Turret_collision">
-            <origin xyz="0.0089380699537615 -0.0803571481976858 -0.002142981347950717" rpy="-0.000446138853596889 -1.0791087584284575e-15 -6.58871241935617e-05" />
-            <geometry>
-                <!-- mesh filename="file://$(find nerf_standalone)/description/meshes/Turret.stl" scale="0.001 0.001 0.001" / -->
-            </geometry>
-        </collision>
+        <!-- collision name="Turret_collision">
+           Collision disabled
+        </collision -->
     </link>
     <link name="Servoarm-v1">
         <inertial>
-            <origin xyz="0.0026217000068642538 0.004143996186734538 -0.000121866399240258" rpy="0.0 -0.0 0.0" />
-            <mass value="0.0018742003163414853" />
-            <inertia ixx="6.432185064591283e-08" iyy="8.097740948868152e-09" izz="5.977319996496844e-08" ixy="-2.9381687092850316e-09" iyz="1.5210177440573648e-09" ixz="8.640739219842197e-11" />
+            <origin xyz="0.003 0.004 0" rpy="0 0 0" />
+            <mass value="0.05" />
+            <inertia ixx="0.0001" iyy="0.0001" izz="0.0001" ixy="0" iyz="0" ixz="0" />
         </inertial>
         <visual name="Servoarm-v1_visual">
@@ -204,17 +180,13 @@
             </geometry>
         </visual>
-        <collision name="Servoarm-v1_collision">
-            <origin xyz="0.004000004389203955 -0.08928319312789187 0.01647600710867764" rpy="0.029400113955168578 -8.659366307345483e-14 -3.141592653583827" />
-            <geometry>
-                <!-- mesh filename="file://$(find nerf_standalone)/description/meshes/Servoarm-v1.stl" scale="0.001 0.001 0.001" / -->
-                <!-- Disabled to isolate collision jitter -->
-            </geometry>
-        </collision>
+        <!-- collision name="Servoarm-v1_collision">
+           Collision disabled
+        </collision -->
     </link>
     <link name="Nerf-Dart-Launcher_Servo-MG-v1">
         <inertial>
-            <origin xyz="0.013667304718322098 2.2982730654663718e-06 -0.010985884494499025" rpy="0.0 -7.033867778682351e-39 0.0" />
-            <mass value="0.06129281941203147" />
-            <inertia ixx="4.553097622798822e-06" iyy="6.766608690911323e-06" izz="3.7522386670510236e-06" ixy="6.67505294805216e-10" iyz="-1.8244332424663443e-09" ixz="4.1145466064687034e-07" />
+            <origin xyz="0.01 0 -0.01" rpy="0 0 0" />
+            <mass value="0.1" />
+            <inertia ixx="0.0001" iyy="0.0001" izz="0.0001" ixy="0" iyz="0" ixz="0" />
         </inertial>
         <visual name="Nerf-Dart-Launcher_Servo-MG-v1_visual">
@@ -224,11 +196,7 @@
             </geometry>
         </visual>
-        <collision name="Nerf-Dart-Launcher_Servo-MG-v1_collision">
-            <origin xyz="0.032232880187464355 0.10890697936911703 -0.024499995611303272" rpy="-8.077935669498046e-28 7.226432496549954e-26 1.570796326794921" />
-            <geometry>
-                <!-- mesh filename="file://$(find nerf_standalone)/description/meshes/Nerf-Dart-Launcher_Servo-MG-v1.stl" scale="0.001 0.001 0.001" / -->
-                <!-- Disabled to isolate collision jitter -->
-            </geometry>
-        </collision>
+        <!-- collision name="Nerf-Dart-Launcher_Servo-MG-v1_collision">
+           Collision disabled
+        </collision -->
     </link>
     <joint name="trigger_joint" type="revolute">

File: src/nerf_standalone/description/urdf/ros2_control.xacro (robot description, xacro)
@@ -18,5 +18,5 @@
                 <state_interface name="velocity"/>
                 <state_interface name="position">
-                  <param name="initial_value">5.75</param>
+                  <param name="initial_value">6.28</param>
                 </state_interface>
             </joint>

Commit message: feat: Implement ROS2 control hardware interface and firmware for the Nerf blaster.

File: src/nerf_standalone/description/urdf/launcher.urdf.xacro (robot description, xacro)
@@ -274,5 +274,20 @@
         <origin xyz="0 0 0.5" rpy="0 0 0"/>
     </joint>
+    <xacro:arg name="use_hardware" default="false"/>
+    <xacro:if value="$(arg use_hardware)">
+        <xacro:include filename="ros2_control_hardware.xacro" />
+        <xacro:nerf_ros2_control_hardware />
+    </xacro:if>
+    <xacro:unless value="$(arg use_hardware)">
+        <link name="arming_switch_link" />
+    <joint name="system_arming_joint" type="revolute">
+        <parent link="bottom_plate"/>
+        <child link="arming_switch_link"/>
+        <origin xyz="0 0 0" rpy="0 0 0"/>
+        <limit lower="0" upper="1" effort="1" velocity="1"/>
+        <axis xyz="0 0 1"/>
+    </joint>
     <xacro:include filename="ros2_control.xacro" />
-    <xacro:nerf_ros2_control />
+        <xacro:nerf_ros2_control />
+    </xacro:unless>
 </robot>

Commit message: feat: Add STL mesh analysis tool and improve simulation launch stability by delaying controller spawning.

File: src/nerf_standalone/description/urdf/launcher.urdf.xacro (robot description, xacro)
@@ -268,10 +268,14 @@
         <child link="Servoarm-v1" />
     </joint>
-    <link name="world"/>
-    <joint name="world_to_base" type="fixed">
-        <parent link="world"/>
-        <child link="bottom_plate"/>
-        <origin xyz="0 0 0.5" rpy="0 0 0"/>
-    </joint>
+    <!-- World link and joint - only for standalone mode -->
+    <xacro:arg name="integrated_mode" default="false"/>
+    <xacro:unless value="$(arg integrated_mode)">
+        <link name="world"/>
+        <joint name="world_to_base" type="fixed">
+            <parent link="world"/>
+            <child link="bottom_plate"/>
+            <origin xyz="0 0 0.5" rpy="0 0 0"/>
+        </joint>
+    </xacro:unless>
     <xacro:arg name="use_hardware" default="false"/>
     <xacro:if value="$(arg use_hardware)">

File: src/nerf_standalone/description/urdf/ros2_control.xacro (robot description, xacro)
@@ -1,4 +1,5 @@
 <?xml version="1.0"?>
 <robot xmlns:xacro="http://www.ros.org/wiki/xacro">
+    <!-- Full ros2_control macro with gazebo plugin - for standalone mode -->
     <xacro:macro name="nerf_ros2_control">
         <gazebo>
@@ -41,3 +42,31 @@
         </ros2_control>
     </xacro:macro>
+    <!-- Joints-only macro for integration mode (no gazebo plugin) -->
+    <xacro:macro name="nerf_ros2_control_joints_only">
+        <joint name="trigger_joint">
+            <command_interface name="position"/>
+            <state_interface name="velocity"/>
+            <state_interface name="position">
+              <param name="initial_value">6.28</param>
+            </state_interface>
+        </joint>
+        <!-- Pusher Joint (Velocity Control) -->
+        <joint name="dart_pusher_joint">
+            <command_interface name="velocity"/>
+            <state_interface name="velocity"/>
+            <state_interface name="position"/>
+        </joint>
+        <!-- Flywheel Left -->
+        <joint name="flywheel_left_joint">
+            <command_interface name="velocity"/>
+            <state_interface name="velocity"/>
+            <state_interface name="position"/>
+        </joint>
+        <!-- Flywheel Right -->
+        <joint name="flywheel_right_joint">
+            <command_interface name="velocity"/>
+            <state_interface name="velocity"/>
+            <state_interface name="position"/>
+        </joint>
+    </xacro:macro>
 </robot>

Commit message: feat: Integrate `nerf_control_node`, parameterize hardware serial ports for both Pico and Nerf, and update deployment instructions.

File: src/nerf_standalone/description/urdf/launcher.urdf.xacro (robot description, xacro)
@@ -246,7 +246,8 @@
     </xacro:unless>
     <xacro:arg name="use_hardware" default="false"/>
+    <xacro:arg name="port" default="/dev/ttyACM0"/>
     <xacro:if value="$(arg use_hardware)">
         <xacro:include filename="ros2_control_hardware.xacro" />
-        <xacro:nerf_ros2_control_hardware />
+        <xacro:nerf_ros2_control_hardware port="$(arg port)"/>
     </xacro:if>
     <xacro:unless value="$(arg use_hardware)">

File: src/nerf_standalone/description/urdf/ros2_control_hardware.xacro (robot description, xacro)
@@ -1,9 +1,9 @@
 <?xml version="1.0"?>
 <robot xmlns:xacro="http://www.ros.org/wiki/xacro">
-    <xacro:macro name="nerf_ros2_control_hardware">
+    <xacro:macro name="nerf_ros2_control_hardware" params="port">
         <ros2_control name="NerfSystem" type="system">
             <hardware>
                 <plugin>nerf_standalone/NerfSystem</plugin>
-                <param name="port">/dev/ttyACM0</param>
+                <param name="port">$(arg port)</param>
                 <param name="baud_rate">115200</param>
             </hardware>
