Commit message: feat: Implement Nerf launcher teleoperation and joystick control, refine robot URDF, and add STL analysis utility.

File: src/gubot_one/description/robot.urdf.xacro (robot description, xacro)
@@ -14,4 +14,4 @@
     <!-- include filename="depth_camera.xacro" -->
     <xacro:include filename="face.xacro" />
-        <xacro:include filename="nerf_launcher.xacro" />
+    <!-- <xacro:include filename="nerf_launcher.xacro" /> -->
 </robot>

File: src/gubot_one/description/robot_core.xacro (robot description, xacro)
@@ -33,13 +33,16 @@
         <color rgba="1 0 0 1"/>
     </material>
+    <!-- BASE FOOTPRINT (Root Link) -->
+    <link name="base_footprint">
+    </link>
+    <!-- BASE LINK (Offset up by wheel radius) -->
+        <joint name="base_footprint_joint" type="fixed">
+        <parent link="base_footprint"/>
+        <child link="base_link"/>
+        <origin xyz="0 0 ${wheel_radius}"/>
+    </joint>
     <link name="base_link">
     </link>
-    <joint name="base_footprint_joint" type="fixed">
-        <parent link="base_link"/>
-        <child link="base_footprint"/>
-        <origin xyz="0 0 0" rpy="0 0 0"/>
-    </joint>
-    <link name="base_footprint">
-    </link>
+    <!-- CHASSIS -->
     <joint name="chassis_joint" type="fixed">
         <parent link="base_link"/>
@@ -86,5 +89,5 @@
         <collision>
             <geometry>
-                <sphere radius="${wheel_radius}"/>
+                <cylinder length="${wheel_thickness}" radius="${wheel_radius}"/>
             </geometry>
         </collision>
@@ -99,5 +102,5 @@
         <parent link="base_link"/>
         <child link="right_wheel"/>
-        <origin xyz="0 ${-wheel_offset_y} 0" rpy="${pi/2} 0 0" />
+        <origin xyz="0 ${-wheel_offset_y} 0" rpy="-${pi/2} 0 0" />
         <axis xyz="0 0 -1"/>
         <limit effort="10.0" velocity="10.0"/>
@@ -114,5 +117,5 @@
         <collision>
             <geometry>
-                <sphere radius="${wheel_radius}"/>
+                <cylinder length="${wheel_thickness}" radius="${wheel_radius}"/>
             </geometry>
         </collision>
@@ -132,5 +135,5 @@
         <visual>
             <geometry>
-                <sphere radius="${caster_wheel_radius}"/>
+                <sphere radius="0.03"/>
             </geometry>
             <material name="white"/>
@@ -138,8 +141,8 @@
         <collision>
             <geometry>
-                <sphere radius="${caster_wheel_radius}"/>
+                <sphere radius="0.03"/>
             </geometry>
         </collision>
-        <xacro:inertial_sphere mass="${caster_wheel_mass}" radius="${caster_wheel_radius}">
+        <xacro:inertial_sphere mass="0.05" radius="0.03">
             <origin xyz="0 0 0" rpy="0 0 0"/>
         </xacro:inertial_sphere>
@@ -147,6 +150,4 @@
     <gazebo reference="caster_wheel">
         <material>Gazebo/White</material>
-        <mu1 value="0.001"/>
-        <mu2 value="0.001"/>
     </gazebo>
 </robot>

Commit message: feat: Add support for Nerf hardware integration and update launch configurations

File: src/gubot_one/description/robot.urdf.xacro (robot description, xacro)
@@ -4,4 +4,6 @@
     <xacro:arg name="sim_mode" default="false"/>
     <xacro:arg name="integrated_mode" default="true"/>
+    <xacro:arg name="use_nerf_hardware" default="true"/>
+    <xacro:arg name="nerf_port" default="/dev/serial/by-id/usb-Arduino_LLC_Arduino_Leonardo-if00"/>
     <xacro:include filename="robot_core.xacro" />
     <xacro:if value="$(arg use_ros2_control)">

File: src/gubot_one/description/ros2_control.xacro (robot description, xacro)
@@ -1,4 +1,6 @@
 <?xml version="1.0"?>
 <robot xmlns:xacro="http://www.ros.org/wiki/xacro">
+    <xacro:arg name="use_nerf_hardware" default="true"/>
+    <xacro:arg name="nerf_port" default="/dev/serial/by-id/usb-Arduino_LLC_Arduino_Leonardo-if00"/>
     <xacro:unless value="$(arg sim_mode)">
         <ros2_control name="RealRobot" type="system">
@@ -30,30 +32,32 @@
             </joint>
         </ros2_control>
-        <ros2_control name="NerfSystem" type="system">
-            <hardware>
-                <plugin>nerf_standalone/NerfSystem</plugin>
-                <param name="port">/dev/serial/by-id/usb-Arduino_LLC_Arduino_Leonardo-if00</param>
-                <param name="baud_rate">115200</param>
-            </hardware>
-            <joint name="trigger_joint">
-                <command_interface name="position"/>
-                <state_interface name="position"/>
-            </joint>
-            <joint name="dart_pusher_joint">
-                <command_interface name="velocity"/>
-                <state_interface name="velocity"/>
-            </joint>
-            <joint name="flywheel_left_joint">
-                <command_interface name="velocity"/>
-                <state_interface name="velocity"/>
-            </joint>
-            <joint name="flywheel_right_joint">
-                <command_interface name="velocity"/>
-                <state_interface name="velocity"/>
-            </joint>
-            <joint name="system_arming_joint">
-                <command_interface name="position"/>
-            </joint>
-        </ros2_control>
+        <xacro:if value="$(arg use_nerf_hardware)">
+            <ros2_control name="NerfSystem" type="system">
+                <hardware>
+                    <plugin>nerf_standalone/NerfSystem</plugin>
+                    <param name="port">$(arg nerf_port)</param>
+                    <param name="baud_rate">115200</param>
+                </hardware>
+                <joint name="trigger_joint">
+                    <command_interface name="position"/>
+                    <state_interface name="position"/>
+                </joint>
+                <joint name="dart_pusher_joint">
+                    <command_interface name="velocity"/>
+                    <state_interface name="velocity"/>
+                </joint>
+                <joint name="flywheel_left_joint">
+                    <command_interface name="velocity"/>
+                    <state_interface name="velocity"/>
+                </joint>
+                <joint name="flywheel_right_joint">
+                    <command_interface name="velocity"/>
+                    <state_interface name="velocity"/>
+                </joint>
+                <joint name="system_arming_joint">
+                    <command_interface name="position"/>
+                </joint>
+            </ros2_control>
+        </xacro:if>
     </xacro:unless>
     <xacro:if value="$(arg sim_mode)">
