Commit message: feat: update robot_core.xacro and launch_sim.launch.py for improved package structure and world argument configuration

File: src/gubot_one/description/robot_core.xacro (robot description, xacro)
@@ -1,5 +1,10 @@
 <?xml version="1.0"?>
 <robot xmlns:xacro="http://www.ros.org/wiki/xacro" >
+    <!-- Packages -->
+    <xacro:property name="package_share_dir" value="$(find gubot_one)"/>
+    <!-- Including files -->
+    <xacro:property name="package_share_dir" value="$(find gubot_one)"/>
     <xacro:include filename="inertial_macros.xacro"/>
+    <!-- Variablen -->
     <xacro:property name="chassis_length" value="0.335"/>
     <xacro:property name="chassis_width" value="0.265"/>
@@ -16,4 +21,6 @@
     <xacro:property name="caster_wheel_offset_x" value="0.075"/>
     <xacro:property name="caster_wheel_offset_z" value="${wheel_offset_z - wheel_radius + caster_wheel_radius}"/>
+    <xacro:property name="mesh_scale" value="0.001 0.001 0.001"/>
+    <!-- Colors -->
     <material name="white">
         <color rgba="1 1 1 1" />
@@ -54,5 +61,6 @@
             <origin xyz="${chassis_length/2} 0 0" rpy="0 0 0"/>
             <geometry>
-                <mesh filename="package://gubot_one/meshes/bases/waffle_pi_base.stl" scale="0.001 0.001 0.001"/>
+                <mesh filename="file://${package_share_dir}/meshes/bases/waffle_pi_base.stl" scale="${mesh_scale}"/>
+                <!-- <mesh filename="file://${package_share_dir}/meshes/bases/waffle_pi_base.stl" scale="0.001 0.001 0.001"/> -->
             </geometry>
             <material name="orange"/>
@@ -84,5 +92,5 @@
             <origin xyz="0 0 0" rpy="${pi/2} 0 0"/>
             <geometry>
-                <mesh filename="package://gubot_one/meshes/wheels/mecanum_a.dae"/>
+                <mesh filename="file://${package_share_dir}/meshes/wheels/mecanum_a.dae"/>
             </geometry>
             <material name="blue"/>
@@ -113,5 +121,5 @@
             <origin xyz="0 0 0" rpy="${pi/2} 0 0"/>
             <geometry>
-                <mesh filename="package://gubot_one/meshes/wheels/mecanum_b.dae"/>
+                <mesh filename="file://${package_share_dir}/meshes/wheels/mecanum_b.dae"/>
             </geometry>
             <material name="blue"/>

Commit message: feat: Add ICM-20948 IMU drivers and integration for diffdrive Arduino,

File: src/gubot_one/description/robot_core.xacro (robot description, xacro)
@@ -69,4 +69,92 @@
         <material>Gazebo/Orange</material>
     </gazebo>
+    <!-- IMU LINK -->
+    <joint name="imu_joint" type="fixed">
+        <parent link="chassis"/>
+        <child link="imu_link"/>
+        <origin xyz="0 0 0.05" rpy="0 0 0"/>
+    </joint>
+    <gazebo reference="imu_joint">
+        <disableFixedJointLumping>true</disableFixedJointLumping>
+    </gazebo>
+    <link name="imu_link">
+        <visual>
+            <geometry>
+                <box size="0.02 0.02 0.02"/>
+            </geometry>
+            <material name="black"/>
+        </visual>
+        <collision>
+            <geometry>
+                <box size="0.02 0.02 0.02"/>
+            </geometry>
+        </collision>
+        <xacro:inertial_box mass="0.01" x="0.02" y="0.02" z="0.02">
+            <origin xyz="0 0 0" rpy="0 0 0"/>
+        </xacro:inertial_box>
+    </link>
+    <gazebo reference="imu_link">
+        <material>Gazebo/Black</material>
+        <sensor name="imu_sensor" type="imu">
+            <always_on>true</always_on>
+            <update_rate>50</update_rate>
+            <visualize>false</visualize>
+            <topic>imu_sensor/imu_data</topic>
+            <imu>
+                <angular_velocity>
+                    <x>
+                        <noise type="gaussian">
+                            <mean>0.0</mean>
+                            <stddev>0.0002</stddev>
+                            <bias_mean>0.0000075</bias_mean>
+                            <bias_stddev>0.0000008</bias_stddev>
+                        </noise>
+                    </x>
+                    <y>
+                        <noise type="gaussian">
+                            <mean>0.0</mean>
+                            <stddev>0.0002</stddev>
+                            <bias_mean>0.0000075</bias_mean>
+                            <bias_stddev>0.0000008</bias_stddev>
+                        </noise>
+                    </y>
+                    <z>
+                        <noise type="gaussian">
+                            <mean>0.0</mean>
+                            <stddev>0.0002</stddev>
+                            <bias_mean>0.0000075</bias_mean>
+                            <bias_stddev>0.0000008</bias_stddev>
+                        </noise>
+                    </z>
+                </angular_velocity>
+                <linear_acceleration>
+                    <x>
+                        <noise type="gaussian">
+                            <mean>0.0</mean>
+                            <stddev>0.017</stddev>
+                            <bias_mean>0.1</bias_mean>
+                            <bias_stddev>0.001</bias_stddev>
+                        </noise>
+                    </x>
+                    <y>
+                        <noise type="gaussian">
+                            <mean>0.0</mean>
+                            <stddev>0.017</stddev>
+                            <bias_mean>0.1</bias_mean>
+                            <bias_stddev>0.001</bias_stddev>
+                        </noise>
+                    </y>
+                    <z>
+                        <noise type="gaussian">
+                            <mean>0.0</mean>
+                            <stddev>0.017</stddev>
+                            <bias_mean>0.1</bias_mean>
+                            <bias_stddev>0.001</bias_stddev>
+                        </noise>
+                    </z>
+                </linear_acceleration>
+            </imu>
+        </sensor>
+    </gazebo>
     <!-- LEFT WHEEL LINK -->
     <joint name="left_wheel_joint" type="continuous">

File: src/gubot_one/description/ros2_control.xacro (robot description, xacro)
@@ -11,5 +11,5 @@
                 <param name="loop_rate">30</param>
                 <param name="device">/dev/serial/by-id/usb-Raspberry_Pi_Pico_50443405786ACA1C-if00</param>
-                <param name="baud_rate">57600</param>
+                <param name="baud_rate">115200</param>
                 <param name="timeout_ms">1000</param>
                 <param name="enc_counts_per_rev">3436</param>
@@ -31,4 +31,12 @@
                 <state_interface name="velocity"/>
             </joint>
+            <sensor name="imu_sensor">
+                <state_interface name="linear_acceleration.x"/>
+                <state_interface name="linear_acceleration.y"/>
+                <state_interface name="linear_acceleration.z"/>
+                <state_interface name="angular_velocity.x"/>
+                <state_interface name="angular_velocity.y"/>
+                <state_interface name="angular_velocity.z"/>
+            </sensor>
         </ros2_control>
         <xacro:if value="$(arg use_nerf_hardware)">
@@ -107,4 +115,16 @@
                 <state_interface name="position"/>
             </joint>
+            <sensor name="imu_sensor">
+                <state_interface name="linear_acceleration.x"/>
+                <state_interface name="linear_acceleration.y"/>
+                <state_interface name="linear_acceleration.z"/>
+                <state_interface name="angular_velocity.x"/>
+                <state_interface name="angular_velocity.y"/>
+                <state_interface name="angular_velocity.z"/>
+                <state_interface name="orientation.x"/>
+                <state_interface name="orientation.y"/>
+                <state_interface name="orientation.z"/>
+                <state_interface name="orientation.w"/>
+            </sensor>
         </ros2_control>
     </xacro:if>
