Commit message: added gazebo classic back to repo

File: src/gubot_one/description/camera.xacro (robot description, xacro)
@@ -33,5 +33,4 @@
             <visualize>false</visualize>
             <update_rate>10</update_rate>
-            <topic>camera/image_raw</topic>
             <camera>
                 <horizontal_fov>1.089</horizontal_fov>
@@ -46,4 +45,12 @@
                 </clip>
             </camera>
+            <xacro:if value="$(arg use_gazebo_classic)">
+                <plugin name="camera_controller" filename="libgazebo_ros_camera.so">
+                    <frame_name>camera_link_optical</frame_name>
+                </plugin>
+            </xacro:if>
+            <xacro:unless value="$(arg use_gazebo_classic)">
+                <topic>camera/image_raw</topic>
+            </xacro:unless>
         </sensor>
     </gazebo>

File: src/gubot_one/description/lidar.xacro (robot description, xacro)
@@ -31,26 +31,56 @@
     <gazebo reference="laser_frame">
         <material>Gazebo/Black</material>
-        <sensor name="laser" type="gpu_lidar">
-            <pose> 0 0 0 0 0 0 </pose>
-            <visualize>false</visualize>
-            <update_rate>10</update_rate>
-            <topic>scan</topic>
-            <lidar>
-                <scan>
-                    <horizontal>
-                        <samples>360</samples>
-                        <resolution>1</resolution>
-                        <min_angle>-3.14</min_angle>
-                        <max_angle>3.14</max_angle>
-                    </horizontal>
-                </scan>
-                <range>
-                    <min>0.3</min>
-                    <max>12</max>
-                    <resolution>0.01</resolution>
-                </range>
-            </lidar>
-            <!-- Ignition handles publishing via Bridge, so no plugin needed here -->
-        </sensor>
+        <xacro:if value="$(arg use_gazebo_classic)">
+            <sensor name="laser" type="ray">
+                <pose> 0 0 0 0 0 0 </pose>
+                <visualize>true</visualize>
+                <update_rate>10</update_rate>
+                <ray>
+                    <scan>
+                        <horizontal>
+                            <samples>360</samples>
+                            <resolution>1</resolution>
+                            <min_angle>-3.14</min_angle>
+                            <max_angle>3.14</max_angle>
+                        </horizontal>
+                    </scan>
+                    <range>
+                        <min>0.3</min>
+                        <max>12</max>
+                        <resolution>0.01</resolution>
+                    </range>
+                </ray>
+                <plugin name="laser_controller" filename="libgazebo_ros_ray_sensor.so">
+                    <ros>
+                        <remapping>~/out:=/scan</remapping>
+                    </ros>
+                    <output_type>sensor_msgs/LaserScan</output_type>
+                    <frame_name>laser_frame</frame_name>
+                </plugin>
+            </sensor>
+        </xacro:if>
+        <xacro:unless value="$(arg use_gazebo_classic)">
+            <sensor name="laser" type="gpu_lidar">
+                <pose> 0 0 0 0 0 0 </pose>
+                <visualize>false</visualize>
+                <update_rate>10</update_rate>
+                <topic>scan</topic>
+                <lidar>
+                    <scan>
+                        <horizontal>
+                            <samples>360</samples>
+                            <resolution>1</resolution>
+                            <min_angle>-3.14</min_angle>
+                            <max_angle>3.14</max_angle>
+                        </horizontal>
+                    </scan>
+                    <range>
+                        <min>0.3</min>
+                        <max>12</max>
+                        <resolution>0.01</resolution>
+                    </range>
+                </lidar>
+            </sensor>
+        </xacro:unless>
     </gazebo>
 </robot>

File: src/gubot_one/description/robot.urdf.xacro (robot description, xacro)
@@ -6,7 +6,13 @@
     <xacro:arg name="use_nerf_hardware" default="true"/>
     <xacro:arg name="nerf_port" default="/dev/serial/by-id/usb-Arduino_LLC_Arduino_Leonardo-if00"/>
+    <xacro:arg name="use_gazebo_classic" default="false"/>
     <xacro:include filename="robot_core.xacro" />
     <xacro:if value="$(arg use_ros2_control)">
-        <xacro:include filename="ros2_control.xacro" />
+        <xacro:if value="$(arg use_gazebo_classic)">
+            <xacro:include filename="gz_classic_ros2_control.xacro" />
+        </xacro:if>
+        <xacro:unless value="$(arg use_gazebo_classic)">
+            <xacro:include filename="ros2_control.xacro" />
+        </xacro:unless>
     </xacro:if>
     <xacro:unless value="$(arg use_ros2_control)">

File: src/gubot_one/description/robot_core.xacro (robot description, xacro)
@@ -62,5 +62,5 @@
             </geometry>
         </collision>
-        <xacro:inertial_box mass="0.5" x="${chassis_length}" y="${chassis_width}" z="${chassis_height}">
+        <xacro:inertial_box mass="${chassis_mass}" x="${chassis_length}" y="${chassis_width}" z="${chassis_height}">
             <origin xyz="${chassis_length/2} 0 ${chassis_height/2}" rpy="0 0 0"/>
         </xacro:inertial_box>
@@ -100,5 +100,4 @@
             <update_rate>50</update_rate>
             <visualize>false</visualize>
-            <topic>imu_sensor/imu_data</topic>
             <imu>
                 <angular_velocity>
@@ -155,4 +154,15 @@
                 </linear_acceleration>
             </imu>
+            <xacro:if value="$(arg use_gazebo_classic)">
+                <plugin name="imu_plugin" filename="libgazebo_ros_imu_sensor.so">
+                    <ros>
+                        <remapping>~/out:=imu/data</remapping>
+                    </ros>
+                    <initial_orientation_as_reference>false</initial_orientation_as_reference>
+                </plugin>
+            </xacro:if>
+            <xacro:unless value="$(arg use_gazebo_classic)">
+                <topic>imu_sensor/imu_data</topic>
+            </xacro:unless>
         </sensor>
     </gazebo>
@@ -182,4 +192,10 @@
     <gazebo reference="left_wheel">
         <material>Gazebo/Blue</material>
+        <mu1 value="1.0"/>
+        <mu2 value="1.0"/>
+        <kp value="1000000.0" />
+        <kd value="10.0" />
+        <fdir1 value="1 0 0"/>
+        <minDepth>0.001</minDepth>
     </gazebo>
     <!-- RIGHT WHEEL LINK -->
@@ -208,4 +224,10 @@
     <gazebo reference="right_wheel">
         <material>Gazebo/Blue</material>
+        <mu1 value="1.0"/>
+        <mu2 value="1.0"/>
+        <kp value="1000000.0" />
+        <kd value="10.0" />
+        <fdir1 value="1 0 0"/>
+        <minDepth>0.001</minDepth>
     </gazebo>
     <!-- CASTER WHEEL LINK -->

File: src/nerf_standalone/description/urdf/launcher.urdf.xacro (robot description, xacro)
@@ -4,6 +4,6 @@
         <inertial>
             <origin xyz="0.07506008367977571 0.06788755296524361 -0.015949194976296238" rpy="0.0 0.0 0.0" />
-            <mass value="0.04" />
-            <inertia ixx="0.00037557930532003186" iyy="5.362127850969058e-05" izz="0.00041640489807794057" ixy="-1.2945646322185759e-06" iyz="-1.5574886339585816e-05" ixz="9.440243990688213e-08" />
+            <mass value="0.1" />
+            <inertia ixx="0.001" iyy="0.001" izz="0.001" ixy="0.0" iyz="0.0" ixz="0.0" />
         </inertial>
         <visual name="bottom_plate_visual">
@@ -14,7 +14,7 @@
         </visual>
         <collision name="bottom_plate_collision">
-            <origin xyz="0.08 0.05 -0.01" rpy="0.0 0.0 0.0" />
-            <geometry>
-                 <box size="0.2 0.15 0.02"/>
+            <origin xyz="0.08 0.05 0.05" rpy="0.0 0.0 0.0" />
+            <geometry>
+                 <box size="0.25 0.20 0.20"/>
             </geometry>
         </collision>
@@ -23,6 +23,6 @@
         <inertial>
             <origin xyz="0.06 0 0" rpy="0 0 0" />
-            <mass value="0.03" />
-            <inertia ixx="0.001" iyy="0.001" izz="0.001" ixy="0" iyz="0" ixz="0" />
+            <mass value="0.1" />
+            <inertia ixx="0.001" iyy="0.001" izz="0.001" ixy="0.0" iyz="0.0" ixz="0.0" />
         </inertial>
         <visual name="motor_bracket_visual">
@@ -32,16 +32,10 @@
             </geometry>
         </visual>
-        <collision name="motor_bracket_collision">
-            <origin xyz="0.05 0.08 -0.02" rpy="0 0 0" />
-            <geometry>
-                <box size="0.15 0.12 0.08" />
-            </geometry>
-        </collision>
     </link>
     <link name="magazin">
         <inertial>
             <origin xyz="0 -0.02 0.05" rpy="0 0 0" />
-            <mass value="0.03" />
-            <inertia ixx="0.001" iyy="0.001" izz="0.001" ixy="0" iyz="0" ixz="0" />
+            <mass value="0.1" />
+            <inertia ixx="0.001" iyy="0.001" izz="0.001" ixy="0.0" iyz="0.0" ixz="0.0" />
         </inertial>
         <visual name="magazin_visual">
@@ -55,6 +49,6 @@
         <inertial>
             <origin xyz="0 0 0" rpy="0 0 0" />
-            <mass value="0.01" />
-            <inertia ixx="0.0001" iyy="0.0001" izz="0.0001" ixy="0" iyz="0" ixz="0" />
+            <mass value="0.1" />
+            <inertia ixx="0.001" iyy="0.001" izz="0.001" ixy="0.0" iyz="0.0" ixz="0.0" />
         </inertial>
         <visual name="motor_right_visual">
@@ -68,6 +62,6 @@
         <inertial>
             <origin xyz="0 0 0" rpy="0 0 0" />
-            <mass value="0.01" />
-            <inertia ixx="0.0001" iyy="0.0001" izz="0.0001" ixy="0" iyz="0" ixz="0" />
+            <mass value="0.1" />
+            <inertia ixx="0.001" iyy="0.001" izz="0.001" ixy="0.0" iyz="0.0" ixz="0.0" />
         </inertial>
         <visual name="motor_left_visual">
@@ -81,6 +75,6 @@
         <inertial>
             <origin xyz="0 0.02 -0.01" rpy="0 0 0" />
-            <mass value="0.02" />
-            <inertia ixx="0.001" iyy="0.001" izz="0.001" ixy="0" iyz="0" ixz="0" />
+            <mass value="0.1" />
+            <inertia ixx="0.001" iyy="0.001" izz="0.001" ixy="0.0" iyz="0.0" ixz="0.0" />
         </inertial>
         <visual name="Servo_dart_pusher_visual">
@@ -94,6 +88,6 @@
         <inertial>
             <origin xyz="0 0.003 0" rpy="0 0 0" />
-            <mass value="0.01" />
-            <inertia ixx="0.0001" iyy="0.0001" izz="0.0001" ixy="0" iyz="0" ixz="0" />
+            <mass value="0.1" />
+            <inertia ixx="0.001" iyy="0.001" izz="0.001" ixy="0.0" iyz="0.0" ixz="0.0" />
         </inertial>
         <visual name="flywheel_left_visual">
@@ -107,6 +101,6 @@
         <inertial>
             <origin xyz="0 0.003 0" rpy="0 0 0" />
-            <mass value="0.01" />
-            <inertia ixx="0.0001" iyy="0.0001" izz="0.0001" ixy="0" iyz="0" ixz="0" />
+            <mass value="0.1" />
+            <inertia ixx="0.001" iyy="0.001" izz="0.001" ixy="0.0" iyz="0.0" ixz="0.0" />
         </inertial>
         <visual name="flywheel_right_visual">
@@ -120,6 +114,6 @@
         <inertial>
             <origin xyz="-0.002 -0.002 0" rpy="0 0 0" />
-            <mass value="0.01" />
-            <inertia ixx="0.000001" iyy="0.000001" izz="0.000001" ixy="0" iyz="0" ixz="0" />
+            <mass value="0.1" />
+            <inertia ixx="0.001" iyy="0.001" izz="0.001" ixy="0.0" iyz="0.0" ixz="0.0" />
         </inertial>
         <visual name="pusher_servo_part_visual">
@@ -133,6 +127,6 @@
         <inertial>
             <origin xyz="0 -0.02 0.01" rpy="0 0 0" />
-            <mass value="0.01" />
-            <inertia ixx="0.0001" iyy="0.0001" izz="0.0001" ixy="0" iyz="0" ixz="0" />
+            <mass value="0.1" />
+            <inertia ixx="0.001" iyy="0.001" izz="0.001" ixy="0.0" iyz="0.0" ixz="0.0" />
         </inertial>
         <visual name="Turret_visual">
@@ -146,6 +140,6 @@
         <inertial>
             <origin xyz="0.003 0.004 0" rpy="0 0 0" />
-            <mass value="0.01" />
-            <inertia ixx="0.0001" iyy="0.0001" izz="0.0001" ixy="0" iyz="0" ixz="0" />
+            <mass value="0.1" />
+            <inertia ixx="0.001" iyy="0.001" izz="0.001" ixy="0.0" iyz="0.0" ixz="0.0" />
         </inertial>
         <visual name="Servoarm-v1_visual">
@@ -159,6 +153,6 @@
         <inertial>
             <origin xyz="0.01 0 -0.01" rpy="0 0 0" />
-            <mass value="0.01" />
-            <inertia ixx="0.0001" iyy="0.0001" izz="0.0001" ixy="0" iyz="0" ixz="0" />
+            <mass value="0.1" />
+            <inertia ixx="0.001" iyy="0.001" izz="0.001" ixy="0.0" iyz="0.0" ixz="0.0" />
         </inertial>
         <visual name="Nerf-Dart-Launcher_Servo-MG-v1_visual">
@@ -254,6 +248,6 @@
         <link name="arming_switch_link">
             <inertial>
-                <mass value="0.01" />
-                <inertia ixx="0.0001" ixy="0.0" ixz="0.0" iyy="0.0001" iyz="0.0" izz="0.0001" />
+                <mass value="0.1" />
+                <inertia ixx="0.001" iyy="0.001" izz="0.001" ixy="0.0" iyz="0.0" ixz="0.0" />
             </inertial>
         </link>
@@ -266,5 +260,11 @@
     </joint>
     <xacro:unless value="$(arg integrated_mode)">
-        <xacro:include filename="ros2_control.xacro" />
+        <xacro:arg name="use_gazebo_classic" default="false"/>
+        <xacro:if value="$(arg use_gazebo_classic)">
+            <xacro:include filename="gz_classic_ros2_control.xacro" />
+        </xacro:if>
+        <xacro:unless value="$(arg use_gazebo_classic)">
+            <xacro:include filename="ros2_control.xacro" />
+        </xacro:unless>
         <xacro:nerf_ros2_control />
     </xacro:unless>
