Commit message: feat: Update serial commands for hardware deactivation and improve code formatting.

File: src/gubot_one/description/ros2_control.xacro (robot description, xacro)
@@ -28,4 +28,30 @@
                 <state_interface name="velocity"/>
                 <state_interface name="position"/>
+            </joint>
+        </ros2_control>
+        <ros2_control name="NerfSystem" type="system">
+            <hardware>
+                <plugin>nerf_standalone/NerfSystem</plugin>
+                <param name="port">/dev/ttyACM0</param>
+                <param name="baud_rate">115200</param>
+            </hardware>
+            <joint name="trigger_joint">
+                <command_interface name="position"/>
+                <state_interface name="position"/>
+            </joint>
+            <joint name="dart_pusher_joint">
+                <command_interface name="velocity"/>
+                <state_interface name="velocity"/>
+            </joint>
+            <joint name="flywheel_left_joint">
+                <command_interface name="velocity"/>
+                <state_interface name="velocity"/>
+            </joint>
+            <joint name="flywheel_right_joint">
+                <command_interface name="velocity"/>
+                <state_interface name="velocity"/>
+            </joint>
+            <joint name="system_arming_joint">
+                <command_interface name="position"/>
             </joint>
         </ros2_control>

File: src/nerf_standalone/description/urdf/ros2_control_hardware.xacro (robot description, xacro)
@@ -5,5 +5,5 @@
             <hardware>
                 <plugin>nerf_standalone/NerfSystem</plugin>
-                <param name="port">/dev/ttyUSB0</param>
+                <param name="port">/dev/ttyACM0</param>
                 <param name="baud_rate">115200</param>
             </hardware>

Commit message: feat: Replace ball tracking with face tracking, updating associated configurations, control interfaces, and launch parameters.

File: src/gubot_one/description/ros2_control.xacro (robot description, xacro)
@@ -47,19 +47,11 @@
                     <param name="baud_rate">115200</param>
                 </hardware>
-                <joint name="trigger_joint">
+                <joint name="tilt_joint">
                     <command_interface name="position"/>
                     <state_interface name="position"/>
                 </joint>
-                <joint name="dart_pusher_joint">
-                    <command_interface name="velocity"/>
-                    <state_interface name="velocity"/>
-                </joint>
-                <joint name="flywheel_left_joint">
-                    <command_interface name="velocity"/>
-                    <state_interface name="velocity"/>
-                </joint>
-                <joint name="flywheel_right_joint">
-                    <command_interface name="velocity"/>
-                    <state_interface name="velocity"/>
+                <joint name="shooter_joint">
+                    <command_interface name="position"/>
+                    <state_interface name="position"/>
                 </joint>
                 <joint name="system_arming_joint">

Commit message: feat: add position state interface for system arming joint and update flywheel joint types to fixed.

File: src/gubot_one/description/ros2_control.xacro (robot description, xacro)
@@ -57,4 +57,5 @@
                 <joint name="system_arming_joint">
                     <command_interface name="position"/>
+                    <state_interface name="position"/>
                 </joint>
             </ros2_control>

File: src/nerf_launch_system/description/urdf/launcher.urdf.xacro (robot description, xacro)
@@ -194,19 +194,13 @@
         <child link="motor_right" />
     </joint>
-    <joint name="flywheel_right_joint" type="continuous">
+    <joint name="flywheel_right_joint" type="fixed">
         <origin xyz="0.0 -7.800000000000029e-06 -0.0175" rpy="1.5707963267948966 -7.224685652388453e-18 -2.3543024464062444e-21" />
         <parent link="motor_right" />
         <child link="flywheel_right" />
-        <axis xyz="-7.22468811426675e-18 -1.0 0.0004460000000000001" />
-        <limit effort="10.0" velocity="100.0"/>
-        <dynamics damping="0.0" friction="0.0"/>
-    </joint>
-    <joint name="flywheel_left_joint" type="continuous">
+    </joint>
+    <joint name="flywheel_left_joint" type="fixed">
         <origin xyz="0.0 -7.810000000000317e-06 -0.0175" rpy="1.5707963267948966 -1.0870161501361781e-16 -2.35430244640625e-21" />
         <parent link="motor_left" />
         <child link="flywheel_left" />
-        <axis xyz="-1.0870161747549608e-16 -0.9999999999999999 0.000446" />
-        <limit effort="10.0" velocity="100.0"/>
-        <dynamics damping="0.0" friction="0.0"/>
     </joint>
     <joint name="motor_bracket_torret_on_motor_bracket" type="fixed">

Commit message: docs: Add comprehensive documentation for robot description, nodes, and hardware interfaces, alongside updates to RVIZ, `ros2_control` XACRO, and simulation launch files.

File: src/gubot_one/description/ros2_control.xacro (robot description, xacro)
@@ -118,13 +118,10 @@
                 <state_interface name="position"/>
             </joint>
-            <joint name="trigger_joint">
+            <joint name="tilt_joint">
                 <command_interface name="position"/>
-                <state_interface name="position">
-                  <param name="initial_value">6.28</param>
-                </state_interface>
+                <state_interface name="position"/>
             </joint>
-            <joint name="dart_pusher_joint">
-                <command_interface name="velocity"/>
-                <state_interface name="velocity"/>
+            <joint name="shooter_joint">
+                <command_interface name="position"/>
                 <state_interface name="position"/>
             </joint>
