Commit message: feat: update ros2_control interfaces for launcher, adjust Gazebo environment variables, and refine collision/IMU geometries.

File: src/gubot_one/description/gz_classic_ros2_control.xacro (robot description, xacro)
@@ -90,4 +90,5 @@
                 <state_interface name="position"/>
             </joint>
+            <!--
             <joint name="trigger_joint">
                 <command_interface name="position"/>
@@ -101,4 +102,18 @@
                 <state_interface name="position"/>
             </joint>
+            -->
+            <joint name="tilt_joint">
+                <command_interface name="position"/>
+                <state_interface name="position">
+                    <param name="initial_value">6.28</param>
+                </state_interface>
+            </joint>
+            <joint name="shooter_joint">
+                <command_interface name="position"/>
+                <state_interface name="position">
+                    <param name="initial_value">0.0</param>
+                </state_interface>
+            </joint>
+            <!--
             <joint name="flywheel_left_joint">
                 <command_interface name="velocity"/>
@@ -111,7 +126,10 @@
                 <state_interface name="position"/>
             </joint>
+            -->
             <joint name="system_arming_joint">
                 <command_interface name="position"/>
-                <state_interface name="position"/>
+                <state_interface name="position">
+                    <param name="initial_value">0.0</param>
+                </state_interface>
             </joint>
             <sensor name="imu_sensor">
@@ -129,5 +147,5 @@
         </ros2_control>
     </xacro:if>
- <gazebo>
+    <gazebo>
         <plugin filename="libgazebo_ros2_control.so" name="gazebo_ros2_control">
             <parameters>$(find gubot_one)/config/my_controllers.yaml</parameters>

File: src/gubot_one/description/robot_core.xacro (robot description, xacro)
@@ -1,4 +1,4 @@
 <?xml version="1.0"?>
-<robot xmlns:xacro="http://www.ros.org/wiki/xacro" >
+<robot xmlns:xacro="http://www.ros.org/wiki/xacro">
     <xacro:include filename="inertial_macros.xacro"/>
     <xacro:property name="chassis_length" value="0.335"/>
@@ -73,5 +73,5 @@
         <parent link="chassis"/>
         <child link="imu_link"/>
-        <origin xyz="0 0 0.05" rpy="0 0 0"/>
+        <origin xyz="0 0 0.148" rpy="0 0 0"/>
     </joint>
     <gazebo reference="imu_joint">

File: src/nerf_launch_system/description/urdf/gz_classic_ros2_control.xacro (robot description, xacro)
@@ -11,9 +11,10 @@
                 <plugin>gazebo_ros2_control/GazeboSystem</plugin>
             </hardware>
+            <!--
             <joint name="trigger_joint">
                 <command_interface name="position"/>
                 <state_interface name="velocity"/>
                 <state_interface name="position">
-                  <param name="initial_value">6.28</param>
+                    <param name="initial_value">6.28</param>
                 </state_interface>
             </joint>
@@ -22,6 +23,6 @@
                 <state_interface name="velocity"/>
                 <state_interface name="position"/>
-            </joint>
-            <joint name="flywheel_left_joint">
+            </joint> -->
+            <!-- <joint name="flywheel_left_joint">
                 <command_interface name="velocity"/>
                 <state_interface name="velocity"/>
@@ -31,4 +32,12 @@
                 <command_interface name="velocity"/>
                 <state_interface name="velocity"/>
+                <state_interface name="position"/>
+            </joint> -->
+            <joint name="tilt_joint">
+                <command_interface name="position"/>
+                <state_interface name="position"/>
+            </joint>
+            <joint name="shooter_joint">
+                <command_interface name="position"/>
                 <state_interface name="position"/>
             </joint>
@@ -44,5 +53,5 @@
             <state_interface name="velocity"/>
             <state_interface name="position">
-              <param name="initial_value">6.28</param>
+                <param name="initial_value">6.28</param>
             </state_interface>
         </joint>

File: src/nerf_launch_system/description/urdf/launcher.urdf.xacro (robot description, xacro)
@@ -27,7 +27,7 @@
         </visual>
         <collision name="bottom_plate_collision">
-            <origin xyz="0.08 0.05 0.05" rpy="0.0 0.0 0.0" />
-            <geometry>
-                 <box size="0.25 0.20 0.20"/>
+            <origin xyz="0.08 0.05 0.01" rpy="0.0 0.0 0.0" />
+            <geometry>
+                <box size="0.25 0.20 0.02"/>
             </geometry>
         </collision>

Commit message: Refactor tilt controller integration and improve simulation launch
- Updated `gz_classic_launch_sim.launch.py` to change the z-coordinate for the entity from 0.1 to 0.2 and added `use_sim_time` parameter to RViz launch.
- Modified `joystick.launch.py` to introduce a new launch configuration for `tilt_command_topic` and adjusted remappings for joystick commands.
- Enhanced `launch_sim.launch.py` to implement a TimerAction for delayed spawners, ensuring proper initialization of controllers after the entity spawn.
- Added a new debug script `debug_tilt.py` for testing tilt controller functionality and verifying joint states.
- Updated `nerf_teleop.py` to adjust tilt position limits and initial values to align with new URDF constraints.
- Removed deprecated `nerf_topic_compat.py` as the new topic structure is now in use.
- Created regression tests in `test_tilt_controller_spawner.py` to validate tilt joint configuration and controller settings.
- Adjusted URDF definitions in `launcher.urdf.xacro` to reflect new joint limits and dynamics settings.
- Modified `test.sh` to streamline testing commands.

File: src/gubot_one/description/gz_classic_ros2_control.xacro (robot description, xacro)
@@ -93,5 +93,6 @@
                 <command_interface name="position"/>
                 <state_interface name="position">
-                  <param name="initial_value">6.28</param>
+                  <!-- ALT: <param name="initial_value">6.28</param> -->
+                  <param name="initial_value">0.0</param>
                 </state_interface>
             </joint>

File: src/gubot_one/description/nerf_launcher.xacro (robot description, xacro)
@@ -4,9 +4,10 @@
     <xacro:include filename="$(find nerf_launch_system)/description/urdf/launcher.urdf.xacro" />
     <joint name="nerf_mount_joint" type="fixed">
-    <parent link="chassis"/>
-    <child link="bottom_plate"/>
-    <origin xyz="0.155 0 0.165" rpy="0 0 ${pi/2}"/> </joint>
+        <parent link="chassis"/>
+        <child link="bottom_plate"/>
+        <origin xyz="0.155 0 0.165" rpy="0 0 ${pi/2}"/>
+    </joint>
     <gazebo reference="nerf_mount_joint">
-        <preserveFixedJoint>true</preserveFixedJoint>
+        <preserveFixedJoint>false</preserveFixedJoint>
     </gazebo>
 </robot>

File: src/gubot_one/description/ros2_control.xacro (robot description, xacro)
@@ -72,5 +72,9 @@
         <ros2_control name="IgnitionSystem" type="system">
             <hardware>
+                <!-- ALT: <plugin>gz_ros2_control/GazeboSimSystem</plugin> -->
                 <plugin>ign_ros2_control/IgnitionSystem</plugin>
+                <!-- ALT: In GZ Sim war der Default (0.1) zu schwach fuer sichtbare Tilt-Bewegung -->
+                <!-- ALT: <param name="position_proportional_gain">8.0</param> -->
+                <param name="position_proportional_gain">20.0</param>
             </hardware>
             <joint name="left_wheel_joint">
@@ -91,7 +95,13 @@
             </joint>
             <joint name="trigger_joint">
-                <command_interface name="position"/>
+                <command_interface name="position">
+                    <!-- ADDED FOR IGN_ROS2_CONTROL PID POSITION TRACKING -->
+                    <param name="p">50.0</param>
+                    <param name="d">1.0</param>
+                </command_interface>
                 <state_interface name="position">
-                  <param name="initial_value">6.28</param>
+                    <!-- ALT: <param name="initial_value">0.0</param> -->
+                    <!-- ALT: <param name="initial_value">6.28</param> -->
+                    <param name="initial_value">0.0</param>
                 </state_interface>
             </joint>
@@ -129,5 +139,6 @@
         </ros2_control>
     </xacro:if>
- <gazebo>
+    <gazebo>
+        <!-- ALT: <plugin filename="gz_ros2_control-system" name="gz_ros2_control::GazeboSimROS2ControlPlugin"> -->
         <plugin filename="ign_ros2_control-system" name="ign_ros2_control::IgnitionROS2ControlPlugin">
             <parameters>$(find gubot_one)/config/my_controllers.yaml</parameters>

File: src/nerf_launch_system/description/urdf/launcher.urdf.xacro (robot description, xacro)
@@ -14,7 +14,7 @@
         </visual>
         <collision name="bottom_plate_collision">
-            <origin xyz="0.08 0.05 0.05" rpy="0.0 0.0 0.0" />
-            <geometry>
-                 <box size="0.25 0.20 0.20"/>
+            <origin xyz="0.075 0.0 -0.015" rpy="0.0 0.0 0.0" />
+            <geometry>
+                <box size="0.17 0.12 0.03"/>
             </geometry>
         </collision>
@@ -168,6 +168,9 @@
         <child link="motor_bracket" />
         <axis xyz="1.1287570791617654e-07 2.227474133869779e-15 1.0000000021779938" />
-        <limit lower="5.23" upper="6.28" effort="1.0" velocity="5.0" />
-        <dynamics damping="10.0" friction="5.0"/>
+        <!-- ALT: <limit lower="-1.05" upper="0.0" effort="10.0" velocity="5.0" /> -->
+        <!-- ALT: <limit lower="5.23" upper="6.28" effort="10.0" velocity="5.0" /> -->
+        <!-- ALT: <limit lower="-1.05" upper="0.0" effort="10.0" velocity="5.0" /> -->
+        <limit lower="-0.52" upper="0.52" effort="10.0" velocity="5.0" />
+        <dynamics damping="0.2" friction="0.05"/>
     </joint>
     <joint name="motor_bracket_motor_left_fix_motor_bracket" type="fixed">
@@ -181,19 +184,13 @@
         <child link="motor_right" />
     </joint>
-    <joint name="flywheel_right_joint" type="continuous">
+    <joint name="flywheel_right_joint" type="fixed">
         <origin xyz="0.0 -7.800000000000029e-06 -0.0175" rpy="1.5707963267948966 -7.224685652388453e-18 -2.3543024464062444e-21" />
         <parent link="motor_right" />
         <child link="flywheel_right" />
-        <axis xyz="-7.22468811426675e-18 -1.0 0.0004460000000000001" />
-        <limit effort="10.0" velocity="100.0"/>
-        <dynamics damping="0.0" friction="0.0"/>
-    </joint>
-    <joint name="flywheel_left_joint" type="continuous">
+    </joint>
+    <joint name="flywheel_left_joint" type="fixed">
         <origin xyz="0.0 -7.810000000000317e-06 -0.0175" rpy="1.5707963267948966 -1.0870161501361781e-16 -2.35430244640625e-21" />
         <parent link="motor_left" />
         <child link="flywheel_left" />
-        <axis xyz="-1.0870161747549608e-16 -0.9999999999999999 0.000446" />
-        <limit effort="10.0" velocity="100.0"/>
-        <dynamics damping="0.0" friction="0.0"/>
     </joint>
     <joint name="motor_bracket_torret_on_motor_bracket" type="fixed">
@@ -218,5 +215,5 @@
         <axis xyz="-2.7546953265439552e-21 1.0 -0.000446" />
         <limit effort="0.1" velocity="20.0"/>
-        <dynamics damping="0.0" friction="0.0"/>
+        <dynamics damping="0.05" friction="0.01"/>
     </joint>
     <joint name="bottom_plate_servo_fix_bottom_plate" type="fixed">
@@ -252,21 +249,21 @@
             </inertial>
         </link>
-    <joint name="system_arming_joint" type="revolute">
-        <parent link="bottom_plate"/>
-        <child link="arming_switch_link"/>
-        <origin xyz="0 0 0" rpy="0 0 0"/>
-        <limit lower="0" upper="1" effort="1" velocity="1"/>
-        <axis xyz="0 0 1"/>
-    </joint>
-    <xacro:unless value="$(arg integrated_mode)">
-        <xacro:arg name="use_gazebo_classic" default="false"/>
-        <xacro:if value="$(arg use_gazebo_classic)">
-            <xacro:include filename="gz_classic_ros2_control.xacro" />
-        </xacro:if>
-        <xacro:unless value="$(arg use_gazebo_classic)">
-            <xacro:include filename="ros2_control.xacro" />
+        <joint name="system_arming_joint" type="revolute">
+            <parent link="bottom_plate"/>
+            <child link="arming_switch_link"/>
+            <origin xyz="0 0 0" rpy="0 0 0"/>
+            <limit lower="0" upper="1" effort="1" velocity="1"/>
+            <axis xyz="0 0 1"/>
+        </joint>
+        <xacro:unless value="$(arg integrated_mode)">
+            <xacro:arg name="use_gazebo_classic" default="false"/>
+            <xacro:if value="$(arg use_gazebo_classic)">
+                <xacro:include filename="gz_classic_ros2_control.xacro" />
+            </xacro:if>
+            <xacro:unless value="$(arg use_gazebo_classic)">
+                <xacro:include filename="ros2_control.xacro" />
+            </xacro:unless>
+            <xacro:nerf_ros2_control />
         </xacro:unless>
-        <xacro:nerf_ros2_control />
-    </xacro:unless>
     </xacro:unless>
 </robot>

Commit message: feat: Bereinigung und Optimierung von XACRO-Dateien für Robotermodell und Simulation

File: src/gubot_one/description/gz_classic_ros2_control.xacro (robot description, xacro)
@@ -93,6 +93,5 @@
                 <command_interface name="position"/>
                 <state_interface name="position">
-                  <!-- ALT: <param name="initial_value">6.28</param> -->
-                  <param name="initial_value">0.0</param>
+                    <param name="initial_value">0.0</param>
                 </state_interface>
             </joint>
@@ -130,5 +129,5 @@
         </ros2_control>
     </xacro:if>
- <gazebo>
+    <gazebo>
         <plugin filename="libgazebo_ros2_control.so" name="gazebo_ros2_control">
             <parameters>$(find gubot_one)/config/my_controllers.yaml</parameters>

File: src/gubot_one/description/ros2_control.xacro (robot description, xacro)
@@ -72,8 +72,5 @@
         <ros2_control name="IgnitionSystem" type="system">
             <hardware>
-                <!-- ALT: <plugin>gz_ros2_control/GazeboSimSystem</plugin> -->
                 <plugin>ign_ros2_control/IgnitionSystem</plugin>
-                <!-- ALT: In GZ Sim war der Default (0.1) zu schwach fuer sichtbare Tilt-Bewegung -->
-                <!-- ALT: <param name="position_proportional_gain">8.0</param> -->
                 <param name="position_proportional_gain">20.0</param>
             </hardware>
@@ -96,11 +93,8 @@
             <joint name="trigger_joint">
                 <command_interface name="position">
-                    <!-- ADDED FOR IGN_ROS2_CONTROL PID POSITION TRACKING -->
                     <param name="p">50.0</param>
                     <param name="d">1.0</param>
                 </command_interface>
                 <state_interface name="position">
-                    <!-- ALT: <param name="initial_value">0.0</param> -->
-                    <!-- ALT: <param name="initial_value">6.28</param> -->
                     <param name="initial_value">0.0</param>
                 </state_interface>
@@ -140,5 +134,4 @@
     </xacro:if>
     <gazebo>
-        <!-- ALT: <plugin filename="gz_ros2_control-system" name="gz_ros2_control::GazeboSimROS2ControlPlugin"> -->
         <plugin filename="ign_ros2_control-system" name="ign_ros2_control::IgnitionROS2ControlPlugin">
             <parameters>$(find gubot_one)/config/my_controllers.yaml</parameters>

File: src/nerf_launch_system/description/urdf/launcher.urdf.xacro (robot description, xacro)
@@ -168,7 +168,4 @@
         <child link="motor_bracket" />
         <axis xyz="1.1287570791617654e-07 2.227474133869779e-15 1.0000000021779938" />
-        <!-- ALT: <limit lower="-1.05" upper="0.0" effort="10.0" velocity="5.0" /> -->
-        <!-- ALT: <limit lower="5.23" upper="6.28" effort="10.0" velocity="5.0" /> -->
-        <!-- ALT: <limit lower="-1.05" upper="0.0" effort="10.0" velocity="5.0" /> -->
         <limit lower="-0.52" upper="0.52" effort="10.0" velocity="5.0" />
         <dynamics damping="0.2" friction="0.05"/>
