Commit message: feat: Refine `gubot_one` and `nerf_launcher` URDF definitions by removing `nerf_standalone` export assets and tuning physics parameters.

File: src/gubot_one/description/nerf_launcher.xacro (robot description, xacro)
@@ -4,8 +4,7 @@
     <xacro:include filename="$(find nerf_standalone)/description/urdf/launcher.urdf.xacro" />
     <joint name="nerf_mount_joint" type="fixed">
-        <parent link="chassis"/>
-        <child link="bottom_plate"/>
-        <origin xyz="0.16 0 0.15" rpy="0 0 0"/>
-    </joint>
+    <parent link="chassis"/>
+    <child link="bottom_plate"/>
+    <origin xyz="0.155 0 0.15" rpy="0 0 ${pi/2}"/> </joint>
     <gazebo reference="nerf_mount_joint">
         <preserveFixedJoint>true</preserveFixedJoint>

File: src/gubot_one/description/robot.urdf.xacro (robot description, xacro)
@@ -3,4 +3,5 @@
     <xacro:arg name="use_ros2_control" default="true"/>
     <xacro:arg name="sim_mode" default="false"/>
+    <xacro:arg name="integrated_mode" default="true"/>
     <xacro:include filename="robot_core.xacro" />
     <xacro:if value="$(arg use_ros2_control)">
@@ -14,4 +15,4 @@
     <!-- include filename="depth_camera.xacro" -->
     <xacro:include filename="face.xacro" />
-    <!-- <xacro:include filename="nerf_launcher.xacro" /> -->
+    <xacro:include filename="nerf_launcher.xacro" />
 </robot>

File: src/gubot_one/description/ros2_control.xacro (robot description, xacro)
@@ -54,7 +54,6 @@
             <joint name="trigger_joint">
                 <command_interface name="position"/>
-                <state_interface name="velocity"/>
                 <state_interface name="position">
-                  <param name="initial_value">6.28</param>
+                  <param name="initial_value">0.0</param>
                 </state_interface>
             </joint>

File: src/nerf_standalone/description/urdf/launcher.urdf.xacro (robot description, xacro)
@@ -4,5 +4,5 @@
         <inertial>
             <origin xyz="0.07506008367977571 0.06788755296524361 -0.015949194976296238" rpy="0.0 0.0 0.0" />
-            <mass value="0.2021986172178209" />
+            <mass value="0.04" />
             <inertia ixx="0.00037557930532003186" iyy="5.362127850969058e-05" izz="0.00041640489807794057" ixy="-1.2945646322185759e-06" iyz="-1.5574886339585816e-05" ixz="9.440243990688213e-08" />
         </inertial>
@@ -23,5 +23,5 @@
         <inertial>
             <origin xyz="0.06 0 0" rpy="0 0 0" />
-            <mass value="0.25" />
+            <mass value="0.03" />
             <inertia ixx="0.001" iyy="0.001" izz="0.001" ixy="0" iyz="0" ixz="0" />
         </inertial>
@@ -42,5 +42,5 @@
         <inertial>
             <origin xyz="0 -0.02 0.05" rpy="0 0 0" />
-            <mass value="0.4" />
+            <mass value="0.03" />
             <inertia ixx="0.001" iyy="0.001" izz="0.001" ixy="0" iyz="0" ixz="0" />
         </inertial>
@@ -55,5 +55,5 @@
         <inertial>
             <origin xyz="0 0 0" rpy="0 0 0" />
-            <mass value="0.1" />
+            <mass value="0.01" />
             <inertia ixx="0.0001" iyy="0.0001" izz="0.0001" ixy="0" iyz="0" ixz="0" />
         </inertial>
@@ -68,5 +68,5 @@
         <inertial>
             <origin xyz="0 0 0" rpy="0 0 0" />
-            <mass value="0.1" />
+            <mass value="0.01" />
             <inertia ixx="0.0001" iyy="0.0001" izz="0.0001" ixy="0" iyz="0" ixz="0" />
         </inertial>
@@ -81,5 +81,5 @@
         <inertial>
             <origin xyz="0 0.02 -0.01" rpy="0 0 0" />
-            <mass value="0.25" />
+            <mass value="0.02" />
             <inertia ixx="0.001" iyy="0.001" izz="0.001" ixy="0" iyz="0" ixz="0" />
         </inertial>
@@ -94,5 +94,5 @@
         <inertial>
             <origin xyz="0 0.003 0" rpy="0 0 0" />
-            <mass value="0.1" />
+            <mass value="0.01" />
             <inertia ixx="0.0001" iyy="0.0001" izz="0.0001" ixy="0" iyz="0" ixz="0" />
         </inertial>
@@ -107,5 +107,5 @@
         <inertial>
             <origin xyz="0 0.003 0" rpy="0 0 0" />
-            <mass value="0.1" />
+            <mass value="0.01" />
             <inertia ixx="0.0001" iyy="0.0001" izz="0.0001" ixy="0" iyz="0" ixz="0" />
         </inertial>
@@ -120,6 +120,6 @@
         <inertial>
             <origin xyz="-0.002 -0.002 0" rpy="0 0 0" />
-            <mass value="0.05" />
-            <inertia ixx="0.0001" iyy="0.0001" izz="0.0001" ixy="0" iyz="0" ixz="0" />
+            <mass value="0.01" />
+            <inertia ixx="0.000001" iyy="0.000001" izz="0.000001" ixy="0" iyz="0" ixz="0" />
         </inertial>
         <visual name="pusher_servo_part_visual">
@@ -133,5 +133,5 @@
         <inertial>
             <origin xyz="0 -0.02 0.01" rpy="0 0 0" />
-            <mass value="0.1" />
+            <mass value="0.01" />
             <inertia ixx="0.0001" iyy="0.0001" izz="0.0001" ixy="0" iyz="0" ixz="0" />
         </inertial>
@@ -146,5 +146,5 @@
         <inertial>
             <origin xyz="0.003 0.004 0" rpy="0 0 0" />
-            <mass value="0.05" />
+            <mass value="0.01" />
             <inertia ixx="0.0001" iyy="0.0001" izz="0.0001" ixy="0" iyz="0" ixz="0" />
         </inertial>
@@ -159,5 +159,5 @@
         <inertial>
             <origin xyz="0.01 0 -0.01" rpy="0 0 0" />
-            <mass value="0.1" />
+            <mass value="0.01" />
             <inertia ixx="0.0001" iyy="0.0001" izz="0.0001" ixy="0" iyz="0" ixz="0" />
         </inertial>
@@ -174,5 +174,5 @@
         <child link="motor_bracket" />
         <axis xyz="1.1287570791617654e-07 2.227474133869779e-15 1.0000000021779938" />
-        <limit lower="5.235988" upper="6.283185" effort="100.0" velocity="5.0" />
+        <limit lower="0.0" upper="1.5" effort="1.0" velocity="5.0" />
         <dynamics damping="10.0" friction="5.0"/>
     </joint>
@@ -193,5 +193,5 @@
         <axis xyz="-7.22468811426675e-18 -1.0 0.0004460000000000001" />
         <limit effort="10.0" velocity="100.0"/>
-        <dynamics damping="0.1" friction="0.01"/>
+        <dynamics damping="0.0" friction="0.0"/>
     </joint>
     <joint name="flywheel_left_joint" type="continuous">
@@ -201,5 +201,5 @@
         <axis xyz="-1.0870161747549608e-16 -0.9999999999999999 0.000446" />
         <limit effort="10.0" velocity="100.0"/>
-        <dynamics damping="0.1" friction="0.01"/>
+        <dynamics damping="0.0" friction="0.0"/>
     </joint>
     <joint name="motor_bracket_torret_on_motor_bracket" type="fixed">
@@ -223,6 +223,6 @@
         <child link="pusher_servo_part" />
         <axis xyz="-2.7546953265439552e-21 1.0 -0.000446" />
-        <limit effort="10.0" velocity="10.0"/>
-        <dynamics damping="0.1" friction="0.01"/>
+        <limit effort="0.1" velocity="20.0"/>
+        <dynamics damping="0.0" friction="0.0"/>
     </joint>
     <joint name="bottom_plate_servo_fix_bottom_plate" type="fixed">

Commit message: feat: Implement launcher tilt control by reconfiguring trigger joint limits and initial position, updating teleop commands, and adjusting launcher mount height.

File: src/gubot_one/description/nerf_launcher.xacro (robot description, xacro)
@@ -6,5 +6,5 @@
     <parent link="chassis"/>
     <child link="bottom_plate"/>
-    <origin xyz="0.155 0 0.15" rpy="0 0 ${pi/2}"/> </joint>
+    <origin xyz="0.155 0 0.165" rpy="0 0 ${pi/2}"/> </joint>
     <gazebo reference="nerf_mount_joint">
         <preserveFixedJoint>true</preserveFixedJoint>

File: src/gubot_one/description/ros2_control.xacro (robot description, xacro)
@@ -55,5 +55,5 @@
                 <command_interface name="position"/>
                 <state_interface name="position">
-                  <param name="initial_value">0.0</param>
+                  <param name="initial_value">6.28</param>
                 </state_interface>
             </joint>

File: src/nerf_standalone/description/urdf/launcher.urdf.xacro (robot description, xacro)
@@ -174,5 +174,5 @@
         <child link="motor_bracket" />
         <axis xyz="1.1287570791617654e-07 2.227474133869779e-15 1.0000000021779938" />
-        <limit lower="0.0" upper="1.5" effort="1.0" velocity="5.0" />
+        <limit lower="5.23" upper="6.28" effort="1.0" velocity="5.0" />
         <dynamics damping="10.0" friction="5.0"/>
     </joint>

Commit message: Refactor Nerf Launcher URDF and related files for improved simulation performance
- Renamed `launcher.urdf.xacro` to `nerf_launcher.urdf.xacro` for clarity.
- Updated references in `robot.urdf.xacro`, documentation, and scripts to reflect the new filename.
- Introduced separate URDF files for Gazebo Classic and Ignition simulation (`ros2_control_gazebo_classic.xacro` and `ros2_control_gazebo_fortress.xacro`).
- Added hardware interface definitions in `ros2_control_hardware_nerf.xacro`.
- Adjusted joint limits and dynamics for `trigger_joint` and `dart_pusher_joint` to enhance stability during simulation.
- Improved tilt control logic in `nerf_teleop.py` to accommodate different simulation environments.
- Updated launch files to utilize the new URDF structure.

File: src/gubot_one/description/nerf_launcher.xacro (robot description, xacro)
@@ -2,5 +2,5 @@
 <robot xmlns:xacro="http://www.ros.org/wiki/xacro">
     <xacro:arg name="integrated_mode" default="true"/>
-    <xacro:include filename="$(find nerf_launch_system)/description/urdf/launcher.urdf.xacro" />
+    <xacro:include filename="$(find nerf_launch_system)/description/urdf/nerf_launcher.urdf.xacro" />
     <joint name="nerf_mount_joint" type="fixed">
         <parent link="chassis"/>

File: src/gubot_one/description/robot.urdf.xacro (robot description, xacro)
@@ -3,9 +3,9 @@
     <xacro:arg name="use_ros2_control" default="true"/>
     <xacro:arg name="sim_mode" default="false"/>
+    <xacro:include filename="robot_core.xacro" />
     <xacro:arg name="integrated_mode" default="true"/>
     <xacro:arg name="use_nerf_hardware" default="true"/>
     <xacro:arg name="nerf_port" default="/dev/serial/by-id/usb-Arduino_LLC_Arduino_Leonardo-if00"/>
     <xacro:arg name="use_gazebo_classic" default="false"/>
-    <xacro:include filename="robot_core.xacro" />
     <xacro:if value="$(arg use_ros2_control)">
         <xacro:if value="$(arg use_gazebo_classic)">

File: src/nerf_launch_system/description/urdf/nerf_launcher.urdf.xacro (robot description, xacro)
@@ -168,5 +168,12 @@
         <child link="motor_bracket" />
         <axis xyz="1.1287570791617654e-07 2.227474133869779e-15 1.0000000021779938" />
-        <limit lower="-0.52" upper="0.52" effort="10.0" velocity="5.0" />
+        <xacro:if value="$(arg use_gazebo_classic)">
+            <!-- Classic Simulation parser requires the original bounds -->
+            <limit lower="-1.05" upper="0.0" effort="10.0" velocity="5.0" />
+        </xacro:if>
+        <xacro:unless value="$(arg use_gazebo_classic)">
+            <!-- Ignition Simulation bounds (symmetrical) -->
+            <limit lower="-0.52" upper="0.52" effort="10.0" velocity="5.0" />
+        </xacro:unless>
         <dynamics damping="0.2" friction="0.05"/>
     </joint>
@@ -236,5 +243,5 @@
     <xacro:arg name="port" default="/dev/ttyACM0"/>
     <xacro:if value="$(arg use_hardware)">
-        <xacro:include filename="ros2_control_hardware.xacro" />
+        <xacro:include filename="ros2_control_hardware_nerf.xacro" />
         <xacro:nerf_ros2_control_hardware port="$(arg port)"/>
     </xacro:if>
@@ -256,8 +263,8 @@
             <xacro:arg name="use_gazebo_classic" default="false"/>
             <xacro:if value="$(arg use_gazebo_classic)">
-                <xacro:include filename="gz_classic_ros2_control.xacro" />
+                <xacro:include filename="ros2_control_gazebo_classic.xacro" />
             </xacro:if>
             <xacro:unless value="$(arg use_gazebo_classic)">
-                <xacro:include filename="ros2_control.xacro" />
+                <xacro:include filename="ros2_control_gazebo_fortress.xacro" />
             </xacro:unless>
             <xacro:nerf_ros2_control />
