Commit message: feat: Aktualisierung der Roboterdokumentation und Konfigurationsdateien für verbesserte Simulation

File: src/gubot_one/description/ros2_control_gazebo_classic.xacro (robot description, xacro)
@@ -32,14 +32,4 @@
             <state_interface name="position"/>
         </joint>
-        <joint name="flywheel_left_joint">
-            <command_interface name="velocity"/>
-            <state_interface name="velocity"/>
-            <state_interface name="position"/>
-        </joint>
-        <joint name="flywheel_right_joint">
-            <command_interface name="velocity"/>
-            <state_interface name="velocity"/>
-            <state_interface name="position"/>
-        </joint>
         <joint name="system_arming_joint">
             <command_interface name="position"/>

File: src/gubot_one/description/ros2_control_gazebo_ign_fortress.xacro (robot description, xacro)
@@ -3,5 +3,5 @@
     <ros2_control name="IgnitionSystem" type="system">
         <hardware>
-            <plugin>ign_ros2_control/IgnitionSystem</plugin>
+            <plugin>gz_ros2_control/GazeboSimSystem</plugin>
             <param name="position_proportional_gain">20.0</param>
         </hardware>
@@ -36,14 +36,4 @@
             <state_interface name="position"/>
         </joint>
-        <joint name="flywheel_left_joint">
-            <command_interface name="velocity"/>
-            <state_interface name="velocity"/>
-            <state_interface name="position"/>
-        </joint>
-        <joint name="flywheel_right_joint">
-            <command_interface name="velocity"/>
-            <state_interface name="velocity"/>
-            <state_interface name="position"/>
-        </joint>
         <joint name="system_arming_joint">
             <command_interface name="position"/>
@@ -64,5 +54,5 @@
     </ros2_control>
     <gazebo>
-        <plugin filename="ign_ros2_control-system" name="ign_ros2_control::IgnitionROS2ControlPlugin">
+        <plugin filename="gz_ros2_control-system" name="gz_ros2_control::GazeboSimROS2ControlPlugin">
             <parameters>$(find gubot_one)/config/my_controllers.yaml</parameters>
             <parameters>$(find gubot_one)/config/gaz_ros2_ctl_use_sim.yaml</parameters>

File: src/gubot_one/description/ros2_control_hardware.xacro (robot description, xacro)
@@ -54,12 +54,4 @@
                 <state_interface name="velocity"/>
             </joint>
-            <joint name="flywheel_left_joint">
-                <command_interface name="velocity"/>
-                <state_interface name="velocity"/>
-            </joint>
-            <joint name="flywheel_right_joint">
-                <command_interface name="velocity"/>
-                <state_interface name="velocity"/>
-            </joint>
             <joint name="system_arming_joint">
                 <command_interface name="position"/>
