Commit message: feat: add mecanum drive controller configuration and update robot launch system parameters

File: src/gubot_one/description/ros2_control_gazebo_ign_fortress.xacro (robot description, xacro)
@@ -30,6 +30,10 @@
                     <param name="max">10</param>
                 </command_interface>
-                <state_interface name="velocity"/>
-                <state_interface name="position"/>
+                <state_interface name="velocity">
+                    <param name="initial_value">0.0</param>
+                </state_interface>
+                <state_interface name="position">
+                    <param name="initial_value">0.0</param>
+                </state_interface>
             </joint>
             <joint name="front_right_wheel_joint">
@@ -38,6 +42,10 @@
                     <param name="max">10</param>
                 </command_interface>
-                <state_interface name="velocity"/>
-                <state_interface name="position"/>
+                <state_interface name="velocity">
+                    <param name="initial_value">0.0</param>
+                </state_interface>
+                <state_interface name="position">
+                    <param name="initial_value">0.0</param>
+                </state_interface>
             </joint>
             <joint name="rear_left_wheel_joint">
@@ -46,6 +54,10 @@
                     <param name="max">10</param>
                 </command_interface>
-                <state_interface name="velocity"/>
-                <state_interface name="position"/>
+                <state_interface name="velocity">
+                    <param name="initial_value">0.0</param>
+                </state_interface>
+                <state_interface name="position">
+                    <param name="initial_value">0.0</param>
+                </state_interface>
             </joint>
             <joint name="rear_right_wheel_joint">
@@ -54,26 +66,34 @@
                     <param name="max">10</param>
                 </command_interface>
+                <state_interface name="velocity">
+                    <param name="initial_value">0.0</param>
+                </state_interface>
+                <state_interface name="position">
+                    <param name="initial_value">0.0</param>
+                </state_interface>
+            </joint>
+        </xacro:if>
+        <!-- Nerf-Joints: NUR wenn use_nerf_hardware=true, sonst existieren diese Joints nicht in der URDF -->
+        <!-- ALT: xacro:if value="$(arg use_nerf_hardware)" — "false" wurde als wahr evaluiert -->
+        <xacro:if value="${'$(arg use_nerf_hardware)' == 'true'}">
+            <joint name="trigger_joint">
+                <command_interface name="position">
+                    <param name="p">50.0</param>
+                    <param name="d">1.0</param>
+                </command_interface>
+                <state_interface name="position">
+                    <param name="initial_value">0.0</param>
+                </state_interface>
+            </joint>
+            <joint name="dart_pusher_joint">
+                <command_interface name="velocity"/>
                 <state_interface name="velocity"/>
                 <state_interface name="position"/>
             </joint>
+            <joint name="system_arming_joint">
+                <command_interface name="position"/>
+                <state_interface name="position"/>
+            </joint>
         </xacro:if>
-        <joint name="trigger_joint">
-            <command_interface name="position">
-                <param name="p">50.0</param>
-                <param name="d">1.0</param>
-            </command_interface>
-            <state_interface name="position">
-                <param name="initial_value">0.0</param>
-            </state_interface>
-        </joint>
-        <joint name="dart_pusher_joint">
-            <command_interface name="velocity"/>
-            <state_interface name="velocity"/>
-            <state_interface name="position"/>
-        </joint>
-        <joint name="system_arming_joint">
-            <command_interface name="position"/>
-            <state_interface name="position"/>
-        </joint>
         <sensor name="imu_sensor">
             <state_interface name="linear_acceleration.x"/>
