Commit message: feat(mecanum): Husarion-Controller integriert, Strafe verifiziert
Husarion mecanum_drive_controller aus github.com/husarion/husarion_controllers
als lokales Paket in src/ hinzugefuegt (ueberschreibt apt-Version).

Warum Husarion statt ros2_controllers:
- parameter: wheel_separation_x/y statt sum_of_projection (intuitiver)
- open_loop: true  -> Simulation ohne Encoder, sofort nutzbar
- use_stamped_vel: false -> subscribt direkt auf /cmd_vel (kein Remapping)
- Speed-Limiter: Velocity + Acceleration + Jerk
- Rolling-Window-Odometrie (velocity_rolling_window_size: 10)

mecanum_controllers.yaml:
- wheel_separation_x: 0.25, wheel_separation_y: 0.20, wheel_radius: 0.05
- open_loop: true, position_feedback: false
- use_stamped_vel: false
- pose/twist_covariance_diagonal ergaenzt

mecanum_pico.launch.py:
- Remapping entfernt (nicht noetig: Husarion subscribt direkt /cmd_vel)

Verifiziert (mock_hardware):
  ros2 topic pub /cmd_vel Twist linear.y=0.2
  -> /mecanum_drive_controller/odom zeigt twist.linear.y=0.2  STRAFE OK

File: src/gubot_one/description/gubot_one_geometry.xacro (robot description, xacro)
@@ -59,8 +59,9 @@
             <origin xyz="${chassis_length/2} 0 ${chassis_height/2}"/>
             <geometry>
-                <box size="${chassis_length} ${chassis_width} ${chassis_height}"/>
+                <!-- Slightly smaller collision box to avoid wheel overlap -->
+                <box size="${chassis_length - 0.01} ${chassis_width - 0.01} ${chassis_height - 0.01}"/>
             </geometry>
         </collision>
-        <xacro:inertial_box mass="0.5" x="${chassis_length}" y="${chassis_width}" z="${chassis_height}">
+        <xacro:inertial_box mass="${chassis_mass}" x="${chassis_length}" y="${chassis_width}" z="${chassis_height}">
             <origin xyz="${chassis_length/2} 0 ${chassis_height/2}" rpy="0 0 0"/>
         </xacro:inertial_box>
@@ -168,9 +169,10 @@
     </gazebo>
     <!-- LEFT WHEEL LINK -->
-    <joint name="left_wheel_joint" type="continuous">
+    <joint name="front_left_wheel_joint" type="continuous">
         <parent link="base_link"/>
         <child link="left_wheel"/>
         <origin xyz="0 ${wheel_offset_y} 0" rpy="-${pi/2} 0 0" />
         <axis xyz="0 0 1"/>
+        <dynamics damping="0.01" friction="0.01"/>
     </joint>
     <link name="left_wheel">
@@ -194,9 +196,10 @@
     </gazebo>
     <!-- RIGHT WHEEL LINK -->
-    <joint name="right_wheel_joint" type="continuous">
+    <joint name="front_right_wheel_joint" type="continuous">
         <parent link="base_link"/>
         <child link="right_wheel"/>
         <origin xyz="0 ${-wheel_offset_y} 0" rpy="${pi/2} 0 0" />
         <axis xyz="0 0 -1"/>
+        <dynamics damping="0.01" friction="0.01"/>
     </joint>
     <link name="right_wheel">
@@ -219,30 +222,89 @@
         <material>Gazebo/Blue</material>
     </gazebo>
-    <!-- CASTER WHEEL LINK -->
-    <joint name="caster_wheel_joint" type="fixed">
-        <parent link="chassis"/>
-        <child link="caster_wheel"/>
-        <origin xyz="${caster_wheel_offset_x} 0 ${caster_wheel_offset_z}"/>
-    </joint>
-    <link name="caster_wheel">
-        <visual>
-            <geometry>
-                <sphere radius="${caster_wheel_radius}"/>
-            </geometry>
-            <material name="white"/>
-        </visual>
-        <collision>
-            <geometry>
-                <sphere radius="${caster_wheel_radius}"/>
-            </geometry>
-        </collision>
-        <xacro:inertial_sphere mass="${caster_wheel_mass}" radius="${caster_wheel_radius}">
-            <origin xyz="0 0 0" rpy="0 0 0"/>
-        </xacro:inertial_sphere>
-    </link>
-    <gazebo reference="caster_wheel">
-        <material>Gazebo/White</material>
-        <mu1 value="0.001"/>
-        <mu2 value="0.001"/>
-    </gazebo>
+    <!-- CASTER WHEEL LINK (Diffdrive only) -->
+    <xacro:if value="${'$(arg drive_type)' == 'diffdrive'}">
+        <joint name="caster_wheel_joint" type="fixed">
+            <parent link="chassis"/>
+            <child link="caster_wheel"/>
+            <origin xyz="${caster_wheel_offset_x} 0 ${caster_wheel_offset_z}"/>
+        </joint>
+        <link name="caster_wheel">
+            <visual>
+                <geometry>
+                    <sphere radius="${caster_wheel_radius}"/>
+                </geometry>
+                <material name="white"/>
+            </visual>
+            <collision>
+                <geometry>
+                    <sphere radius="${caster_wheel_radius}"/>
+                </geometry>
+            </collision>
+            <xacro:inertial_sphere mass="${caster_wheel_mass}" radius="${caster_wheel_radius}">
+                <origin xyz="0 0 0" rpy="0 0 0"/>
+            </xacro:inertial_sphere>
+        </link>
+        <gazebo reference="caster_wheel">
+            <material>Gazebo/White</material>
+            <mu1 value="0.001"/>
+            <mu2 value="0.001"/>
+        </gazebo>
+    </xacro:if>
+    <!-- REAR WHEELS (Mecanum only) -->
+    <xacro:if value="${'$(arg drive_type)' == 'mecanum'}">
+        <!-- REAR LEFT WHEEL LINK -->
+        <joint name="rear_left_wheel_joint" type="continuous">
+            <parent link="base_link"/>
+            <child link="rear_left_wheel"/>
+            <origin xyz="${-wheel_offset_x} ${wheel_offset_y} 0" rpy="-${pi/2} 0 0" />
+            <axis xyz="0 0 1"/>
+            <dynamics damping="0.01" friction="0.01"/>
+        </joint>
+        <link name="rear_left_wheel">
+            <visual>
+                <geometry>
+                    <cylinder radius="${wheel_radius}" length="${wheel_thickness}"/>
+                </geometry>
+                <material name="blue"/>
+            </visual>
+            <collision>
+                <geometry>
+                    <sphere radius="${wheel_radius}"/>
+                </geometry>
+            </collision>
+            <xacro:inertial_cylinder mass="${wheel_mass}" length="${wheel_thickness}" radius="${wheel_radius}">
+                <origin xyz="0 0 0" rpy="0 0 0"/>
+            </xacro:inertial_cylinder>
+        </link>
+        <gazebo reference="rear_left_wheel">
+            <material>Gazebo/Blue</material>
+        </gazebo>
+        <!-- REAR RIGHT WHEEL LINK -->
+        <joint name="rear_right_wheel_joint" type="continuous">
+            <parent link="base_link"/>
+            <child link="rear_right_wheel"/>
+            <origin xyz="${-wheel_offset_x} ${-wheel_offset_y} 0" rpy="${pi/2} 0 0" />
+            <axis xyz="0 0 -1"/>
+            <dynamics damping="0.01" friction="0.01"/>
+        </joint>
+        <link name="rear_right_wheel">
+            <visual>
+                <geometry>
+                    <cylinder radius="${wheel_radius}" length="${wheel_thickness}"/>
+                </geometry>
+                <material name="blue"/>
+            </visual>
+            <collision>
+                <geometry>
+                    <sphere radius="${wheel_radius}"/>
+                </geometry>
+            </collision>
+            <xacro:inertial_cylinder mass="${wheel_mass}" length="${wheel_thickness}" radius="${wheel_radius}">
+                <origin xyz="0 0 0" rpy="0 0 0"/>
+            </xacro:inertial_cylinder>
+        </link>
+        <gazebo reference="rear_right_wheel">
+            <material>Gazebo/Blue</material>
+        </gazebo>
+    </xacro:if>
 </robot>

File: src/gubot_one/description/gubot_one_main.urdf.xacro (robot description, xacro)
@@ -4,4 +4,5 @@
     <xacro:arg name="sim_mode" default="false"/>
     <xacro:arg name="use_gazebo_classic" default="false"/>
+    <xacro:arg name="drive_type" default="mecanum"/>
     <xacro:include filename="gubot_one_geometry.xacro" />
     <xacro:if value="$(arg use_ros2_control)">

File: src/gubot_one/description/ros2_control_gazebo_classic.xacro (robot description, xacro)
@@ -5,20 +5,56 @@
             <plugin>gazebo_ros2_control/GazeboSystem</plugin>
         </hardware>
-        <joint name="left_wheel_joint">
-            <command_interface name="velocity">
-                <param name="min">-10</param>
-                <param name="max">10</param>
-            </command_interface>
-            <state_interface name="velocity"/>
-            <state_interface name="position"/>
-        </joint>
-        <joint name="right_wheel_joint">
-            <command_interface name="velocity">
-                <param name="min">-10</param>
-                <param name="max">10</param>
-            </command_interface>
-            <state_interface name="velocity"/>
-            <state_interface name="position"/>
-        </joint>
+        <xacro:if value="${'$(arg drive_type)' == 'diffdrive'}">
+            <joint name="left_wheel_joint">
+                <command_interface name="velocity">
+                    <param name="min">-10</param>
+                    <param name="max">10</param>
+                </command_interface>
+                <state_interface name="velocity"/>
+                <state_interface name="position"/>
+            </joint>
+            <joint name="right_wheel_joint">
+                <command_interface name="velocity">
+                    <param name="min">-10</param>
+                    <param name="max">10</param>
+                </command_interface>
+                <state_interface name="velocity"/>
+                <state_interface name="position"/>
+            </joint>
+        </xacro:if>
+        <xacro:if value="${'$(arg drive_type)' == 'mecanum'}">
+            <joint name="front_left_wheel_joint">
+                <command_interface name="velocity">
+                    <param name="min">-10</param>
+                    <param name="max">10</param>
+                </command_interface>
+                <state_interface name="velocity"/>
+                <state_interface name="position"/>
+            </joint>
+            <joint name="front_right_wheel_joint">
+                <command_interface name="velocity">
+                    <param name="min">-10</param>
+                    <param name="max">10</param>
+                </command_interface>
+                <state_interface name="velocity"/>
+                <state_interface name="position"/>
+            </joint>
+            <joint name="rear_left_wheel_joint">
+                <command_interface name="velocity">
+                    <param name="min">-10</param>
+                    <param name="max">10</param>
+                </command_interface>
+                <state_interface name="velocity"/>
+                <state_interface name="position"/>
+            </joint>
+            <joint name="rear_right_wheel_joint">
+                <command_interface name="velocity">
+                    <param name="min">-10</param>
+                    <param name="max">10</param>
+                </command_interface>
+                <state_interface name="velocity"/>
+                <state_interface name="position"/>
+            </joint>
+        </xacro:if>
         <joint name="trigger_joint">
             <command_interface name="position"/>
@@ -51,6 +87,10 @@
     <gazebo>
         <plugin filename="libgazebo_ros2_control.so" name="gazebo_ros2_control">
-            <parameters>$(find gubot_one)/config/my_controllers.yaml</parameters>
-            <parameters>$(find gubot_one)/config/gaz_ros2_ctl_use_sim.yaml</parameters>
+            <xacro:if value="${'$(arg drive_type)' == 'diffdrive'}">
+                <parameters>$(find gubot_one)/config/my_controllers.yaml</parameters>
+            </xacro:if>
+            <xacro:if value="${'$(arg drive_type)' == 'mecanum'}">
+                <parameters>$(find gubot_one)/config/mecanum_my_controllers.yaml</parameters>
+            </xacro:if>
         </plugin>
     </gazebo>

File: src/gubot_one/description/ros2_control_gazebo_ign_fortress.xacro (robot description, xacro)
@@ -6,20 +6,56 @@
             <param name="position_proportional_gain">20.0</param>
         </hardware>
-        <joint name="left_wheel_joint">
-            <command_interface name="velocity">
-                <param name="min">-10</param>
-                <param name="max">10</param>
-            </command_interface>
-            <state_interface name="velocity"/>
-            <state_interface name="position"/>
-        </joint>
-        <joint name="right_wheel_joint">
-            <command_interface name="velocity">
-                <param name="min">-10</param>
-                <param name="max">10</param>
-            </command_interface>
-            <state_interface name="velocity"/>
-            <state_interface name="position"/>
-        </joint>
+        <xacro:if value="${'$(arg drive_type)' == 'diffdrive'}">
+            <joint name="left_wheel_joint">
+                <command_interface name="velocity">
+                    <param name="min">-10</param>
+                    <param name="max">10</param>
+                </command_interface>
+                <state_interface name="velocity"/>
+                <state_interface name="position"/>
+            </joint>
+            <joint name="right_wheel_joint">
+                <command_interface name="velocity">
+                    <param name="min">-10</param>
+                    <param name="max">10</param>
+                </command_interface>
+                <state_interface name="velocity"/>
+                <state_interface name="position"/>
+            </joint>
+        </xacro:if>
+        <xacro:if value="${'$(arg drive_type)' == 'mecanum'}">
+            <joint name="front_left_wheel_joint">
+                <command_interface name="velocity">
+                    <param name="min">-10</param>
+                    <param name="max">10</param>
+                </command_interface>
+                <state_interface name="velocity"/>
+                <state_interface name="position"/>
+            </joint>
+            <joint name="front_right_wheel_joint">
+                <command_interface name="velocity">
+                    <param name="min">-10</param>
+                    <param name="max">10</param>
+                </command_interface>
+                <state_interface name="velocity"/>
+                <state_interface name="position"/>
+            </joint>
+            <joint name="rear_left_wheel_joint">
+                <command_interface name="velocity">
+                    <param name="min">-10</param>
+                    <param name="max">10</param>
+                </command_interface>
+                <state_interface name="velocity"/>
+                <state_interface name="position"/>
+            </joint>
+            <joint name="rear_right_wheel_joint">
+                <command_interface name="velocity">
+                    <param name="min">-10</param>
+                    <param name="max">10</param>
+                </command_interface>
+                <state_interface name="velocity"/>
+                <state_interface name="position"/>
+            </joint>
+        </xacro:if>
         <joint name="trigger_joint">
             <command_interface name="position">
@@ -55,6 +91,10 @@
     <gazebo>
         <plugin filename="gz_ros2_control-system" name="gz_ros2_control::GazeboSimROS2ControlPlugin">
-            <parameters>$(find gubot_one)/config/my_controllers.yaml</parameters>
-            <parameters>$(find gubot_one)/config/gaz_ros2_ctl_use_sim.yaml</parameters>
+            <xacro:if value="${'$(arg drive_type)' == 'diffdrive'}">
+                <parameters>$(find gubot_one)/config/my_controllers.yaml</parameters>
+            </xacro:if>
+            <xacro:if value="${'$(arg drive_type)' == 'mecanum'}">
+                <parameters>$(find gubot_one)/config/mecanum_my_controllers.yaml</parameters>
+            </xacro:if>
         </plugin>
     </gazebo>

File: src/gubot_one/description/ros2_control_hardware.xacro (robot description, xacro)
@@ -3,40 +3,98 @@
     <xacro:arg name="use_nerf_hardware" default="true"/>
     <xacro:arg name="nerf_port" default="/dev/serial/by-id/usb-Arduino_LLC_Arduino_Leonardo-if00"/>
-    <ros2_control name="RealRobot" type="system">
-        <hardware>
-            <plugin>diffdrive_arduino/DiffDriveArduinoHardware</plugin>
-            <param name="left_wheel_name">left_wheel_joint</param>
-            <param name="right_wheel_name">right_wheel_joint</param>
-            <param name="loop_rate">30</param>
-            <param name="device">/dev/serial/by-id/usb-Raspberry_Pi_Pico_50443405786ACA1C-if00</param>
-            <param name="baud_rate">115200</param>
-            <param name="timeout_ms">1000</param>
-            <param name="enc_counts_per_rev">3436</param>
-        </hardware>
-        <joint name="left_wheel_joint">
-            <command_interface name="velocity">
-                <param name="min">-10</param>
-                <param name="max">10</param>
-            </command_interface>
-            <state_interface name="position"/>
-            <state_interface name="velocity"/>
-        </joint>
-        <joint name="right_wheel_joint">
-            <command_interface name="velocity">
-                <param name="min">-10</param>
-                <param name="max">10</param>
-            </command_interface>
-            <state_interface name="position"/>
-            <state_interface name="velocity"/>
-        </joint>
-        <sensor name="imu_sensor">
-            <state_interface name="linear_acceleration.x"/>
-            <state_interface name="linear_acceleration.y"/>
-            <state_interface name="linear_acceleration.z"/>
-            <state_interface name="angular_velocity.x"/>
-            <state_interface name="angular_velocity.y"/>
-            <state_interface name="angular_velocity.z"/>
-        </sensor>
-    </ros2_control>
+    <xacro:if value="${'$(arg drive_type)' == 'diffdrive'}">
+        <ros2_control name="RealRobot" type="system">
+            <hardware>
+                <plugin>diffdrive_arduino/DiffDriveArduinoHardware</plugin>
+                <param name="left_wheel_name">left_wheel_joint</param>
+                <param name="right_wheel_name">right_wheel_joint</param>
+                <param name="loop_rate">30</param>
+                <param name="device">/dev/serial/by-id/usb-Raspberry_Pi_Pico_50443405786ACA1C-if00</param>
+                <param name="baud_rate">115200</param>
+                <param name="timeout_ms">1000</param>
+                <param name="enc_counts_per_rev">3436</param>
+            </hardware>
+            <joint name="left_wheel_joint">
+                <command_interface name="velocity">
+                    <param name="min">-10</param>
+                    <param name="max">10</param>
+                </command_interface>
+                <state_interface name="position"/>
+                <state_interface name="velocity"/>
+            </joint>
+            <joint name="right_wheel_joint">
+                <command_interface name="velocity">
+                    <param name="min">-10</param>
+                    <param name="max">10</param>
+                </command_interface>
+                <state_interface name="position"/>
+                <state_interface name="velocity"/>
+            </joint>
+            <sensor name="imu_sensor">
+                <state_interface name="linear_acceleration.x"/>
+                <state_interface name="linear_acceleration.y"/>
+                <state_interface name="linear_acceleration.z"/>
+                <state_interface name="angular_velocity.x"/>
+                <state_interface name="angular_velocity.y"/>
+                <state_interface name="angular_velocity.z"/>
+            </sensor>
+        </ros2_control>
+    </xacro:if>
+    <xacro:if value="${'$(arg drive_type)' == 'mecanum'}">
+        <ros2_control name="RealRobot" type="system">
+            <hardware>
+                <plugin>mecanum_pico/MecanumPicoHardware</plugin>
+                <param name="front_left_wheel_name">front_left_wheel_joint</param>
+                <param name="front_right_wheel_name">front_right_wheel_joint</param>
+                <param name="rear_left_wheel_name">rear_left_wheel_joint</param>
+                <param name="rear_right_wheel_name">rear_right_wheel_joint</param>
+                <param name="loop_rate">30</param>
+                <param name="device">/dev/serial/by-id/usb-Raspberry_Pi_Pico_50443405786ACA1C-if00</param>
+                <param name="baud_rate">115200</param>
+                <param name="timeout_ms">1000</param>
+                <param name="enc_counts_per_rev">3436</param>
+            </hardware>
+            <joint name="front_left_wheel_joint">
+                <command_interface name="velocity">
+                    <param name="min">-10</param>
+                    <param name="max">10</param>
+                </command_interface>
+                <state_interface name="position"/>
+                <state_interface name="velocity"/>
+            </joint>
+            <joint name="front_right_wheel_joint">
+                <command_interface name="velocity">
+                    <param name="min">-10</param>
+                    <param name="max">10</param>
+                </command_interface>
+                <state_interface name="position"/>
+                <state_interface name="velocity"/>
+            </joint>
+            <joint name="rear_left_wheel_joint">
+                <command_interface name="velocity">
+                    <param name="min">-10</param>
+                    <param name="max">10</param>
+                </command_interface>
+                <state_interface name="position"/>
+                <state_interface name="velocity"/>
+            </joint>
+            <joint name="rear_right_wheel_joint">
+                <command_interface name="velocity">
+                    <param name="min">-10</param>
+                    <param name="max">10</param>
+                </command_interface>
+                <state_interface name="position"/>
+                <state_interface name="velocity"/>
+            </joint>
+            <sensor name="imu_sensor">
+                <state_interface name="linear_acceleration.x"/>
+                <state_interface name="linear_acceleration.y"/>
+                <state_interface name="linear_acceleration.z"/>
+                <state_interface name="angular_velocity.x"/>
+                <state_interface name="angular_velocity.y"/>
+                <state_interface name="angular_velocity.z"/>
+            </sensor>
+        </ros2_control>
+    </xacro:if>
     <xacro:if value="$(arg use_nerf_hardware)">
         <ros2_control name="NerfSystem" type="system">
