Commit message: feat(gubot_one): Mecanum drive integration — plans 01, 02, 05 done
- launch_robot.launch.py: mecanum_cont spawner, drive_type arg, correct remap
- gubot_one_geometry.xacro: symmetric wheel_offset_x=0.113 for mecanum
- mecanum_my_controllers.yaml: Humble schema, duplicates removed
- tests: test_controller_yaml, test_launch_robot, test_urdf_geometry (all green)
- test_tilt_controller_spawner: fixed file refs, pep257 compliance
- Moved docs/scripts to proper directories

File: src/gubot_one/description/gubot_one_geometry.xacro (robot description, xacro)
@@ -9,5 +9,6 @@
     <xacro:property name="wheel_thickness" value="0.026"/>
     <xacro:property name="wheel_mass" value="0.05"/>
-    <xacro:property name="wheel_offset_x" value="0.226"/>
+    <!-- ALT (Asymmetrisch): <xacro:property name="wheel_offset_x" value="0.226"/> -->
+    <xacro:property name="wheel_offset_x" value="0.113"/>
     <xacro:property name="wheel_offset_y" value="0.1485"/>
     <xacro:property name="wheel_offset_z" value="0.01"/>
@@ -172,5 +173,6 @@
         <parent link="base_link"/>
         <child link="left_wheel"/>
-        <origin xyz="0 ${wheel_offset_y} 0" rpy="-${pi/2} 0 0" />
+        <!-- ALT (X=0): <origin xyz="0 ${wheel_offset_y} 0" rpy="-${pi/2} 0 0" /> -->
+        <origin xyz="${wheel_offset_x} ${wheel_offset_y} 0" rpy="-${pi/2} 0 0" />
         <axis xyz="0 0 1"/>
         <dynamics damping="0.01" friction="0.01"/>
@@ -199,5 +201,6 @@
         <parent link="base_link"/>
         <child link="right_wheel"/>
-        <origin xyz="0 ${-wheel_offset_y} 0" rpy="${pi/2} 0 0" />
+        <!-- ALT (X=0): <origin xyz="0 ${-wheel_offset_y} 0" rpy="${pi/2} 0 0" /> -->
+        <origin xyz="${wheel_offset_x} ${-wheel_offset_y} 0" rpy="${pi/2} 0 0" />
         <axis xyz="0 0 -1"/>
         <dynamics damping="0.01" friction="0.01"/>
