Commit message: refactor: remove diffdrive_arduino workspace and update gubot_one configuration files

File: src/gubot_one/description/gubot_one_geometry.xacro (robot description, xacro)
@@ -196,4 +196,7 @@
     <gazebo reference="left_wheel">
         <material>Gazebo/Blue</material>
+        <mu1>1.0</mu1>
+        <mu2>0.0</mu2>
+        <fdir1>1 -1 0</fdir1>
     </gazebo>
     <!-- RIGHT WHEEL LINK -->
@@ -224,36 +227,9 @@
     <gazebo reference="right_wheel">
         <material>Gazebo/Blue</material>
-    </gazebo>
-    <!-- CASTER WHEEL LINK (Diffdrive only) -->
-    <xacro:if value="${'$(arg drive_type)' == 'diffdrive'}">
-        <joint name="caster_wheel_joint" type="fixed">
-            <parent link="chassis"/>
-            <child link="caster_wheel"/>
-            <origin xyz="${caster_wheel_offset_x} 0 ${caster_wheel_offset_z}"/>
-        </joint>
-        <link name="caster_wheel">
-            <visual>
-                <geometry>
-                    <sphere radius="${caster_wheel_radius}"/>
-                </geometry>
-                <material name="white"/>
-            </visual>
-            <collision>
-                <geometry>
-                    <sphere radius="${caster_wheel_radius}"/>
-                </geometry>
-            </collision>
-            <xacro:inertial_sphere mass="${caster_wheel_mass}" radius="${caster_wheel_radius}">
-                <origin xyz="0 0 0" rpy="0 0 0"/>
-            </xacro:inertial_sphere>
-        </link>
-        <gazebo reference="caster_wheel">
-            <material>Gazebo/White</material>
-            <mu1 value="0.001"/>
-            <mu2 value="0.001"/>
-        </gazebo>
-    </xacro:if>
-    <!-- REAR WHEELS (Mecanum only) -->
-    <xacro:if value="${'$(arg drive_type)' == 'mecanum'}">
+        <mu1>1.0</mu1>
+        <mu2>0.0</mu2>
+        <fdir1>1 1 0</fdir1>
+    </gazebo>
+    <!-- REAR WHEELS -->
         <!-- REAR LEFT WHEEL LINK -->
         <joint name="rear_left_wheel_joint" type="continuous">
@@ -282,4 +258,7 @@
         <gazebo reference="rear_left_wheel">
             <material>Gazebo/Blue</material>
+            <mu1>1.0</mu1>
+            <mu2>0.0</mu2>
+            <fdir1>1 1 0</fdir1>
         </gazebo>
         <!-- REAR RIGHT WHEEL LINK -->
@@ -309,5 +288,7 @@
         <gazebo reference="rear_right_wheel">
             <material>Gazebo/Blue</material>
+            <mu1>1.0</mu1>
+            <mu2>0.0</mu2>
+            <fdir1>1 -1 0</fdir1>
         </gazebo>
-    </xacro:if>
 </robot>

File: src/gubot_one/description/gubot_one_main.urdf.xacro (robot description, xacro)
@@ -4,5 +4,4 @@
     <xacro:arg name="sim_mode" default="false"/>
     <xacro:arg name="use_gazebo_classic" default="false"/>
-    <xacro:arg name="drive_type" default="mecanum"/>
     <xacro:include filename="gubot_one_geometry.xacro" />
     <xacro:if value="$(arg use_ros2_control)">
@@ -19,7 +18,4 @@
         </xacro:unless>
     </xacro:if>
-    <xacro:unless value="$(arg use_ros2_control)">
-        <xacro:include filename="control_gazebo_diff_drive.xacro" />
-    </xacro:unless>
     <xacro:arg name="use_nerf_hardware" default="true"/>
     <!-- <xacro:include filename="sensor_lidar.xacro" /> -->

File: src/gubot_one/description/ros2_control_gazebo_classic.xacro (robot description, xacro)
@@ -5,56 +5,36 @@
             <plugin>gazebo_ros2_control/GazeboSystem</plugin>
         </hardware>
-        <xacro:if value="${'$(arg drive_type)' == 'diffdrive'}">
-            <joint name="left_wheel_joint">
-                <command_interface name="velocity">
-                    <param name="min">-10</param>
-                    <param name="max">10</param>
-                </command_interface>
-                <state_interface name="velocity"/>
-                <state_interface name="position"/>
-            </joint>
-            <joint name="right_wheel_joint">
-                <command_interface name="velocity">
-                    <param name="min">-10</param>
-                    <param name="max">10</param>
-                </command_interface>
-                <state_interface name="velocity"/>
-                <state_interface name="position"/>
-            </joint>
-        </xacro:if>
-        <xacro:if value="${'$(arg drive_type)' == 'mecanum'}">
-            <joint name="front_left_wheel_joint">
-                <command_interface name="velocity">
-                    <param name="min">-10</param>
-                    <param name="max">10</param>
-                </command_interface>
-                <state_interface name="velocity"/>
-                <state_interface name="position"/>
-            </joint>
-            <joint name="front_right_wheel_joint">
-                <command_interface name="velocity">
-                    <param name="min">-10</param>
-                    <param name="max">10</param>
-                </command_interface>
-                <state_interface name="velocity"/>
-                <state_interface name="position"/>
-            </joint>
-            <joint name="rear_left_wheel_joint">
-                <command_interface name="velocity">
-                    <param name="min">-10</param>
-                    <param name="max">10</param>
-                </command_interface>
-                <state_interface name="velocity"/>
-                <state_interface name="position"/>
-            </joint>
-            <joint name="rear_right_wheel_joint">
-                <command_interface name="velocity">
-                    <param name="min">-10</param>
-                    <param name="max">10</param>
-                </command_interface>
-                <state_interface name="velocity"/>
-                <state_interface name="position"/>
-            </joint>
-        </xacro:if>
+        <joint name="front_left_wheel_joint">
+            <command_interface name="velocity">
+                <param name="min">-10</param>
+                <param name="max">10</param>
+            </command_interface>
+            <state_interface name="velocity"/>
+            <state_interface name="position"/>
+        </joint>
+        <joint name="front_right_wheel_joint">
+            <command_interface name="velocity">
+                <param name="min">-10</param>
+                <param name="max">10</param>
+            </command_interface>
+            <state_interface name="velocity"/>
+            <state_interface name="position"/>
+        </joint>
+        <joint name="rear_left_wheel_joint">
+            <command_interface name="velocity">
+                <param name="min">-10</param>
+                <param name="max">10</param>
+            </command_interface>
+            <state_interface name="velocity"/>
+            <state_interface name="position"/>
+        </joint>
+        <joint name="rear_right_wheel_joint">
+            <command_interface name="velocity">
+                <param name="min">-10</param>
+                <param name="max">10</param>
+            </command_interface>
+            <state_interface name="velocity"/>
+            <state_interface name="position"/>
+        </joint>
         <joint name="trigger_joint">
             <command_interface name="position"/>
@@ -87,10 +67,5 @@
     <gazebo>
         <plugin filename="libgazebo_ros2_control.so" name="gazebo_ros2_control">
-            <xacro:if value="${'$(arg drive_type)' == 'diffdrive'}">
-                <parameters>$(find gubot_one)/config/my_controllers.yaml</parameters>
-            </xacro:if>
-            <xacro:if value="${'$(arg drive_type)' == 'mecanum'}">
-                <parameters>$(find gubot_one)/config/mecanum_my_controllers.yaml</parameters>
-            </xacro:if>
+            <parameters>$(find gubot_one)/config/my_controllers.yaml</parameters>
         </plugin>
     </gazebo>

File: src/gubot_one/description/ros2_control_gazebo_ign_fortress.xacro (robot description, xacro)
@@ -6,72 +6,52 @@
             <param name="position_proportional_gain">20.0</param>
         </hardware>
-        <xacro:if value="${'$(arg drive_type)' == 'diffdrive'}">
-            <joint name="left_wheel_joint">
-                <command_interface name="velocity">
-                    <param name="min">-10</param>
-                    <param name="max">10</param>
-                </command_interface>
-                <state_interface name="velocity"/>
-                <state_interface name="position"/>
-            </joint>
-            <joint name="right_wheel_joint">
-                <command_interface name="velocity">
-                    <param name="min">-10</param>
-                    <param name="max">10</param>
-                </command_interface>
-                <state_interface name="velocity"/>
-                <state_interface name="position"/>
-            </joint>
-        </xacro:if>
-        <xacro:if value="${'$(arg drive_type)' == 'mecanum'}">
-            <joint name="front_left_wheel_joint">
-                <command_interface name="velocity">
-                    <param name="min">-10</param>
-                    <param name="max">10</param>
-                </command_interface>
-                <state_interface name="velocity">
-                    <param name="initial_value">0.0</param>
-                </state_interface>
-                <state_interface name="position">
-                    <param name="initial_value">0.0</param>
-                </state_interface>
-            </joint>
-            <joint name="front_right_wheel_joint">
-                <command_interface name="velocity">
-                    <param name="min">-10</param>
-                    <param name="max">10</param>
-                </command_interface>
-                <state_interface name="velocity">
-                    <param name="initial_value">0.0</param>
-                </state_interface>
-                <state_interface name="position">
-                    <param name="initial_value">0.0</param>
-                </state_interface>
-            </joint>
-            <joint name="rear_left_wheel_joint">
-                <command_interface name="velocity">
-                    <param name="min">-10</param>
-                    <param name="max">10</param>
-                </command_interface>
-                <state_interface name="velocity">
-                    <param name="initial_value">0.0</param>
-                </state_interface>
-                <state_interface name="position">
-                    <param name="initial_value">0.0</param>
-                </state_interface>
-            </joint>
-            <joint name="rear_right_wheel_joint">
-                <command_interface name="velocity">
-                    <param name="min">-10</param>
-                    <param name="max">10</param>
-                </command_interface>
-                <state_interface name="velocity">
-                    <param name="initial_value">0.0</param>
-                </state_interface>
-                <state_interface name="position">
-                    <param name="initial_value">0.0</param>
-                </state_interface>
-            </joint>
-        </xacro:if>
+        <joint name="front_left_wheel_joint">
+            <command_interface name="velocity">
+                <param name="min">-10</param>
+                <param name="max">10</param>
+            </command_interface>
+            <state_interface name="velocity">
+                <param name="initial_value">0.0</param>
+            </state_interface>
+            <state_interface name="position">
+                <param name="initial_value">0.0</param>
+            </state_interface>
+        </joint>
+        <joint name="front_right_wheel_joint">
+            <command_interface name="velocity">
+                <param name="min">-10</param>
+                <param name="max">10</param>
+            </command_interface>
+            <state_interface name="velocity">
+                <param name="initial_value">0.0</param>
+            </state_interface>
+            <state_interface name="position">
+                <param name="initial_value">0.0</param>
+            </state_interface>
+        </joint>
+        <joint name="rear_left_wheel_joint">
+            <command_interface name="velocity">
+                <param name="min">-10</param>
+                <param name="max">10</param>
+            </command_interface>
+            <state_interface name="velocity">
+                <param name="initial_value">0.0</param>
+            </state_interface>
+            <state_interface name="position">
+                <param name="initial_value">0.0</param>
+            </state_interface>
+        </joint>
+        <joint name="rear_right_wheel_joint">
+            <command_interface name="velocity">
+                <param name="min">-10</param>
+                <param name="max">10</param>
+            </command_interface>
+            <state_interface name="velocity">
+                <param name="initial_value">0.0</param>
+            </state_interface>
+            <state_interface name="position">
+                <param name="initial_value">0.0</param>
+            </state_interface>
+        </joint>
         <!-- Nerf-Joints: NUR wenn use_nerf_hardware=true, sonst existieren diese Joints nicht in der URDF -->
         <!-- ALT: xacro:if value="$(arg use_nerf_hardware)" — "false" wurde als wahr evaluiert -->
@@ -111,10 +91,5 @@
     <gazebo>
         <plugin filename="gz_ros2_control-system" name="gz_ros2_control::GazeboSimROS2ControlPlugin">
-            <xacro:if value="${'$(arg drive_type)' == 'diffdrive'}">
-                <parameters>$(find gubot_one)/config/my_controllers.yaml</parameters>
-            </xacro:if>
-            <xacro:if value="${'$(arg drive_type)' == 'mecanum'}">
-                <parameters>$(find gubot_one)/config/mecanum_my_controllers.yaml</parameters>
-            </xacro:if>
+            <parameters>$(find gubot_one)/config/my_controllers.yaml</parameters>
         </plugin>
     </gazebo>

File: src/gubot_one/description/ros2_control_hardware.xacro (robot description, xacro)
@@ -3,98 +3,58 @@
     <xacro:arg name="use_nerf_hardware" default="true"/>
     <xacro:arg name="nerf_port" default="/dev/serial/by-id/usb-Arduino_LLC_Arduino_Leonardo-if00"/>
-    <xacro:if value="${'$(arg drive_type)' == 'diffdrive'}">
-        <ros2_control name="RealRobot" type="system">
-            <hardware>
-                <plugin>diffdrive_arduino/DiffDriveArduinoHardware</plugin>
-                <param name="left_wheel_name">left_wheel_joint</param>
-                <param name="right_wheel_name">right_wheel_joint</param>
-                <param name="loop_rate">30</param>
-                <param name="device">/dev/serial/by-id/usb-Raspberry_Pi_Pico_50443405786ACA1C-if00</param>
-                <param name="baud_rate">115200</param>
-                <param name="timeout_ms">1000</param>
-                <param name="enc_counts_per_rev">3436</param>
-            </hardware>
-            <joint name="left_wheel_joint">
-                <command_interface name="velocity">
-                    <param name="min">-10</param>
-                    <param name="max">10</param>
-                </command_interface>
-                <state_interface name="position"/>
-                <state_interface name="velocity"/>
-            </joint>
-            <joint name="right_wheel_joint">
-                <command_interface name="velocity">
-                    <param name="min">-10</param>
-                    <param name="max">10</param>
-                </command_interface>
-                <state_interface name="position"/>
-                <state_interface name="velocity"/>
-            </joint>
-            <sensor name="imu_sensor">
-                <state_interface name="linear_acceleration.x"/>
-                <state_interface name="linear_acceleration.y"/>
-                <state_interface name="linear_acceleration.z"/>
-                <state_interface name="angular_velocity.x"/>
-                <state_interface name="angular_velocity.y"/>
-                <state_interface name="angular_velocity.z"/>
-            </sensor>
-        </ros2_control>
-    </xacro:if>
-    <xacro:if value="${'$(arg drive_type)' == 'mecanum'}">
-        <ros2_control name="RealRobot" type="system">
-            <hardware>
-                <plugin>mecanum_pico/MecanumPicoHardware</plugin>
-                <param name="front_left_wheel_name">front_left_wheel_joint</param>
-                <param name="front_right_wheel_name">front_right_wheel_joint</param>
-                <param name="rear_left_wheel_name">rear_left_wheel_joint</param>
-                <param name="rear_right_wheel_name">rear_right_wheel_joint</param>
-                <param name="loop_rate">30</param>
-                <param name="device">/dev/serial/by-id/usb-Raspberry_Pi_Pico_50443405786ACA1C-if00</param>
-                <param name="baud_rate">115200</param>
-                <param name="timeout_ms">1000</param>
-                <param name="enc_counts_per_rev">3436</param>
-            </hardware>
-            <joint name="front_left_wheel_joint">
-                <command_interface name="velocity">
-                    <param name="min">-10</param>
-                    <param name="max">10</param>
-                </command_interface>
-                <state_interface name="position"/>
-                <state_interface name="velocity"/>
-            </joint>
-            <joint name="front_right_wheel_joint">
-                <command_interface name="velocity">
-                    <param name="min">-10</param>
-                    <param name="max">10</param>
-                </command_interface>
-                <state_interface name="position"/>
-                <state_interface name="velocity"/>
-            </joint>
-            <joint name="rear_left_wheel_joint">
-                <command_interface name="velocity">
-                    <param name="min">-10</param>
-                    <param name="max">10</param>
-                </command_interface>
-                <state_interface name="position"/>
-                <state_interface name="velocity"/>
-            </joint>
-            <joint name="rear_right_wheel_joint">
-                <command_interface name="velocity">
-                    <param name="min">-10</param>
-                    <param name="max">10</param>
-                </command_interface>
-                <state_interface name="position"/>
-                <state_interface name="velocity"/>
-            </joint>
-            <sensor name="imu_sensor">
-                <state_interface name="linear_acceleration.x"/>
-                <state_interface name="linear_acceleration.y"/>
-                <state_interface name="linear_acceleration.z"/>
-                <state_interface name="angular_velocity.x"/>
-                <state_interface name="angular_velocity.y"/>
-                <state_interface name="angular_velocity.z"/>
-            </sensor>
-        </ros2_control>
-    </xacro:if>
+    <ros2_control name="RealRobot" type="system">
+        <hardware>
+            <plugin>mecanum_pico/MecanumPicoHardware</plugin>
+            <param name="front_left_wheel_name">front_left_wheel_joint</param>
+            <param name="front_right_wheel_name">front_right_wheel_joint</param>
+            <param name="rear_left_wheel_name">rear_left_wheel_joint</param>
+            <param name="rear_right_wheel_name">rear_right_wheel_joint</param>
+            <param name="loop_rate">30</param>
+            <param name="device">/dev/serial/by-id/usb-Raspberry_Pi_Pico_50443405786ACA1C-if00</param>
+            <param name="baud_rate">115200</param>
+            <param name="timeout_ms">1000</param>
+            <param name="enc_counts_per_rev">3436</param>
+        </hardware>
+        <joint name="front_left_wheel_joint">
+            <command_interface name="velocity">
+                <param name="min">-10</param>
+                <param name="max">10</param>
+            </command_interface>
+            <state_interface name="position"/>
+            <state_interface name="velocity"/>
+        </joint>
+        <joint name="front_right_wheel_joint">
+            <command_interface name="velocity">
+                <param name="min">-10</param>
+                <param name="max">10</param>
+            </command_interface>
+            <state_interface name="position"/>
+            <state_interface name="velocity"/>
+        </joint>
+        <joint name="rear_left_wheel_joint">
+            <command_interface name="velocity">
+                <param name="min">-10</param>
+                <param name="max">10</param>
+            </command_interface>
+            <state_interface name="position"/>
+            <state_interface name="velocity"/>
+        </joint>
+        <joint name="rear_right_wheel_joint">
+            <command_interface name="velocity">
+                <param name="min">-10</param>
+                <param name="max">10</param>
+            </command_interface>
+            <state_interface name="position"/>
+            <state_interface name="velocity"/>
+        </joint>
+        <sensor name="imu_sensor">
+            <state_interface name="linear_acceleration.x"/>
+            <state_interface name="linear_acceleration.y"/>
+            <state_interface name="linear_acceleration.z"/>
+            <state_interface name="angular_velocity.x"/>
+            <state_interface name="angular_velocity.y"/>
+            <state_interface name="angular_velocity.z"/>
+        </sensor>
+    </ros2_control>
     <xacro:if value="$(arg use_nerf_hardware)">
         <ros2_control name="NerfSystem" type="system">
