Commit message: feat: Enhance agent workflows, code style rules, and add code review skill, alongside updates to Gazebo world and ROS2 control integration.

File: src/nerf_launch_system/description/urdf/gz_classic_ros2_control.xacro (robot description, xacro)
@@ -2,4 +2,9 @@
 <robot xmlns:xacro="http://www.ros.org/wiki/xacro">
     <xacro:macro name="nerf_ros2_control">
+        <gazebo>
+            <plugin filename="libgazebo_ros2_control.so" name="gazebo_ros2_control">
+                <parameters>$(find nerf_launch_system)/config/controllers.yaml</parameters>
+            </plugin>
+        </gazebo>
         <ros2_control name="NerfGazeboSystem" type="system">
             <hardware>
@@ -26,4 +31,8 @@
                 <command_interface name="velocity"/>
                 <state_interface name="velocity"/>
+                <state_interface name="position"/>
+            </joint>
+            <joint name="system_arming_joint">
+                <command_interface name="position"/>
                 <state_interface name="position"/>
             </joint>
@@ -53,4 +62,8 @@
             <state_interface name="position"/>
         </joint>
+        <joint name="system_arming_joint">
+            <command_interface name="position"/>
+            <state_interface name="position"/>
+        </joint>
     </xacro:macro>
 </robot>

File: src/nerf_launch_system/description/urdf/ros2_control.xacro (robot description, xacro)
@@ -3,12 +3,11 @@
     <xacro:macro name="nerf_ros2_control">
         <gazebo>
-            <plugin filename="ign_ros2_control-system" name="ign_ros2_control::IgnitionROS2ControlPlugin">
+            <plugin filename="ign_ros2_control-system" name="gz_ros2_control::GazeboSimROS2ControlPlugin">
                 <parameters>$(find nerf_launch_system)/config/controllers.yaml</parameters>
-                <parameters>$(find nerf_launch_system)/config/gains.yaml</parameters>
             </plugin>
         </gazebo>
         <ros2_control name="IgnitionSystem" type="system">
             <hardware>
-                <plugin>ign_ros2_control/IgnitionSystem</plugin>
+                <plugin>gz_ros2_control/GazeboSimSystem</plugin>
             </hardware>
             <joint name="trigger_joint">
@@ -24,16 +23,16 @@
                 <state_interface name="position"/>
             </joint>
-            <!-- Flywheel Joints entfernt (FSM)
             <joint name="flywheel_left_joint">
-                <command_interface name="velocity"/>
                 <state_interface name="velocity"/>
                 <state_interface name="position"/>
             </joint>
             <joint name="flywheel_right_joint">
-                <command_interface name="velocity"/>
                 <state_interface name="velocity"/>
                 <state_interface name="position"/>
             </joint>
-            -->
+            <joint name="system_arming_joint">
+                <command_interface name="position"/>
+                <state_interface name="position"/>
+            </joint>
         </ros2_control>
     </xacro:macro>
@@ -63,4 +62,8 @@
         </joint>
         -->
+        <joint name="system_arming_joint">
+            <command_interface name="position"/>
+            <state_interface name="position"/>
+        </joint>
     </xacro:macro>
 </robot>
