Commit message: refactor: Rename Nerf launcher's trigger controller to tilt, pusher controller to shooter, and remove explicit flywheel control.

File: src/nerf_launch_system/description/urdf/launcher.urdf.xacro (robot description, xacro)
@@ -163,5 +163,5 @@
         </visual>
     </link>
-    <joint name="trigger_joint" type="revolute">
+    <joint name="tilt_joint" type="revolute">
         <origin xyz="0.08882309 0.10354221000000001 -0.00119223" rpy="-1.5707963267948943 -3.374960801568061e-11 -1.570862213919093" />
         <parent link="bottom_plate" />
@@ -212,5 +212,5 @@
         <child link="Servo_dart_pusher" />
     </joint>
-    <joint name="dart_pusher_joint" type="continuous">
+    <joint name="shooter_joint" type="continuous">
         <origin xyz="0.004999060000000002 0.014171329999999998 0.013443680000000003" rpy="1.5707963267948966 2.7571572048402603e-21 -2.354302446406244e-21" />
         <parent link="Servo_dart_pusher" />

Commit message: refactor: Rename `trigger_joint` to `tilt_joint` and `dart_pusher_joint` to `shooter_joint`, update `shooter_joint` command interface, add `system_arming_joint`, and switch mesh paths to `package://`.

File: src/nerf_launch_system/description/urdf/launcher.urdf.xacro (robot description, xacro)
@@ -1,4 +1,17 @@
 <?xml version='1.0' encoding='utf-8'?>
 <robot xmlns:xacro="http://www.ros.org/wiki/xacro" name="nerf_launch_system">
+    <link name="arming_switch_link">
+        <inertial>
+            <mass value="0.1" />
+            <inertia ixx="0.001" iyy="0.001" izz="0.001" ixy="0.0" iyz="0.0" ixz="0.0" />
+        </inertial>
+    </link>
+    <joint name="system_arming_joint" type="revolute">
+        <parent link="bottom_plate"/>
+        <child link="arming_switch_link"/>
+        <origin xyz="0 0 0" rpy="0 0 0"/>
+        <limit lower="0" upper="1" effort="1" velocity="1"/>
+        <axis xyz="0 0 1"/>
+    </joint>
     <link name="bottom_plate">
         <inertial>
@@ -10,5 +23,5 @@
             <origin xyz="0.0 0.0 0.0" rpy="0.0 0.0 0.0" />
             <geometry>
-                <mesh filename="file://$(find nerf_launch_system)/description/meshes/bottom_plate.stl" scale="0.001 0.001 0.001" />
+                <mesh filename="package://nerf_launch_system/description/meshes/bottom_plate.stl" scale="0.001 0.001 0.001" />
             </geometry>
         </visual>
@@ -29,5 +42,5 @@
             <origin xyz="0.09803428669398517 -4.3732793080548534e-05 -0.013700000763976723" rpy="1.5703501879750486 -1.5707963267948937 0" />
             <geometry>
-                <mesh filename="file://$(find nerf_launch_system)/description/meshes/motor_bracket.stl" scale="0.001 0.001 0.001" />
+                <mesh filename="package://nerf_launch_system/description/meshes/motor_bracket.stl" scale="0.001 0.001 0.001" />
             </geometry>
         </visual>
@@ -42,5 +55,5 @@
             <origin xyz="0.009991696360929777 -0.1260585761325394 0.08876880466816899" rpy="-3.141146514736195 1.079162159671481e-15 3.1415267664655997" />
             <geometry>
-                <mesh filename="file://$(find nerf_launch_system)/description/meshes/magazin.stl" scale="0.001 0.001 0.001" />
+                <mesh filename="package://nerf_launch_system/description/meshes/magazin.stl" scale="0.001 0.001 0.001" />
             </geometry>
         </visual>
@@ -55,5 +68,5 @@
             <origin xyz="-1.73567760164417e-09 3.029328534687181e-09 -1.3556827271887785e-09" rpy="-1.5707188555909968 0.00043936100150414944 1.7453951561374372" />
             <geometry>
-                <mesh filename="file://$(find nerf_launch_system)/description/meshes/motor_right.stl" scale="0.001 0.001 0.001" />
+                <mesh filename="package://nerf_launch_system/description/meshes/motor_right.stl" scale="0.001 0.001 0.001" />
             </geometry>
         </visual>
@@ -68,5 +81,5 @@
             <origin xyz="-1.8333526696778791e-09 -2.050084864091417e-09 -1.355682762715915e-09" rpy="-1.5711117946140916 0.00031546780349864484 0.7854640007616747" />
             <geometry>
-                <mesh filename="file://$(find nerf_launch_system)/description/meshes/motor_left.stl" scale="0.001 0.001 0.001" />
+                <mesh filename="package://nerf_launch_system/description/meshes/motor_left.stl" scale="0.001 0.001 0.001" />
             </geometry>
         </visual>
@@ -81,5 +94,5 @@
             <origin xyz="0.004998394584003245 0.024345667304006825 -0.010460860261822842" rpy="1.570796326794895 -0.0004461388535984491 -1.5707304396707022" />
             <geometry>
-                <mesh filename="file://$(find nerf_launch_system)/description/meshes/Servo_dart_pusher.stl" scale="0.001 0.001 0.001" />
+                <mesh filename="package://nerf_launch_system/description/meshes/Servo_dart_pusher.stl" scale="0.001 0.001 0.001" />
             </geometry>
         </visual>
@@ -94,5 +107,5 @@
             <origin xyz="-0.0631325544432252 0.01313155884148008 -0.0631300993428637" rpy="-1.570165432787083 0.7853321767598774 -3.1411465441724866" />
             <geometry>
-                <mesh filename="file://$(find nerf_launch_system)/description/meshes/flywheel_left.stl" scale="0.001 0.001 0.001" />
+                <mesh filename="package://nerf_launch_system/description/meshes/flywheel_left.stl" scale="0.001 0.001 0.001" />
             </geometry>
         </visual>
@@ -107,5 +120,5 @@
             <origin xyz="-0.01550858803514851 0.013120498025483157 -0.08792554788989197" rpy="-1.568228080674074 1.3961969502773832 -3.139063424976714" />
             <geometry>
-                <mesh filename="file://$(find nerf_launch_system)/description/meshes/flywheel_right.stl" scale="0.001 0.001 0.001" />
+                <mesh filename="package://nerf_launch_system/description/meshes/flywheel_right.stl" scale="0.001 0.001 0.001" />
             </geometry>
         </visual>
@@ -120,5 +133,5 @@
             <origin xyz="5.0358234648939514e-09 -0.0031999983978120905 1.4265863324780527e-06" rpy="-1.5712424656484945 6.588712419531712e-05 9.66531786022265e-16" />
             <geometry>
-                <mesh filename="file://$(find nerf_launch_system)/description/meshes/pusher_servo_part.stl" scale="0.001 0.001 0.001" />
+                <mesh filename="package://nerf_launch_system/description/meshes/pusher_servo_part.stl" scale="0.001 0.001 0.001" />
             </geometry>
         </visual>
@@ -133,5 +146,5 @@
             <origin xyz="0.0089380699537615 -0.0803571481976858 -0.002142981347950717" rpy="-0.000446138853596889 -1.0791087584284575e-15 -6.58871241935617e-05" />
             <geometry>
-                <mesh filename="file://$(find nerf_launch_system)/description/meshes/Turret.stl" scale="0.001 0.001 0.001" />
+                <mesh filename="package://nerf_launch_system/description/meshes/Turret.stl" scale="0.001 0.001 0.001" />
             </geometry>
         </visual>
@@ -146,5 +159,5 @@
             <origin xyz="0.004000004389203955 -0.08928319312789187 0.01647600710867764" rpy="0.029400113955168578 -8.659366307345483e-14 -3.141592653583827" />
             <geometry>
-                <mesh filename="file://$(find nerf_launch_system)/description/meshes/Servoarm-v1.stl" scale="0.001 0.001 0.001" />
+                <mesh filename="package://nerf_launch_system/description/meshes/Servoarm-v1.stl" scale="0.001 0.001 0.001" />
             </geometry>
         </visual>
@@ -159,5 +172,5 @@
             <origin xyz="0.032232880187464355 0.10890697936911703 -0.024499995611303272" rpy="-8.077935669498046e-28 7.226432496549954e-26 1.570796326794921" />
             <geometry>
-                <mesh filename="file://$(find nerf_launch_system)/description/meshes/Nerf-Dart-Launcher_Servo-MG-v1.stl" scale="0.001 0.001 0.001" />
+                <mesh filename="package://nerf_launch_system/description/meshes/Nerf-Dart-Launcher_Servo-MG-v1.stl" scale="0.001 0.001 0.001" />
             </geometry>
         </visual>
@@ -245,18 +258,4 @@
         <xacro:nerf_ros2_control_hardware port="$(arg port)"/>
     </xacro:if>
-    <xacro:unless value="$(arg use_hardware)">
-        <link name="arming_switch_link">
-            <inertial>
-                <mass value="0.1" />
-                <inertia ixx="0.001" iyy="0.001" izz="0.001" ixy="0.0" iyz="0.0" ixz="0.0" />
-            </inertial>
-        </link>
-    <joint name="system_arming_joint" type="revolute">
-        <parent link="bottom_plate"/>
-        <child link="arming_switch_link"/>
-        <origin xyz="0 0 0" rpy="0 0 0"/>
-        <limit lower="0" upper="1" effort="1" velocity="1"/>
-        <axis xyz="0 0 1"/>
-    </joint>
     <xacro:unless value="$(arg integrated_mode)">
         <xacro:arg name="use_gazebo_classic" default="false"/>
@@ -269,4 +268,3 @@
         <xacro:nerf_ros2_control />
     </xacro:unless>
-    </xacro:unless>
 </robot>

File: src/nerf_launch_system/description/urdf/ros2_control.xacro (robot description, xacro)
@@ -11,5 +11,5 @@
                 <plugin>gz_ros2_control/GazeboSimSystem</plugin>
             </hardware>
-            <joint name="trigger_joint">
+            <joint name="tilt_joint">
                 <command_interface name="position"/>
                 <state_interface name="velocity"/>
@@ -18,6 +18,6 @@
                 </state_interface>
             </joint>
-            <joint name="dart_pusher_joint">
-                <command_interface name="velocity"/>
+            <joint name="shooter_joint">
+                <command_interface name="position"/>
                 <state_interface name="velocity"/>
                 <state_interface name="position"/>
@@ -38,5 +38,5 @@
     </xacro:macro>
     <xacro:macro name="nerf_ros2_control_joints_only">
-        <joint name="trigger_joint">
+        <joint name="tilt_joint">
             <command_interface name="position"/>
             <state_interface name="velocity"/>
@@ -45,6 +45,6 @@
             </state_interface>
         </joint>
-        <joint name="dart_pusher_joint">
-            <command_interface name="velocity"/>
+        <joint name="shooter_joint">
+            <command_interface name="position"/>
             <state_interface name="velocity"/>
             <state_interface name="position"/>

File: src/nerf_launch_system/description/urdf/ros2_control_hardware.xacro (robot description, xacro)
@@ -8,11 +8,11 @@
                 <param name="baud_rate">115200</param>
             </hardware>
-            <joint name="trigger_joint">
+            <joint name="tilt_joint">
                 <command_interface name="position"/>
                 <state_interface name="position"/>
             </joint>
-            <joint name="dart_pusher_joint">
-                <command_interface name="velocity"/>
-                <state_interface name="velocity"/>
+            <joint name="shooter_joint">
+                <command_interface name="position"/>
+                <state_interface name="position"/>
             </joint>
             <!-- Flywheel Joints entfernt: Firmware-FSM steuert Flywheels autonom via SHOT -->
@@ -29,4 +29,11 @@
             <joint name="system_arming_joint">
                 <command_interface name="position"/>
+                <state_interface name="position"/>
+            </joint>
+            <joint name="flywheel_left_joint">
+                <state_interface name="position"/>
+            </joint>
+            <joint name="flywheel_right_joint">
+                <state_interface name="position"/>
             </joint>
         </ros2_control>
