Commit message: feat: Implement Gazebo Classic simulation fixes by adjusting URDF physics parameters and introducing a new simulation setup strategy.

File: src/nerf_launch_system/description/urdf/launcher_gazebo_classic.urdf.xacro (robot description, xacro)
@@ -3,6 +3,6 @@
     <link name="arming_switch_link">
         <inertial>
-            <mass value="0.1" />
-            <inertia ixx="0.001" iyy="0.001" izz="0.001" ixy="0.0" iyz="0.0" ixz="0.0" />
+            <mass value="0.001" />
+            <inertia ixx="1.e-06" iyy="1.e-06" izz="1.e-06" ixy="0.0" iyz="0.0" ixz="0.0" />
         </inertial>
     </link>
@@ -13,11 +13,11 @@
         <limit lower="0" upper="1" effort="1" velocity="1"/>
         <axis xyz="0 0 1"/>
-        <dynamics damping="20.0" friction="10.0"/>
+        <dynamics damping="0.1" friction="0.1"/>
     </joint>
     <link name="bottom_plate">
         <inertial>
             <origin xyz="0.07506008367977571 0.06788755296524361 -0.015949194976296238" rpy="0.0 0.0 0.0" />
-            <mass value="0.1" />
-            <inertia ixx="0.001" iyy="0.001" izz="0.001" ixy="0.0" iyz="0.0" ixz="0.0" />
+            <mass value="0.001" />
+            <inertia ixx="1.e-06" iyy="1.e-06" izz="1.e-06" ixy="0.0" iyz="0.0" ixz="0.0" />
         </inertial>
         <visual name="bottom_plate_visual">
@@ -37,6 +37,6 @@
         <inertial>
             <origin xyz="0.06 0 0" rpy="0 0 0" />
-            <mass value="0.1" />
-            <inertia ixx="0.001" iyy="0.001" izz="0.001" ixy="0.0" iyz="0.0" ixz="0.0" />
+            <mass value="0.001" />
+            <inertia ixx="1.e-06" iyy="1.e-06" izz="1.e-06" ixy="0.0" iyz="0.0" ixz="0.0" />
         </inertial>
         <visual name="motor_bracket_visual">
@@ -50,6 +50,6 @@
         <inertial>
             <origin xyz="0 -0.02 0.05" rpy="0 0 0" />
-            <mass value="0.1" />
-            <inertia ixx="0.001" iyy="0.001" izz="0.001" ixy="0.0" iyz="0.0" ixz="0.0" />
+            <mass value="0.001" />
+            <inertia ixx="1.e-06" iyy="1.e-06" izz="1.e-06" ixy="0.0" iyz="0.0" ixz="0.0" />
         </inertial>
         <visual name="magazin_visual">
@@ -63,6 +63,6 @@
         <inertial>
             <origin xyz="0 0 0" rpy="0 0 0" />
-            <mass value="0.1" />
-            <inertia ixx="0.001" iyy="0.001" izz="0.001" ixy="0.0" iyz="0.0" ixz="0.0" />
+            <mass value="0.001" />
+            <inertia ixx="1.e-06" iyy="1.e-06" izz="1.e-06" ixy="0.0" iyz="0.0" ixz="0.0" />
         </inertial>
         <visual name="motor_right_visual">
@@ -76,6 +76,6 @@
         <inertial>
             <origin xyz="0 0 0" rpy="0 0 0" />
-            <mass value="0.1" />
-            <inertia ixx="0.001" iyy="0.001" izz="0.001" ixy="0.0" iyz="0.0" ixz="0.0" />
+            <mass value="0.001" />
+            <inertia ixx="1.e-06" iyy="1.e-06" izz="1.e-06" ixy="0.0" iyz="0.0" ixz="0.0" />
         </inertial>
         <visual name="motor_left_visual">
@@ -89,6 +89,6 @@
         <inertial>
             <origin xyz="0 0.02 -0.01" rpy="0 0 0" />
-            <mass value="0.1" />
-            <inertia ixx="0.001" iyy="0.001" izz="0.001" ixy="0.0" iyz="0.0" ixz="0.0" />
+            <mass value="0.001" />
+            <inertia ixx="1.e-06" iyy="1.e-06" izz="1.e-06" ixy="0.0" iyz="0.0" ixz="0.0" />
         </inertial>
         <visual name="Servo_dart_pusher_visual">
@@ -102,6 +102,6 @@
         <inertial>
             <origin xyz="0 0.003 0" rpy="0 0 0" />
-            <mass value="0.1" />
-            <inertia ixx="0.001" iyy="0.001" izz="0.001" ixy="0.0" iyz="0.0" ixz="0.0" />
+            <mass value="0.001" />
+            <inertia ixx="1.e-06" iyy="1.e-06" izz="1.e-06" ixy="0.0" iyz="0.0" ixz="0.0" />
         </inertial>
         <visual name="flywheel_left_visual">
@@ -115,6 +115,6 @@
         <inertial>
             <origin xyz="0 0.003 0" rpy="0 0 0" />
-            <mass value="0.1" />
-            <inertia ixx="0.001" iyy="0.001" izz="0.001" ixy="0.0" iyz="0.0" ixz="0.0" />
+            <mass value="0.001" />
+            <inertia ixx="1.e-06" iyy="1.e-06" izz="1.e-06" ixy="0.0" iyz="0.0" ixz="0.0" />
         </inertial>
         <visual name="flywheel_right_visual">
@@ -128,6 +128,6 @@
         <inertial>
             <origin xyz="-0.002 -0.002 0" rpy="0 0 0" />
-            <mass value="0.1" />
-            <inertia ixx="0.001" iyy="0.001" izz="0.001" ixy="0.0" iyz="0.0" ixz="0.0" />
+            <mass value="0.001" />
+            <inertia ixx="1.e-06" iyy="1.e-06" izz="1.e-06" ixy="0.0" iyz="0.0" ixz="0.0" />
         </inertial>
         <visual name="pusher_servo_part_visual">
@@ -141,6 +141,6 @@
         <inertial>
             <origin xyz="0 -0.02 0.01" rpy="0 0 0" />
-            <mass value="0.1" />
-            <inertia ixx="0.001" iyy="0.001" izz="0.001" ixy="0.0" iyz="0.0" ixz="0.0" />
+            <mass value="0.001" />
+            <inertia ixx="1.e-06" iyy="1.e-06" izz="1.e-06" ixy="0.0" iyz="0.0" ixz="0.0" />
         </inertial>
         <visual name="Turret_visual">
@@ -154,6 +154,6 @@
         <inertial>
             <origin xyz="0.003 0.004 0" rpy="0 0 0" />
-            <mass value="0.1" />
-            <inertia ixx="0.001" iyy="0.001" izz="0.001" ixy="0.0" iyz="0.0" ixz="0.0" />
+            <mass value="0.001" />
+            <inertia ixx="1.e-06" iyy="1.e-06" izz="1.e-06" ixy="0.0" iyz="0.0" ixz="0.0" />
         </inertial>
         <visual name="Servoarm-v1_visual">
@@ -167,6 +167,6 @@
         <inertial>
             <origin xyz="0.01 0 -0.01" rpy="0 0 0" />
-            <mass value="0.1" />
-            <inertia ixx="0.001" iyy="0.001" izz="0.001" ixy="0.0" iyz="0.0" ixz="0.0" />
+            <mass value="0.001" />
+            <inertia ixx="1.e-06" iyy="1.e-06" izz="1.e-06" ixy="0.0" iyz="0.0" ixz="0.0" />
         </inertial>
         <visual name="Nerf-Dart-Launcher_Servo-MG-v1_visual">
@@ -181,8 +181,7 @@
         <parent link="bottom_plate" />
         <child link="motor_bracket" />
-        <axis xyz="1.1287570791617654e-07 2.227474133869779e-15 1.0000000021779938" />
-        <!-- <limit lower="5.23" upper="6.28" effort="1.0" velocity="5.0" /> -->
-        <limit lower="-0.52" upper="0.52" effort="1.0" velocity="5.0" />
-        <dynamics damping="10.0" friction="5.0"/>
+        <axis xyz="0 0 -1" />
+        <limit lower="0.0" upper="0.52" effort="1.0" velocity="5.0" />
+        <dynamics damping="0.1" friction="0.1"/>
     </joint>
     <joint name="motor_bracket_motor_left_fix_motor_bracket" type="fixed">
@@ -226,6 +225,6 @@
         <child link="pusher_servo_part" />
         <axis xyz="-2.7546953265439552e-21 1.0 -0.000446" />
-        <limit effort="0.1" velocity="20.0"/>
-        <dynamics damping="15.0" friction="8.0"/>
+        <limit effort="1.0" velocity="20.0"/>
+        <dynamics damping="0.1" friction="0.1"/>
     </joint>
     <joint name="bottom_plate_servo_fix_bottom_plate" type="fixed">
