Commit message: fix(nerf): Tilt auf Joint-Space vereinheitlicht, Achse invertiert, Feuern auf RT
- trigger_joint-Achse invertiert (0 0 -1): positiv = Launcher hoch aus dem
  Koerper. ALT: CAD-Achse drehte bei positiven Kommandos in den Koerper —
  das Init "UP=+max" fuhr genau falsch herum
- Alle Steuer-Nodes (nerf_joy, Keyboard, nerf_control_node) kommandieren
  Joint-Space ±0.52 rad. ALT: Servo-Rohwerte 5.23–6.28 rad wurden in der
  Sim dauerhaft ans URDF-Limit geclampt — keine sichtbare Bewegung
- NerfSystem clampt Tilt-Kommandos auf tilt_min/tilt_max (URDF-Params);
  Firmware bleibt deltabasiert (UP/DN-Pulse), Verhalten auf HW unveraendert
- Feuern von A auf RT verlegt (Achse 5 analog + Button-7-Fallback,
  Flanken-Erkennung). ALT: A kollidierte mit dem teleop_twist_joy-Deadman
  (enable_button 0) — Fahren-Enable haette im armed-Zustand geschossen
- nerf_joy: LB/RB-Richtungen zu Doku und Achse konsistent (LB=down, RB=up)

Co-Authored-By: Claude Fable 5 <noreply@anthropic.com>

File: src/nerf_launch_system/description/urdf/nerf_launcher.urdf.xacro (robot description, xacro)
@@ -167,5 +167,10 @@
         <parent link="bottom_plate" />
         <child link="motor_bracket" />
-        <axis xyz="1.1287570791617654e-07 2.227474133869779e-15 1.0000000021779938" />
+        <!-- Achse invertiert: positiv = Launcher hoch (aus dem Körper heraus).
+             ALT: xyz="1.1e-07 2.2e-15 1.0" (CAD-Export) — positiv drehte den
+             Launcher NACH UNTEN in den Roboterkörper; das Init-Kommando
+             "UP = +tilt_max" fuhr ihn damit genau falsch herum. Hardware ist
+             deltabasiert (UP-Pulse bei steigendem Soll) und bleibt konsistent. -->
+        <axis xyz="0 0 -1" />
         <!-- <xacro:if value="$(arg use_gazebo_classic)"> -->
         <!--     <!- - Classic Simulation parser requires the original bounds - -> -->
