Commit message: refactor(pakete): gubot_one nach rosbot-Muster in 6 Pakete + Metapaket aufgeteilt
Monopaket gubot_one aufgesplittet (Vorlage rosbot_ros, flaches
share/<pkg>-Layout, git mv fuer History):

- gubot_description: URDF/Xacro, Meshes, RViz, load_urdf.launch.py
- gubot_controller:  controller.launch.py, controllers.yaml, twist_mux.yaml
- gubot_gazebo:      simulation.launch.py, Welten, Modelle, gz-Bridge, env-hook
- gubot_localization: ekf.launch.py, ekf.yaml
- gubot_bringup:     launch_all_real.launch.py, Joystick/Kamera/LiDAR, joystick.yaml
- gubot_utils:       Skripte, Autostart-Service, CycloneDDS-Configs, Doku
- gubot_one:         nur noch Metapaket (exec_depend auf die 6 Pakete)

Alle Pfad-Kompositionen, Includes, Tests und Doku auf die neuen Pakete
umgestellt; Gazebo-Modellname bleibt gubot_one (Bridge-Topics unveraendert).
ball_tracker.launch.py entfernt (war nur Vorlage fuer face_tracker).
Tilt-Spawner-Test an declare_parameter und ausgelagertes
nerf_ros2_control_hardware-Makro angepasst.

Verifiziert: colcon build (13 Pakete), 23/23 pytest gruen, check_urdf,
Launch-Smoke (-s) fuer bringup/gazebo/controller, 90-s-Sim-Lauf mit
allen 6 aktiven Controllern.

Co-Authored-By: Claude Fable 5 <noreply@anthropic.com>

File: src/nerf_launch_system/description/urdf/ros2_control_gazebo_fortress.xacro (robot description, xacro)
@@ -16,5 +16,5 @@
                 <state_interface name="velocity"/>
                 <state_interface name="position">
-                  <param name="initial_value">6.28</param>
+                  <param name="initial_value">0.52</param>
                 </state_interface>
             </joint>
@@ -24,16 +24,8 @@
                 <state_interface name="position"/>
             </joint>
-            <!-- Flywheel Joints entfernt (FSM)
-            <joint name="flywheel_left_joint">
-                <command_interface name="velocity"/>
-                <state_interface name="velocity"/>
+            <joint name="system_arming_joint">
+                <command_interface name="position"/>
                 <state_interface name="position"/>
             </joint>
-            <joint name="flywheel_right_joint">
-                <command_interface name="velocity"/>
-                <state_interface name="velocity"/>
-                <state_interface name="position"/>
-            </joint>
-            -->
         </ros2_control>
     </xacro:macro>
@@ -51,16 +43,8 @@
             <state_interface name="position"/>
         </joint>
-        <!-- Flywheel Joints entfernt (FSM)
-        <joint name="flywheel_left_joint">
-            <command_interface name="velocity"/>
-            <state_interface name="velocity"/>
+        <joint name="system_arming_joint">
+            <command_interface name="position"/>
             <state_interface name="position"/>
         </joint>
-        <joint name="flywheel_right_joint">
-            <command_interface name="velocity"/>
-            <state_interface name="velocity"/>
-            <state_interface name="position"/>
-        </joint>
-        -->
     </xacro:macro>
 </robot>

File: src/nerf_launch_system/description/urdf/ros2_control_hardware_nerf.xacro (robot description, xacro)
@@ -1,10 +1,15 @@
 <?xml version="1.0"?>
 <robot xmlns:xacro="http://www.ros.org/wiki/xacro">
-    <xacro:macro name="nerf_ros2_control_hardware" params="port">
+    <!-- tilt_min/tilt_max: Joint-Space-Range (rad) für den Tilt-Servo =
+         trigger_joint URDF-Limits. Einzige Quelle der Wahrheit; NerfSystem
+         clampt Kommandos zusätzlich darauf. Default ±0.52 rad. -->
+    <xacro:macro name="nerf_ros2_control_hardware" params="port tilt_min:=-0.52 tilt_max:=0.52">
         <ros2_control name="NerfSystem" type="system">
             <hardware>
                 <plugin>nerf_launch_system/NerfSystem</plugin>
-                <param name="port">$(arg port)</param>
+                <param name="port">${port}</param>
                 <param name="baud_rate">115200</param>
+                <param name="tilt_min">${tilt_min}</param>
+                <param name="tilt_max">${tilt_max}</param>
             </hardware>
             <joint name="trigger_joint">
@@ -16,15 +21,4 @@
                 <state_interface name="velocity"/>
             </joint>
-            <!-- Flywheel Joints entfernt: Firmware-FSM steuert Flywheels autonom via SHOT -->
-            <!--
-            <joint name="flywheel_left_joint">
-                <command_interface name="velocity"/>
-                <state_interface name="velocity"/>
-            </joint>
-            <joint name="flywheel_right_joint">
-                <command_interface name="velocity"/>
-                <state_interface name="velocity"/>
-            </joint>
-            -->
             <joint name="system_arming_joint">
                 <command_interface name="position"/>
