Commit message: Add URDF and SDF models for nerf_launch_system
- Created a new URDF file `gz_classic_launcher.urdf.xacro` to define the robot model with various links and joints.
- Added a new URDF file `launcher_gazebo_classic.urdf.xacro` for the Gazebo Classic simulation.
- Updated the existing `launcher.urdf.xacro` to modify the limits of the `tilt_joint`.
- Introduced `model.config` and `model.sdf` files to provide metadata and structure for the nerf_launch_system model in Gazebo.
- Updated `CMakeLists.txt` to install the new model configuration and SDF files.

File: src/gubot_one_description/description/camera.xacro (robot description, xacro)
@@ -45,13 +45,6 @@
                 </clip>
             </camera>
-            <xacro:if value="$(arg use_gazebo_classic)">
-                <plugin name="camera_controller" filename="libgazebo_ros_camera.so">
-                    <frame_name>camera_link_optical</frame_name>
-                </plugin>
-            </xacro:if>
-            <xacro:unless value="$(arg use_gazebo_classic)">
                 <topic>camera/image_raw</topic>
-            </xacro:unless>
-        </sensor>
+            </sensor>
     </gazebo>
 </robot>

File: src/gubot_one_description/description/robot.urdf.xacro (robot description, xacro)
@@ -6,18 +6,7 @@
     <xacro:arg name="use_nerf_hardware" default="true"/>
     <xacro:arg name="nerf_port" default="/dev/serial/by-id/usb-Arduino_LLC_Arduino_Leonardo-if00"/>
-    <xacro:arg name="use_gazebo_classic" default="false"/>
     <xacro:arg name="use_fake_hardware" default="false"/>
     <xacro:include filename="robot_core.xacro" />
-    <xacro:if value="$(arg use_ros2_control)">
-        <xacro:if value="$(arg use_gazebo_classic)">
-            <xacro:include filename="gz_classic_ros2_control.xacro" />
-        </xacro:if>
-        <xacro:unless value="$(arg use_gazebo_classic)">
-            <xacro:include filename="ros2_control.xacro" />
-        </xacro:unless>
-    </xacro:if>
-    <xacro:unless value="$(arg use_ros2_control)">
-        <xacro:include filename="gazebo_control.xacro" />
-    </xacro:unless>
+    <xacro:include filename="ros2_control.xacro" />
     <!-- <xacro:include filename="lidar.xacro" /> -->
     <xacro:include filename="camera.xacro" />

File: src/gubot_one_description/description/robot_core_classic.xacro (robot description, xacro)
@@ -1,4 +1,4 @@
 <?xml version="1.0"?>
-<robot xmlns:xacro="http://www.ros.org/wiki/xacro" >
+<robot xmlns:xacro="http://www.ros.org/wiki/xacro">
     <xacro:include filename="inertial_macros.xacro"/>
     <xacro:property name="chassis_length" value="0.335"/>
@@ -38,5 +38,6 @@
         <parent link="base_link"/>
         <child link="base_footprint"/>
-        <origin xyz="0 0 0" rpy="0 0 0"/>
+        <!-- <origin xyz="0 0 0" rpy="0 0 0"/> -->
+        <origin xyz="0 0 -${wheel_radius}" rpy="0 0 0"/>
     </joint>
     <link name="base_footprint">
@@ -68,4 +69,5 @@
     <gazebo reference="chassis">
         <material>Gazebo/Orange</material>
+        <self_collide>false</self_collide>
     </gazebo>
     <!-- IMU LINK -->
@@ -154,5 +156,7 @@
                 </linear_acceleration>
             </imu>
-                <topic>imu_sensor/imu_data</topic>
+            <plugin name="imu_plugin" filename="libgazebo_ros_imu_sensor.so">
+                <initial_orientation_as_reference>false</initial_orientation_as_reference>
+            </plugin>
         </sensor>
     </gazebo>
@@ -163,4 +167,5 @@
         <origin xyz="0 ${wheel_offset_y} 0" rpy="-${pi/2} 0 0" />
         <axis xyz="0 0 1"/>
+        <dynamics damping="20.0" friction="8.0"/>
     </joint>
     <link name="left_wheel">
@@ -182,4 +187,7 @@
     <gazebo reference="left_wheel">
         <material>Gazebo/Blue</material>
+        <mu1 value="1.0"/>
+        <mu2 value="1.0"/>
+        <self_collide>false</self_collide>
     </gazebo>
     <!-- RIGHT WHEEL LINK -->
@@ -189,4 +197,5 @@
         <origin xyz="0 ${-wheel_offset_y} 0" rpy="${pi/2} 0 0" />
         <axis xyz="0 0 -1"/>
+        <dynamics damping="20.0" friction="8.0"/>
     </joint>
     <link name="right_wheel">
@@ -208,4 +217,7 @@
     <gazebo reference="right_wheel">
         <material>Gazebo/Blue</material>
+        <mu1 value="1.0"/>
+        <mu2 value="1.0"/>
+        <self_collide>false</self_collide>
     </gazebo>
     <!-- CASTER WHEEL LINK -->

File: src/nerf_launch_system/description/urdf/gz_classic_launcher.urdf.xacro (robot description, xacro)
@@ -23,5 +23,5 @@
             <origin xyz="0.0 0.0 0.0" rpy="0.0 0.0 0.0" />
             <geometry>
-                <mesh filename="package://nerf_launch_system/description/meshes/bottom_plate.stl" scale="0.001 0.001 0.001" />
+                <mesh filename="file://$(find nerf_launch_system)/description/meshes/bottom_plate.stl" scale="0.001 0.001 0.001" />
             </geometry>
         </visual>
@@ -42,5 +42,5 @@
             <origin xyz="0.09803428669398517 -4.3732793080548534e-05 -0.013700000763976723" rpy="1.5703501879750486 -1.5707963267948937 0" />
             <geometry>
-                <mesh filename="package://nerf_launch_system/description/meshes/motor_bracket.stl" scale="0.001 0.001 0.001" />
+                <mesh filename="file://$(find nerf_launch_system)/description/meshes/motor_bracket.stl" scale="0.001 0.001 0.001" />
             </geometry>
         </visual>
@@ -55,5 +55,5 @@
             <origin xyz="0.009991696360929777 -0.1260585761325394 0.08876880466816899" rpy="-3.141146514736195 1.079162159671481e-15 3.1415267664655997" />
             <geometry>
-                <mesh filename="package://nerf_launch_system/description/meshes/magazin.stl" scale="0.001 0.001 0.001" />
+                <mesh filename="file://$(find nerf_launch_system)/description/meshes/magazin.stl" scale="0.001 0.001 0.001" />
             </geometry>
         </visual>
@@ -68,5 +68,5 @@
             <origin xyz="-1.73567760164417e-09 3.029328534687181e-09 -1.3556827271887785e-09" rpy="-1.5707188555909968 0.00043936100150414944 1.7453951561374372" />
             <geometry>
-                <mesh filename="package://nerf_launch_system/description/meshes/motor_right.stl" scale="0.001 0.001 0.001" />
+                <mesh filename="file://$(find nerf_launch_system)/description/meshes/motor_right.stl" scale="0.001 0.001 0.001" />
             </geometry>
         </visual>
@@ -81,5 +81,5 @@
             <origin xyz="-1.8333526696778791e-09 -2.050084864091417e-09 -1.355682762715915e-09" rpy="-1.5711117946140916 0.00031546780349864484 0.7854640007616747" />
             <geometry>
-                <mesh filename="package://nerf_launch_system/description/meshes/motor_left.stl" scale="0.001 0.001 0.001" />
+                <mesh filename="file://$(find nerf_launch_system)/description/meshes/motor_left.stl" scale="0.001 0.001 0.001" />
             </geometry>
         </visual>
@@ -94,5 +94,5 @@
             <origin xyz="0.004998394584003245 0.024345667304006825 -0.010460860261822842" rpy="1.570796326794895 -0.0004461388535984491 -1.5707304396707022" />
             <geometry>
-                <mesh filename="package://nerf_launch_system/description/meshes/Servo_dart_pusher.stl" scale="0.001 0.001 0.001" />
+                <mesh filename="file://$(find nerf_launch_system)/description/meshes/Servo_dart_pusher.stl" scale="0.001 0.001 0.001" />
             </geometry>
         </visual>
@@ -107,5 +107,5 @@
             <origin xyz="-0.0631325544432252 0.01313155884148008 -0.0631300993428637" rpy="-1.570165432787083 0.7853321767598774 -3.1411465441724866" />
             <geometry>
-                <mesh filename="package://nerf_launch_system/description/meshes/flywheel_left.stl" scale="0.001 0.001 0.001" />
+                <mesh filename="file://$(find nerf_launch_system)/description/meshes/flywheel_left.stl" scale="0.001 0.001 0.001" />
             </geometry>
         </visual>
@@ -120,5 +120,5 @@
             <origin xyz="-0.01550858803514851 0.013120498025483157 -0.08792554788989197" rpy="-1.568228080674074 1.3961969502773832 -3.139063424976714" />
             <geometry>
-                <mesh filename="package://nerf_launch_system/description/meshes/flywheel_right.stl" scale="0.001 0.001 0.001" />
+                <mesh filename="file://$(find nerf_launch_system)/description/meshes/flywheel_right.stl" scale="0.001 0.001 0.001" />
             </geometry>
         </visual>
@@ -133,5 +133,5 @@
             <origin xyz="5.0358234648939514e-09 -0.0031999983978120905 1.4265863324780527e-06" rpy="-1.5712424656484945 6.588712419531712e-05 9.66531786022265e-16" />
             <geometry>
-                <mesh filename="package://nerf_launch_system/description/meshes/pusher_servo_part.stl" scale="0.001 0.001 0.001" />
+                <mesh filename="file://$(find nerf_launch_system)/description/meshes/pusher_servo_part.stl" scale="0.001 0.001 0.001" />
             </geometry>
         </visual>
@@ -146,5 +146,5 @@
             <origin xyz="0.0089380699537615 -0.0803571481976858 -0.002142981347950717" rpy="-0.000446138853596889 -1.0791087584284575e-15 -6.58871241935617e-05" />
             <geometry>
-                <mesh filename="package://nerf_launch_system/description/meshes/Turret.stl" scale="0.001 0.001 0.001" />
+                <mesh filename="file://$(find nerf_launch_system)/description/meshes/Turret.stl" scale="0.001 0.001 0.001" />
             </geometry>
         </visual>
@@ -159,5 +159,5 @@
             <origin xyz="0.004000004389203955 -0.08928319312789187 0.01647600710867764" rpy="0.029400113955168578 -8.659366307345483e-14 -3.141592653583827" />
             <geometry>
-                <mesh filename="package://nerf_launch_system/description/meshes/Servoarm-v1.stl" scale="0.001 0.001 0.001" />
+                <mesh filename="file://$(find nerf_launch_system)/description/meshes/Servoarm-v1.stl" scale="0.001 0.001 0.001" />
             </geometry>
         </visual>
@@ -172,5 +172,5 @@
             <origin xyz="0.032232880187464355 0.10890697936911703 -0.024499995611303272" rpy="-8.077935669498046e-28 7.226432496549954e-26 1.570796326794921" />
             <geometry>
-                <mesh filename="package://nerf_launch_system/description/meshes/Nerf-Dart-Launcher_Servo-MG-v1.stl" scale="0.001 0.001 0.001" />
+                <mesh filename="file://$(find nerf_launch_system)/description/meshes/Nerf-Dart-Launcher_Servo-MG-v1.stl" scale="0.001 0.001 0.001" />
             </geometry>
         </visual>
@@ -181,6 +181,5 @@
         <child link="motor_bracket" />
         <axis xyz="1.1287570791617654e-07 2.227474133869779e-15 1.0000000021779938" />
-        <!-- <limit lower="5.23" upper="6.28" effort="1.0" velocity="5.0" /> -->
-        <limit lower="-0.52" upper="0.52" effort="1.0" velocity="5.0" />
+        <limit lower="5.23" upper="6.28" effort="1.0" velocity="5.0" />
         <dynamics damping="10.0" friction="5.0"/>
     </joint>
@@ -226,5 +225,6 @@
         <axis xyz="-2.7546953265439552e-21 1.0 -0.000446" />
         <limit effort="0.1" velocity="20.0"/>
-        <dynamics damping="0.0" friction="0.0"/>
+        <!-- <dynamics damping="0.0" friction="0.0"/> -->
+        <dynamics damping="15.0" friction="8.0"/>
     </joint>
     <joint name="bottom_plate_servo_fix_bottom_plate" type="fixed">

File: src/nerf_launch_system/description/urdf/launcher_gazebo_classic.urdf.xacro (robot description, xacro)
@@ -13,4 +13,5 @@
         <limit lower="0" upper="1" effort="1" velocity="1"/>
         <axis xyz="0 0 1"/>
+        <dynamics damping="20.0" friction="10.0"/>
     </joint>
     <link name="bottom_plate">
@@ -23,5 +24,5 @@
             <origin xyz="0.0 0.0 0.0" rpy="0.0 0.0 0.0" />
             <geometry>
-                <mesh filename="package://nerf_launch_system/description/meshes/bottom_plate.stl" scale="0.001 0.001 0.001" />
+                <mesh filename="file://$(find nerf_launch_system)/description/meshes/bottom_plate.stl" scale="0.001 0.001 0.001" />
             </geometry>
         </visual>
@@ -42,5 +43,5 @@
             <origin xyz="0.09803428669398517 -4.3732793080548534e-05 -0.013700000763976723" rpy="1.5703501879750486 -1.5707963267948937 0" />
             <geometry>
-                <mesh filename="package://nerf_launch_system/description/meshes/motor_bracket.stl" scale="0.001 0.001 0.001" />
+                <mesh filename="file://$(find nerf_launch_system)/description/meshes/motor_bracket.stl" scale="0.001 0.001 0.001" />
             </geometry>
         </visual>
@@ -55,5 +56,5 @@
             <origin xyz="0.009991696360929777 -0.1260585761325394 0.08876880466816899" rpy="-3.141146514736195 1.079162159671481e-15 3.1415267664655997" />
             <geometry>
-                <mesh filename="package://nerf_launch_system/description/meshes/magazin.stl" scale="0.001 0.001 0.001" />
+                <mesh filename="file://$(find nerf_launch_system)/description/meshes/magazin.stl" scale="0.001 0.001 0.001" />
             </geometry>
         </visual>
@@ -68,5 +69,5 @@
             <origin xyz="-1.73567760164417e-09 3.029328534687181e-09 -1.3556827271887785e-09" rpy="-1.5707188555909968 0.00043936100150414944 1.7453951561374372" />
             <geometry>
-                <mesh filename="package://nerf_launch_system/description/meshes/motor_right.stl" scale="0.001 0.001 0.001" />
+                <mesh filename="file://$(find nerf_launch_system)/description/meshes/motor_right.stl" scale="0.001 0.001 0.001" />
             </geometry>
         </visual>
@@ -81,5 +82,5 @@
             <origin xyz="-1.8333526696778791e-09 -2.050084864091417e-09 -1.355682762715915e-09" rpy="-1.5711117946140916 0.00031546780349864484 0.7854640007616747" />
             <geometry>
-                <mesh filename="package://nerf_launch_system/description/meshes/motor_left.stl" scale="0.001 0.001 0.001" />
+                <mesh filename="file://$(find nerf_launch_system)/description/meshes/motor_left.stl" scale="0.001 0.001 0.001" />
             </geometry>
         </visual>
@@ -94,5 +95,5 @@
             <origin xyz="0.004998394584003245 0.024345667304006825 -0.010460860261822842" rpy="1.570796326794895 -0.0004461388535984491 -1.5707304396707022" />
             <geometry>
-                <mesh filename="package://nerf_launch_system/description/meshes/Servo_dart_pusher.stl" scale="0.001 0.001 0.001" />
+                <mesh filename="file://$(find nerf_launch_system)/description/meshes/Servo_dart_pusher.stl" scale="0.001 0.001 0.001" />
             </geometry>
         </visual>
@@ -107,5 +108,5 @@
             <origin xyz="-0.0631325544432252 0.01313155884148008 -0.0631300993428637" rpy="-1.570165432787083 0.7853321767598774 -3.1411465441724866" />
             <geometry>
-                <mesh filename="package://nerf_launch_system/description/meshes/flywheel_left.stl" scale="0.001 0.001 0.001" />
+                <mesh filename="file://$(find nerf_launch_system)/description/meshes/flywheel_left.stl" scale="0.001 0.001 0.001" />
             </geometry>
         </visual>
@@ -120,5 +121,5 @@
             <origin xyz="-0.01550858803514851 0.013120498025483157 -0.08792554788989197" rpy="-1.568228080674074 1.3961969502773832 -3.139063424976714" />
             <geometry>
-                <mesh filename="package://nerf_launch_system/description/meshes/flywheel_right.stl" scale="0.001 0.001 0.001" />
+                <mesh filename="file://$(find nerf_launch_system)/description/meshes/flywheel_right.stl" scale="0.001 0.001 0.001" />
             </geometry>
         </visual>
@@ -133,5 +134,5 @@
             <origin xyz="5.0358234648939514e-09 -0.0031999983978120905 1.4265863324780527e-06" rpy="-1.5712424656484945 6.588712419531712e-05 9.66531786022265e-16" />
             <geometry>
-                <mesh filename="package://nerf_launch_system/description/meshes/pusher_servo_part.stl" scale="0.001 0.001 0.001" />
+                <mesh filename="file://$(find nerf_launch_system)/description/meshes/pusher_servo_part.stl" scale="0.001 0.001 0.001" />
             </geometry>
         </visual>
@@ -146,5 +147,5 @@
             <origin xyz="0.0089380699537615 -0.0803571481976858 -0.002142981347950717" rpy="-0.000446138853596889 -1.0791087584284575e-15 -6.58871241935617e-05" />
             <geometry>
-                <mesh filename="package://nerf_launch_system/description/meshes/Turret.stl" scale="0.001 0.001 0.001" />
+                <mesh filename="file://$(find nerf_launch_system)/description/meshes/Turret.stl" scale="0.001 0.001 0.001" />
             </geometry>
         </visual>
@@ -159,5 +160,5 @@
             <origin xyz="0.004000004389203955 -0.08928319312789187 0.01647600710867764" rpy="0.029400113955168578 -8.659366307345483e-14 -3.141592653583827" />
             <geometry>
-                <mesh filename="package://nerf_launch_system/description/meshes/Servoarm-v1.stl" scale="0.001 0.001 0.001" />
+                <mesh filename="file://$(find nerf_launch_system)/description/meshes/Servoarm-v1.stl" scale="0.001 0.001 0.001" />
             </geometry>
         </visual>
@@ -172,5 +173,5 @@
             <origin xyz="0.032232880187464355 0.10890697936911703 -0.024499995611303272" rpy="-8.077935669498046e-28 7.226432496549954e-26 1.570796326794921" />
             <geometry>
-                <mesh filename="package://nerf_launch_system/description/meshes/Nerf-Dart-Launcher_Servo-MG-v1.stl" scale="0.001 0.001 0.001" />
+                <mesh filename="file://$(find nerf_launch_system)/description/meshes/Nerf-Dart-Launcher_Servo-MG-v1.stl" scale="0.001 0.001 0.001" />
             </geometry>
         </visual>
@@ -226,5 +227,5 @@
         <axis xyz="-2.7546953265439552e-21 1.0 -0.000446" />
         <limit effort="0.1" velocity="20.0"/>
-        <dynamics damping="0.0" friction="0.0"/>
+        <dynamics damping="15.0" friction="8.0"/>
     </joint>
     <joint name="bottom_plate_servo_fix_bottom_plate" type="fixed">

Commit message: ai implementation maybe not working

File: src/gubot_one_description/description/camera.xacro (robot description, xacro)
@@ -27,4 +27,6 @@
     </joint>
     <link name="camera_link_optical"></link>
+    <xacro:arg name="use_gazebo_classic" default="false"/>
+    <!-- VORHER:
     <gazebo reference="camera_link">
         <material>Gazebo/Black</material>
@@ -48,3 +50,53 @@
             </sensor>
     </gazebo>
+    -->
+    <gazebo reference="camera_link">
+        <material>Gazebo/Black</material>
+        <!-- Ignition / Harmonic -->
+        <xacro:unless value="$(arg use_gazebo_classic)">
+            <sensor name="camera" type="camera">
+                <pose>0 0 0 0 0 0</pose>
+                <visualize>false</visualize>
+                <update_rate>10</update_rate>
+                <camera>
+                    <horizontal_fov>1.089</horizontal_fov>
+                    <image>
+                        <format>R8G8B8</format>
+                        <width>640</width>
+                        <height>480</height>
+                    </image>
+                    <clip>
+                        <near>0.05</near>
+                        <far>8.0</far>
+                    </clip>
+                </camera>
+                <topic>camera/image_raw</topic>
+            </sensor>
+        </xacro:unless>
+        <!-- Gazebo Classic -->
+        <xacro:if value="$(arg use_gazebo_classic)">
+            <sensor type="camera" name="camera">
+                <update_rate>10</update_rate>
+                <camera>
+                    <horizontal_fov>1.089</horizontal_fov>
+                    <image>
+                        <format>R8G8B8</format>
+                        <width>640</width>
+                        <height>480</height>
+                    </image>
+                    <clip>
+                        <near>0.05</near>
+                        <far>8.0</far>
+                    </clip>
+                </camera>
+                <plugin name="camera_controller" filename="libgazebo_ros_camera.so">
+                    <ros>
+                        <remapping>image_raw:=camera/image_raw</remapping>
+                        <remapping>camera_info:=camera/camera_info</remapping>
+                    </ros>
+                    <frame_name>camera_link_optical</frame_name>
+                </plugin>
+            </sensor>
+        </xacro:if>
+    </gazebo>
 </robot>

File: src/gubot_one_description/description/robot.urdf.xacro (robot description, xacro)
@@ -2,4 +2,5 @@
 <robot xmlns:xacro="http://www.ros.org/wiki/xacro"  name="robot">
     <xacro:arg name="use_ros2_control" default="true"/>
+    <xacro:arg name="use_gazebo_classic" default="false"/>
     <xacro:arg name="sim_mode" default="false"/>
     <xacro:arg name="integrated_mode" default="true"/>

File: src/gubot_one_description/description/robot_classic.urdf.xacro (robot description, xacro)
@@ -2,8 +2,14 @@
 <robot xmlns:xacro="http://www.ros.org/wiki/xacro" name="robot">
     <xacro:arg name="use_gazebo_classic" default="true"/>
+    <xacro:arg name="use_nerf_hardware" default="true"/>
     <xacro:include filename="robot_core_classic.xacro" />
     <xacro:include filename="gz_classic_ros2_control_sim.xacro" />
     <xacro:arg name="integrated_mode" default="true"/>
+    <!-- VORHER:
     <xacro:include filename="nerf_launcher_classic.xacro" />
+    -->
+    <xacro:if value="$(arg use_nerf_hardware)">
+        <xacro:include filename="nerf_launcher_classic.xacro" />
+    </xacro:if>
     <xacro:include filename="camera.xacro" />
     <xacro:include filename="face.xacro" />
