Commit message: ai implementation maybe not working

File: src/gubot_one_description/description/robot_core_classic.xacro (robot description, xacro)
@@ -63,5 +63,5 @@
             </geometry>
         </collision>
-        <xacro:inertial_box mass="0.5" x="${chassis_length}" y="${chassis_width}" z="${chassis_height}">
+        <xacro:inertial_box mass="${chassis_mass}" x="${chassis_length}" y="${chassis_width}" z="${chassis_height}">
             <origin xyz="${chassis_length/2} 0 ${chassis_height/2}" rpy="0 0 0"/>
         </xacro:inertial_box>
@@ -167,5 +167,5 @@
         <origin xyz="0 ${wheel_offset_y} 0" rpy="-${pi/2} 0 0" />
         <axis xyz="0 0 1"/>
-        <dynamics damping="20.0" friction="8.0"/>
+        <dynamics damping="0.05" friction="0.01"/>
     </joint>
     <link name="left_wheel">
@@ -197,5 +197,5 @@
         <origin xyz="0 ${-wheel_offset_y} 0" rpy="${pi/2} 0 0" />
         <axis xyz="0 0 -1"/>
-        <dynamics damping="20.0" friction="8.0"/>
+        <dynamics damping="0.05" friction="0.01"/>
     </joint>
     <link name="right_wheel">
