Commit message: chore: ALT-Kommentare entfernen, veraltete Doku-Befehle korrigiert
Entfernt historische "ALT:"-Marker (auskommentierter alter Code,
Vorher/Nachher-Notizen) aus Launch-Dateien, URDF/xacro, Configs,
Firmware und Tests — Git-Historie bewahrt den Kontext bereits.
Nicht-obviouse Bugfix-Begruendungen wurden als normaler Kommentar
ohne ALT-Label erhalten.

README.md und docs/Kommandos-Datei korrigiert: gubot_one -> gubot_bringup
(Paket wurde aufgeteilt), nerf_standalone -> nerf_launch_system,
undeklariertes nerf_port-Argument entfernt.

File: src/gubot_description/urdf/gubot_one_geometry.xacro (robot description, xacro)
@@ -9,5 +9,4 @@
     <xacro:property name="wheel_thickness" value="0.026"/>
     <xacro:property name="wheel_mass" value="0.4"/>
-    <!-- ALT (Asymmetrisch): <xacro:property name="wheel_offset_x" value="0.226"/> -->
     <xacro:property name="wheel_offset_x" value="0.113"/>
     <xacro:property name="wheel_offset_y" value="0.1485"/>
@@ -35,16 +34,5 @@
     <link name="base_link">
     </link>
-    <!-- ALT: base_footprint — nicht in rosbot_xl Referenz, auskommentiert -->
-    <!-- <joint name="base_footprint_joint" type="fixed"> -->
-    <!--     <parent link="base_link"/> -->
-    <!--     <child link="base_footprint"/> -->
-    <!--     <origin xyz="0 0 0" rpy="0 0 0"/> -->
-    <!-- </joint> -->
-    <!-- <link name="base_footprint"/> -->
     <!-- BODY_LINK (wie Referenz rosbot_xl: base_link -> body_link mit Z=wheel_radius Offset) -->
-    <!-- ALT: Z=0.0 — Chassis saß auf dem Boden, Räder sanken durch den Boden -->
-    <!-- <joint name="base_to_body_joint" type="fixed"> -->
-    <!--     <origin xyz="0.0 0.0 0.0" rpy="0.0 0.0 0.0"/> -->
-    <!-- </joint> -->
     <joint name="base_to_body_joint" type="fixed">
         <parent link="base_link"/>
@@ -75,5 +63,4 @@
     <!-- IMU LINK -->
     <joint name="imu_joint" type="fixed">
-        <!-- ALT: <parent link="chassis"/> -->
         <parent link="body_link"/>
         <child link="imu_link"/>
@@ -102,5 +89,4 @@
         <material>Gazebo/Black</material>
         <!-- IMU Sensor — Ignition Fortress Konfiguration (wie Referenz rosbot_xl) -->
-        <!-- ALT: Branching via use_gazebo_classic Arg + topic=imu_sensor/imu_data -->
         <sensor name="imu_sensor" type="imu">
             <always_on>true</always_on>
@@ -125,7 +111,4 @@
     </gazebo>
     <!-- FRONT LEFT WHEEL (wie Referenz: fl_wheel_joint, parent=body_link, axis=Y, RPY=0) -->
-    <!-- ALT: front_left_wheel_joint / left_wheel — umbenannt auf Referenz-Schema fl/fr/rl/rr -->
-    <!-- <joint name="front_left_wheel_joint" type="continuous"> -->
-    <!-- <link name="left_wheel"> -->
     <joint name="fl_wheel_joint" type="continuous">
         <parent link="body_link"/>
@@ -165,7 +148,4 @@
     </gazebo>
     <!-- FRONT RIGHT WHEEL (wie Referenz: fr_wheel_joint, parent=body_link, axis=Y, RPY=0) -->
-    <!-- ALT: front_right_wheel_joint / right_wheel — umbenannt auf Referenz-Schema fl/fr/rl/rr -->
-    <!-- <joint name="front_right_wheel_joint" type="continuous"> -->
-    <!-- <link name="right_wheel"> -->
     <joint name="fr_wheel_joint" type="continuous">
         <parent link="body_link"/>
@@ -206,7 +186,4 @@
     <!-- REAR WHEELS (wie Referenz: rl/rr_wheel_joint, parent=body_link, axis=Y, RPY=0) -->
     <!-- REAR LEFT WHEEL -->
-    <!-- ALT: rear_left_wheel_joint / rear_left_wheel — umbenannt auf Referenz-Schema -->
-    <!-- <joint name="rear_left_wheel_joint" type="continuous"> -->
-    <!-- <link name="rear_left_wheel"> -->
     <joint name="rl_wheel_joint" type="continuous">
         <parent link="body_link"/>
@@ -246,7 +223,4 @@
     </gazebo>
     <!-- REAR RIGHT WHEEL -->
-    <!-- ALT: rear_right_wheel_joint / rear_right_wheel — umbenannt auf Referenz-Schema -->
-    <!-- <joint name="rear_right_wheel_joint" type="continuous"> -->
-    <!-- <link name="rear_right_wheel"> -->
     <joint name="rr_wheel_joint" type="continuous">
         <parent link="body_link"/>

File: src/gubot_description/urdf/nerf_launch_system.xacro (robot description, xacro)
@@ -4,5 +4,4 @@
     <xacro:include filename="$(find nerf_launch_system)/description/urdf/nerf_launcher.urdf.xacro" />
     <joint name="nerf_mount_joint" type="fixed">
-  <!-- ALT: <parent link="chassis"/> -->
         <parent link="body_link"/>
         <child link="bottom_plate"/>

File: src/gubot_description/urdf/ros2_control_gazebo_ign_fortress.xacro (robot description, xacro)
@@ -12,16 +12,11 @@
     -->
     <!-- NEW: controller config path injected by load_urdf.launch.py at runtime -->
-    <!-- ALT: Hard-coded $(find gubot_one)/controller/config/controllers.yaml -->
     <xacro:arg name="controller_config"
         default="$(find gubot_controller)/config/controllers.yaml"/>
     <ros2_control name="GubotIgnitionSystem" type="system">
         <hardware>
-            <!-- ALT: ign_ros2_control/IgnitionSystem (Ignition Fortress plugin name) -->
             <plugin>gz_ros2_control/GazeboSimSystem</plugin>
-            <!-- ALT: position_proportional_gain — wird von GazeboSimSystem nicht unterstützt -->
-            <!-- <param name="position_proportional_gain">20.0</param> -->
         </hardware>
         <!-- Gelenkbezeichnungen: fl/fr/rl/rr_wheel_joint (Referenz rosbot_xl-Schema) -->
-        <!-- ALT: front_left/front_right/rear_left/rear_right_wheel_joint -->
         <joint name="fl_wheel_joint">
             <command_interface name="velocity">
@@ -73,6 +68,4 @@
         </joint>
         <!-- Nerf-Joints: NUR wenn use_nerf_hardware=true, sonst existieren diese Joints nicht in der URDF -->
-        <!-- ALT: value="${'$(arg use_nerf_hardware)' == 'true'}" - fragile String-Vergleich
-             NEU: Standard xacro:arg Substitution -->
         <xacro:if value="$(arg use_nerf_hardware)">
             <joint name="trigger_joint">
@@ -114,9 +107,6 @@
     <gazebo>
         <!-- Referenz: common/gazebo.urdf.xacro macro "controller" -->
-        <!-- ALT: gz_ros2_control::GazeboSimROS2ControlPlugin (Gazebo Garden/Harmonic) -->
-        <!-- <plugin filename="gz_ros2_control-system" name="gz_ros2_control::GazeboSimROS2ControlPlugin"> -->
         <plugin filename="ign_ros2_control-system" name="ign_ros2_control::IgnitionROS2ControlPlugin">
             <controller_manager_name>controller_manager</controller_manager_name>
-            <!-- ALT: Hard-coded Pfad $(find gubot_one)/controller/config/controllers.yaml -->
             <parameters>$(arg controller_config)</parameters>
             <ros>

File: src/gubot_description/urdf/sensor_camera.xacro (robot description, xacro)
@@ -2,5 +2,4 @@
 <robot xmlns:xacro="http://www.ros.org/wiki/xacro" >
     <joint name="camera_joint" type="fixed">
-        <!-- ALT: <parent link="chassis"/> -->
         <parent link="body_link"/>
         <child link="camera_link"/>
@@ -54,14 +53,7 @@
             <!--         <frame_name>camera_link_optical</frame_name> -->
             <!--     </plugin> -->
-            <!-- </xacro:if> -->
-            <!-- <xacro:unless value="$(arg use_gazebo_classic)"> -->
-            <!--     <topic>camera/image_raw</topic> -->
-            <!--     <!- - NEU: Expliziter Frame-ID damit Ignition nicht den auto-generierten -->
-            <!--          Pfad 'gubot_one/base_link/camera' verwendet, sondern den TF-Frame -->
-            <!--          'camera_link_optical' der von robot_state_publisher veroeffentlicht wird. -->
-            <!--          ALT: kein ignition_frame_id -> Ignition nutzt 'modelname/linkname/sensorname' -->
-            <!--              -> RViz kann Frame nicht finden -> queue overflow -> Flackern - -> -->
-            <!--     <ignition_frame_id>camera_link_optical</ignition_frame_id> -->
-            <!-- </xacro:unless> -->
+            <!-- NEU: Expliziter Frame-ID damit Ignition nicht den auto-generierten
+                 Pfad 'gubot_one/base_link/camera' verwendet, sondern den TF-Frame
+                 'camera_link_optical' der von robot_state_publisher veroeffentlicht wird -->
             <topic>camera/image_raw</topic>
             <ignition_frame_id>camera_link_optical</ignition_frame_id>

File: src/gubot_description/urdf/sensor_depth_camera.xacro (robot description, xacro)
@@ -2,5 +2,4 @@
 <robot xmlns:xacro="http://www.ros.org/wiki/xacro" >
     <joint name="camera_joint" type="fixed">
-        <!-- ALT: <parent link="chassis"/> -->
         <parent link="body_link"/>
         <child link="camera_link"/>

File: src/gubot_description/urdf/sensor_lidar.xacro (robot description, xacro)
@@ -2,5 +2,4 @@
 <robot xmlns:xacro="http://www.ros.org/wiki/xacro" >
     <joint name="laser_joint" type="fixed">
-        <!-- ALT: <parent link="chassis"/> -->
         <parent link="body_link"/>
         <child link="laser_frame"/>

File: src/gubot_description/urdf/visual_face.xacro (robot description, xacro)
@@ -2,5 +2,4 @@
 <robot xmlns:xacro="http://www.ros.org/wiki/xacro" >
     <joint name="face_joint" type="fixed">
-        <!-- ALT: <parent link="chassis"/> -->
         <parent link="body_link"/>
         <child link="face_link"/>

File: src/nerf_launch_system/description/urdf/nerf_launcher.urdf.xacro (robot description, xacro)
@@ -168,6 +168,6 @@
         <child link="motor_bracket" />
         <!-- Achse invertiert: positiv = Launcher hoch (aus dem Körper heraus).
-             ALT: xyz="1.1e-07 2.2e-15 1.0" (CAD-Export) — positiv drehte den
-             Launcher NACH UNTEN in den Roboterkörper; das Init-Kommando
+             Der urspruengliche CAD-Export (xyz="1.1e-07 2.2e-15 1.0") drehte
+             den Launcher NACH UNTEN in den Roboterkoerper; das Init-Kommando
              "UP = +tilt_max" fuhr ihn damit genau falsch herum. Hardware ist
              deltabasiert (UP-Pulse bei steigendem Soll) und bleibt konsistent. -->
