Commit message: feat(gubot_description): Chassis- und Rad-Box durch Meshes ersetzt
Chassis-Visual (body_link) nutzt jetzt waffle_pi_base.stl (non-uniform
auf die Chassis-Box skaliert), die vier Raeder mecanum_a.dae/mecanum_b.dae
(100mm Aluminum-Mecanum-Rad, R/L) statt Box/Zylinder-Platzhalter.
Collision-Geometrie bleibt Box/Zylinder fuer performante Physik.

wheel_radius/wheel_thickness auf die reale Mesh-Groesse (0.05/0.05m)
angehoben (vorher 0.033/0.026m Platzhalter) und den kalibrierten
mecanum_drive_controller.wheel_radius in controllers.yaml + den
zugehoerigen Test synchron nachgezogen, damit Odometrie-Kinematik,
Visual und Collision konsistent bleiben.

Mesh-Referenzen nutzen file://$(find gubot_description)/... statt
package://, da Ignition Fortress package:// zu einem nicht aufloesbaren
model://-URI konvertiert.

Co-Authored-By: Claude Sonnet 5 <noreply@anthropic.com>

File: src/gubot_description/urdf/gubot_one_geometry.xacro (robot description, xacro)
@@ -6,6 +6,16 @@
     <xacro:property name="chassis_height" value="0.138"/>
     <xacro:property name="chassis_mass" value="3.5"/>
-    <xacro:property name="wheel_radius" value="0.033"/>
-    <xacro:property name="wheel_thickness" value="0.026"/>
+    <!-- waffle_pi_base.stl Rohmasse in Metern (STL-Einheit ist mm, Faktor 0.001);
+         chassis_mesh_scale_* streckt das Mesh non-uniform auf die Chassis-Box. -->
+    <xacro:property name="chassis_mesh_native_length" value="0.274046234"/>
+    <xacro:property name="chassis_mesh_native_width" value="0.278799988"/>
+    <xacro:property name="chassis_mesh_native_height" value="0.118922503"/>
+    <xacro:property name="chassis_mesh_scale_x" value="${0.001 * chassis_length / chassis_mesh_native_length}"/>
+    <xacro:property name="chassis_mesh_scale_y" value="${0.001 * chassis_width / chassis_mesh_native_width}"/>
+    <xacro:property name="chassis_mesh_scale_z" value="${0.001 * chassis_height / chassis_mesh_native_height}"/>
+    <!-- 100mm Aluminum-Mecanum-Rad (mecanum_a.dae=R, mecanum_b.dae=L); ersetzt den
+         urspruenglichen 33mm-Platzhalter, echte Raeder sind die 100mm-Mecanum-Raeder. -->
+    <xacro:property name="wheel_radius" value="0.05"/>
+    <xacro:property name="wheel_thickness" value="0.05"/>
     <xacro:property name="wheel_mass" value="0.4"/>
     <xacro:property name="wheel_offset_x" value="0.113"/>
@@ -42,7 +52,8 @@
     <link name="body_link">
         <visual>
-            <origin xyz="0.0 0.0 ${chassis_height/2}"/>
-            <geometry>
-                <box size="${chassis_length} ${chassis_width} ${chassis_height}"/>
+            <origin xyz="0.0 0.0 0.0" rpy="0.0 0.0 0.0"/>
+            <geometry>
+                <mesh filename="file://$(find gubot_description)/meshes/bases/waffle_pi_base.stl"
+                      scale="${chassis_mesh_scale_x} ${chassis_mesh_scale_y} ${chassis_mesh_scale_z}"/>
             </geometry>
             <material name="orange"/>
@@ -122,8 +133,7 @@
         <visual>
             <geometry>
-                <cylinder radius="${wheel_radius}" length="${wheel_thickness}"/>
-            </geometry>
-            <origin xyz="0.0 0.0 0.0" rpy="${pi/2} 0.0 0.0"/>
-            <material name="blue"/>
+                <mesh filename="file://$(find gubot_description)/meshes/wheels/mecanum_b.dae"/>
+            </geometry>
+            <origin xyz="0.0 0.0 0.0" rpy="0.0 0.0 0.0"/>
         </visual>
         <collision>
@@ -159,8 +169,7 @@
         <visual>
             <geometry>
-                <cylinder radius="${wheel_radius}" length="${wheel_thickness}"/>
-            </geometry>
-            <origin xyz="0.0 0.0 0.0" rpy="${pi/2} 0.0 0.0"/>
-            <material name="blue"/>
+                <mesh filename="file://$(find gubot_description)/meshes/wheels/mecanum_a.dae"/>
+            </geometry>
+            <origin xyz="0.0 0.0 0.0" rpy="0.0 0.0 0.0"/>
         </visual>
         <collision>
@@ -197,8 +206,7 @@
         <visual>
             <geometry>
-                <cylinder radius="${wheel_radius}" length="${wheel_thickness}"/>
-            </geometry>
-            <origin xyz="0.0 0.0 0.0" rpy="${pi/2} 0.0 0.0"/>
-            <material name="blue"/>
+                <mesh filename="file://$(find gubot_description)/meshes/wheels/mecanum_b.dae"/>
+            </geometry>
+            <origin xyz="0.0 0.0 0.0" rpy="0.0 0.0 0.0"/>
         </visual>
         <collision>
@@ -234,8 +242,7 @@
         <visual>
             <geometry>
-                <cylinder radius="${wheel_radius}" length="${wheel_thickness}"/>
-            </geometry>
-            <origin xyz="0.0 0.0 0.0" rpy="${pi/2} 0.0 0.0"/>
-            <material name="blue"/>
+                <mesh filename="file://$(find gubot_description)/meshes/wheels/mecanum_a.dae"/>
+            </geometry>
+            <origin xyz="0.0 0.0 0.0" rpy="0.0 0.0 0.0"/>
         </visual>
         <collision>
