Commit message: refactor(description): modulare xacros + shared dimensions yaml + urdf tests
Co-Authored-By: Claude Fable 5 <noreply@anthropic.com>

File: src/gubot_description/urdf/gubot_one_geometry.xacro (robot description, xacro)
@@ -1,44 +1,10 @@
 <?xml version="1.0"?>
-<robot xmlns:xacro="http://www.ros.org/wiki/xacro" xmlns:ignition="http://ignitionrobotics.org/schema">
+<robot xmlns:xacro="http://www.ros.org/wiki/xacro">
+    <!-- Reine Geometrie (Links/Joints/Inertials) — keine Gazebo-Tags.
+         Eigenschaften/Materialien: properties.xacro (via gubot_one_main).
+         Sim-spezifisches (IMU-Sensor, Rad-Reibung, Gazebo-Materialien):
+         gazebo_sim.xacro. -->
     <xacro:include filename="inertial_macros.xacro"/>
-    <xacro:property name="chassis_length" value="0.335"/>
-    <xacro:property name="chassis_width" value="0.265"/>
-    <xacro:property name="chassis_height" value="0.138"/>
-    <xacro:property name="chassis_mass" value="3.5"/>
-    <!-- waffle_pi_base.stl Rohmasse in Metern (STL-Einheit ist mm, Faktor 0.001);
-         chassis_mesh_scale_* streckt das Mesh non-uniform auf die Chassis-Box. -->
-    <xacro:property name="chassis_mesh_native_length" value="0.274046234"/>
-    <xacro:property name="chassis_mesh_native_width" value="0.278799988"/>
-    <xacro:property name="chassis_mesh_native_height" value="0.118922503"/>
-    <xacro:property name="chassis_mesh_scale_x" value="${0.001 * chassis_length / chassis_mesh_native_length}"/>
-    <xacro:property name="chassis_mesh_scale_y" value="${0.001 * chassis_width / chassis_mesh_native_width}"/>
-    <xacro:property name="chassis_mesh_scale_z" value="${0.001 * chassis_height / chassis_mesh_native_height}"/>
-    <!-- 100mm Aluminum-Mecanum-Rad (mecanum_a.dae=R, mecanum_b.dae=L); ersetzt den
-         urspruenglichen 33mm-Platzhalter, echte Raeder sind die 100mm-Mecanum-Raeder. -->
-    <xacro:property name="wheel_radius" value="0.05"/>
-    <xacro:property name="wheel_thickness" value="0.05"/>
-    <xacro:property name="wheel_mass" value="0.4"/>
-    <xacro:property name="wheel_offset_x" value="0.113"/>
-    <xacro:property name="wheel_offset_y" value="0.1485"/>
-    <xacro:property name="wheel_offset_z" value="0.01"/>
-    <xacro:property name="caster_wheel_radius" value="0.01"/>
-    <xacro:property name="caster_wheel_mass" value="0.01"/>
-    <xacro:property name="caster_wheel_offset_x" value="0.075"/>
-    <xacro:property name="caster_wheel_offset_z" value="${wheel_offset_z - wheel_radius + caster_wheel_radius}"/>
-    <material name="white">
-        <color rgba="1 1 1 1" />
-    </material>
-    <material name="orange">
-        <color rgba="1 0.3 0.1 1"/>
-    </material>
-    <material name="blue">
-        <color rgba="0.2 0.2 1 1"/>
-    </material>
-    <material name="black">
-        <color rgba="0 0 0 1"/>
-    </material>
-    <material name="red">
-        <color rgba="1 0 0 1"/>
-    </material>
+    <xacro:include filename="mecanum_wheel.xacro"/>
     <!-- BASE LINK -->
     <link name="base_link">
@@ -69,7 +35,4 @@
         </xacro:inertial_box>
     </link>
-    <gazebo reference="body_link">
-        <material>Gazebo/Orange</material>
-    </gazebo>
     <!-- IMU LINK -->
     <joint name="imu_joint" type="fixed">
@@ -78,7 +41,4 @@
         <origin xyz="0 0 0.05" rpy="0 0 0"/>
     </joint>
-    <gazebo reference="imu_joint">
-        <disableFixedJointLumping>true</disableFixedJointLumping>
-    </gazebo>
     <link name="imu_link">
         <visual>
@@ -97,172 +57,8 @@
         </xacro:inertial_box>
     </link>
-    <gazebo reference="imu_link">
-        <material>Gazebo/Black</material>
-        <!-- IMU Sensor — Ignition Fortress Konfiguration (wie Referenz rosbot_xl) -->
-        <sensor name="imu_sensor" type="imu">
-            <always_on>true</always_on>
-            <update_rate>25</update_rate>
-            <visualize>false</visualize>
-            <topic>imu/data_raw</topic>
-            <ignition_frame_id>imu_link</ignition_frame_id>
-            <enable_metrics>false</enable_metrics>
-            <imu>
-                <angular_velocity>
-                    <x><noise type="gaussian"><mean>0.0</mean><stddev>5.24e-3</stddev><bias_mean>2.0e-3</bias_mean><bias_stddev>0.0</bias_stddev></noise></x>
-                    <y><noise type="gaussian"><mean>0.0</mean><stddev>5.24e-3</stddev><bias_mean>2.0e-3</bias_mean><bias_stddev>0.0</bias_stddev></noise></y>
-                    <z><noise type="gaussian"><mean>0.0</mean><stddev>5.24e-3</stddev><bias_mean>2.0e-3</bias_mean><bias_stddev>0.0</bias_stddev></noise></z>
-                </angular_velocity>
-                <linear_acceleration>
-                    <x><noise type="gaussian"><mean>0.0</mean><stddev>1.86e-3</stddev><bias_mean>1.0e-3</bias_mean><bias_stddev>0.0</bias_stddev></noise></x>
-                    <y><noise type="gaussian"><mean>0.0</mean><stddev>1.86e-3</stddev><bias_mean>1.0e-3</bias_mean><bias_stddev>0.0</bias_stddev></noise></y>
-                    <z><noise type="gaussian"><mean>0.0</mean><stddev>1.86e-3</stddev><bias_mean>1.0e-3</bias_mean><bias_stddev>0.0</bias_stddev></noise></z>
-                </linear_acceleration>
-            </imu>
-        </sensor>
-    </gazebo>
-    <!-- FRONT LEFT WHEEL (wie Referenz: fl_wheel_joint, parent=body_link, axis=Y, RPY=0) -->
-    <joint name="fl_wheel_joint" type="continuous">
-        <parent link="body_link"/>
-        <child link="fl_wheel_link"/>
-        <origin xyz="${wheel_offset_x} ${wheel_offset_y} 0.0" rpy="0.0 0.0 0.0"/>
-        <axis xyz="0.0 1.0 0.0"/>
-        <limit effort="1.5" velocity="30.0"/>
-        <dynamics damping="0.001" friction="0.001"/>
-    </joint>
-    <link name="fl_wheel_link">
-        <visual>
-            <geometry>
-                <mesh filename="file://$(find gubot_description)/meshes/wheels/mecanum_b.dae"/>
-            </geometry>
-            <origin xyz="0.0 0.0 0.0" rpy="0.0 0.0 0.0"/>
-        </visual>
-        <collision>
-            <geometry>
-                <cylinder radius="${wheel_radius}" length="${wheel_thickness}"/>
-            </geometry>
-            <origin xyz="0.0 0.0 0.0" rpy="${pi/2} 0.0 0.0"/>
-        </collision>
-        <xacro:inertial_cylinder mass="${wheel_mass}" length="${wheel_thickness}" radius="${wheel_radius}">
-            <origin xyz="0 0 0" rpy="0 0 0"/>
-        </xacro:inertial_cylinder>
-    </link>
-    <gazebo reference="fl_wheel_link">
-        <material>Gazebo/Blue</material>
-        <collision>
-            <surface><friction><ode>
-                <mu>0.8</mu><mu2>0.2</mu2>
-                <slip1>0.035</slip1><slip2>0.0</slip2>
-                <fdir1 ignition:expressed_in="base_link">1 -1 0</fdir1>
-            </ode></friction></surface>
-        </collision>
-    </gazebo>
-    <!-- FRONT RIGHT WHEEL (wie Referenz: fr_wheel_joint, parent=body_link, axis=Y, RPY=0) -->
-    <joint name="fr_wheel_joint" type="continuous">
-        <parent link="body_link"/>
-        <child link="fr_wheel_link"/>
-        <origin xyz="${wheel_offset_x} ${-wheel_offset_y} 0.0" rpy="0.0 0.0 0.0"/>
-        <axis xyz="0.0 1.0 0.0"/>
-        <limit effort="1.5" velocity="30.0"/>
-        <dynamics damping="0.001" friction="0.001"/>
-    </joint>
-    <link name="fr_wheel_link">
-        <visual>
-            <geometry>
-                <mesh filename="file://$(find gubot_description)/meshes/wheels/mecanum_a.dae"/>
-            </geometry>
-            <origin xyz="0.0 0.0 0.0" rpy="0.0 0.0 0.0"/>
-        </visual>
-        <collision>
-            <geometry>
-                <cylinder radius="${wheel_radius}" length="${wheel_thickness}"/>
-            </geometry>
-            <origin xyz="0.0 0.0 0.0" rpy="${pi/2} 0.0 0.0"/>
-        </collision>
-        <xacro:inertial_cylinder mass="${wheel_mass}" length="${wheel_thickness}" radius="${wheel_radius}">
-            <origin xyz="0 0 0" rpy="0 0 0"/>
-        </xacro:inertial_cylinder>
-    </link>
-    <gazebo reference="fr_wheel_link">
-        <material>Gazebo/Blue</material>
-        <collision>
-            <surface><friction><ode>
-                <mu>0.8</mu><mu2>0.2</mu2>
-                <slip1>0.035</slip1><slip2>0.0</slip2>
-                <fdir1 ignition:expressed_in="base_link">1 1 0</fdir1>
-            </ode></friction></surface>
-        </collision>
-    </gazebo>
-    <!-- REAR WHEELS (wie Referenz: rl/rr_wheel_joint, parent=body_link, axis=Y, RPY=0) -->
-    <!-- REAR LEFT WHEEL -->
-    <joint name="rl_wheel_joint" type="continuous">
-        <parent link="body_link"/>
-        <child link="rl_wheel_link"/>
-        <origin xyz="${-wheel_offset_x} ${wheel_offset_y} 0.0" rpy="0.0 0.0 0.0"/>
-        <axis xyz="0.0 1.0 0.0"/>
-        <limit effort="1.5" velocity="30.0"/>
-        <dynamics damping="0.001" friction="0.001"/>
-    </joint>
-    <link name="rl_wheel_link">
-        <visual>
-            <geometry>
-                <mesh filename="file://$(find gubot_description)/meshes/wheels/mecanum_b.dae"/>
-            </geometry>
-            <origin xyz="0.0 0.0 0.0" rpy="0.0 0.0 0.0"/>
-        </visual>
-        <collision>
-            <geometry>
-                <cylinder radius="${wheel_radius}" length="${wheel_thickness}"/>
-            </geometry>
-            <origin xyz="0.0 0.0 0.0" rpy="${pi/2} 0.0 0.0"/>
-        </collision>
-        <xacro:inertial_cylinder mass="${wheel_mass}" length="${wheel_thickness}" radius="${wheel_radius}">
-            <origin xyz="0 0 0" rpy="0 0 0"/>
-        </xacro:inertial_cylinder>
-    </link>
-    <gazebo reference="rl_wheel_link">
-        <material>Gazebo/Blue</material>
-        <collision>
-            <surface><friction><ode>
-                <mu>0.8</mu><mu2>0.2</mu2>
-                <slip1>0.035</slip1><slip2>0.0</slip2>
-                <fdir1 ignition:expressed_in="base_link">1 1 0</fdir1>
-            </ode></friction></surface>
-        </collision>
-    </gazebo>
-    <!-- REAR RIGHT WHEEL -->
-    <joint name="rr_wheel_joint" type="continuous">
-        <parent link="body_link"/>
-        <child link="rr_wheel_link"/>
-        <origin xyz="${-wheel_offset_x} ${-wheel_offset_y} 0.0" rpy="0.0 0.0 0.0"/>
-        <axis xyz="0.0 1.0 0.0"/>
-        <limit effort="1.5" velocity="30.0"/>
-        <dynamics damping="0.001" friction="0.001"/>
-    </joint>
-    <link name="rr_wheel_link">
-        <visual>
-            <geometry>
-                <mesh filename="file://$(find gubot_description)/meshes/wheels/mecanum_a.dae"/>
-            </geometry>
-            <origin xyz="0.0 0.0 0.0" rpy="0.0 0.0 0.0"/>
-        </visual>
-        <collision>
-            <geometry>
-                <cylinder radius="${wheel_radius}" length="${wheel_thickness}"/>
-            </geometry>
-            <origin xyz="0.0 0.0 0.0" rpy="${pi/2} 0.0 0.0"/>
-        </collision>
-        <xacro:inertial_cylinder mass="${wheel_mass}" length="${wheel_thickness}" radius="${wheel_radius}">
-            <origin xyz="0 0 0" rpy="0 0 0"/>
-        </xacro:inertial_cylinder>
-    </link>
-    <gazebo reference="rr_wheel_link">
-        <material>Gazebo/Blue</material>
-        <collision>
-            <surface><friction><ode>
-                <mu>0.8</mu><mu2>0.2</mu2>
-                <slip1>0.035</slip1><slip2>0.0</slip2>
-                <fdir1 ignition:expressed_in="base_link">1 -1 0</fdir1>
-            </ode></friction></surface>
-        </collision>
-    </gazebo>
+    <!-- WHEELS (wie Referenz: fl/fr/rl/rr_wheel_joint, parent=body_link, axis=Y, RPY=0) -->
+    <xacro:mecanum_wheel prefix="fl" x_reflect="1"  y_reflect="1"  mesh="mecanum_b"/>
+    <xacro:mecanum_wheel prefix="fr" x_reflect="1"  y_reflect="-1" mesh="mecanum_a"/>
+    <xacro:mecanum_wheel prefix="rl" x_reflect="-1" y_reflect="1"  mesh="mecanum_b"/>
+    <xacro:mecanum_wheel prefix="rr" x_reflect="-1" y_reflect="-1" mesh="mecanum_a"/>
 </robot>

File: src/gubot_description/urdf/gubot_one_main.urdf.xacro (robot description, xacro)
@@ -1,4 +1,4 @@
 <?xml version="1.0"?>
-<robot xmlns:xacro="http://www.ros.org/wiki/xacro"  name="gubot_one">
+<robot xmlns:xacro="http://www.ros.org/wiki/xacro" xmlns:ignition="http://ignitionrobotics.org/schema" name="gubot_one">
     <xacro:arg name="use_ros2_control" default="true"/>
     <xacro:arg name="sim_mode" default="false"/>
@@ -8,5 +8,11 @@
          bleiben immer erhalten. -->
     <xacro:arg name="use_camera" default="true"/>
+    <!-- use_depth_camera=true fuegt eine (Sim-)Tiefenkamera hinzu; Standard aus. -->
+    <xacro:arg name="use_depth_camera" default="false"/>
+    <xacro:include filename="properties.xacro" />
     <xacro:include filename="gubot_one_geometry.xacro" />
+    <xacro:if value="$(arg sim_mode)">
+        <xacro:include filename="gazebo_sim.xacro" />
+    </xacro:if>
     <xacro:if value="$(arg use_ros2_control)">
         <xacro:if value="$(arg sim_mode)">
@@ -19,5 +25,7 @@
     <xacro:include filename="sensor_lidar.xacro" />
     <xacro:include filename="sensor_camera.xacro" />
-    <!-- <xacro:include filename="sensor_depth_camera.xacro" /> -->
+    <xacro:if value="$(arg use_depth_camera)">
+        <xacro:include filename="sensor_depth_camera.xacro" />
+    </xacro:if>
     <xacro:include filename="visual_face.xacro" />
     <xacro:if value="$(arg use_nerf_hardware)">

File: src/gubot_description/urdf/ros2_control_gazebo_ign_fortress.xacro (robot description, xacro)
@@ -9,9 +9,10 @@
          - position_proportional_gain entfernt (wird von GazeboSimSystem nicht unterstützt)
          - Sensor-Name "imu_sensor" konsistent mit controllers.yaml sensor_name und
-           dem Gazebo-Sensor in gubot_one_geometry.xacro
+           dem Gazebo-Sensor in gazebo_sim.xacro
     -->
     <!-- NEW: controller config path injected by load_urdf.launch.py at runtime -->
     <xacro:arg name="controller_config"
         default="$(find gubot_controller)/config/controllers.yaml"/>
+    <xacro:include filename="ros2_control_common.xacro"/>
     <ros2_control name="GubotIgnitionSystem" type="system">
         <hardware>
@@ -19,52 +20,8 @@
         </hardware>
         <!-- Gelenkbezeichnungen: fl/fr/rl/rr_wheel_joint (Referenz rosbot_xl-Schema) -->
-        <joint name="fl_wheel_joint">
-            <command_interface name="velocity">
-                <param name="min">-10</param>
-                <param name="max">10</param>
-            </command_interface>
-            <state_interface name="velocity">
-                <param name="initial_value">0.0</param>
-            </state_interface>
-            <state_interface name="position">
-                <param name="initial_value">0.0</param>
-            </state_interface>
-        </joint>
-        <joint name="fr_wheel_joint">
-            <command_interface name="velocity">
-                <param name="min">-10</param>
-                <param name="max">10</param>
-            </command_interface>
-            <state_interface name="velocity">
-                <param name="initial_value">0.0</param>
-            </state_interface>
-            <state_interface name="position">
-                <param name="initial_value">0.0</param>
-            </state_interface>
-        </joint>
-        <joint name="rl_wheel_joint">
-            <command_interface name="velocity">
-                <param name="min">-10</param>
-                <param name="max">10</param>
-            </command_interface>
-            <state_interface name="velocity">
-                <param name="initial_value">0.0</param>
-            </state_interface>
-            <state_interface name="position">
-                <param name="initial_value">0.0</param>
-            </state_interface>
-        </joint>
-        <joint name="rr_wheel_joint">
-            <command_interface name="velocity">
-                <param name="min">-10</param>
-                <param name="max">10</param>
-            </command_interface>
-            <state_interface name="velocity">
-                <param name="initial_value">0.0</param>
-            </state_interface>
-            <state_interface name="position">
-                <param name="initial_value">0.0</param>
-            </state_interface>
-        </joint>
+        <xacro:ros2_control_wheel_joint name="fl_wheel_joint" sim="true"/>
+        <xacro:ros2_control_wheel_joint name="fr_wheel_joint" sim="true"/>
+        <xacro:ros2_control_wheel_joint name="rl_wheel_joint" sim="true"/>
+        <xacro:ros2_control_wheel_joint name="rr_wheel_joint" sim="true"/>
         <!-- Nerf-Joints: NUR wenn use_nerf_hardware=true, sonst existieren diese Joints nicht in der URDF -->
         <xacro:if value="$(arg use_nerf_hardware)">
@@ -88,20 +45,5 @@
             </joint>
         </xacro:if>
-        <!-- Sensor-Name "imu_sensor": muss übereinstimmen mit:
-             1. Gazebo-Sensor name="imu_sensor" in gubot_one_geometry.xacro
-             2. controllers.yaml: imu_broadcaster.ros__parameters.sensor_name: imu_sensor
-        -->
-        <sensor name="imu_sensor">
-            <state_interface name="linear_acceleration.x"/>
-            <state_interface name="linear_acceleration.y"/>
-            <state_interface name="linear_acceleration.z"/>
-            <state_interface name="angular_velocity.x"/>
-            <state_interface name="angular_velocity.y"/>
-            <state_interface name="angular_velocity.z"/>
-            <state_interface name="orientation.x"/>
-            <state_interface name="orientation.y"/>
-            <state_interface name="orientation.z"/>
-            <state_interface name="orientation.w"/>
-        </sensor>
+        <xacro:ros2_control_imu_sensor/>
     </ros2_control>
     <gazebo>

File: src/gubot_description/urdf/ros2_control_hardware.xacro (robot description, xacro)
@@ -3,71 +3,38 @@
     <xacro:arg name="use_nerf_hardware" default="true"/>
     <xacro:arg name="nerf_port" default="/dev/serial/by-id/usb-Arduino_LLC_Arduino_Leonardo-if00"/>
+    <!-- Hardware-Parameter als xacro-Args (Defaults = bisherige Festwerte),
+         von aussen ueberschreibbar, z. B. drive_device:=/dev/ttyACM0 -->
+    <xacro:arg name="drive_device" default="/dev/serial/by-id/usb-Raspberry_Pi_Pico_50443405786ACA1C-if00"/>
+    <xacro:arg name="drive_baud_rate" default="115200"/>
+    <xacro:arg name="drive_loop_rate" default="30"/>
+    <xacro:arg name="drive_timeout_ms" default="1000"/>
+    <xacro:arg name="enc_counts_per_rev" default="3436"/>
+    <xacro:arg name="nerf_tilt_min" default="-0.52"/>
+    <xacro:arg name="nerf_tilt_max" default="0.52"/>
     <xacro:include filename="$(find nerf_launch_system)/description/urdf/ros2_control_hardware_nerf.xacro" />
+    <xacro:include filename="ros2_control_common.xacro"/>
     <ros2_control name="RealRobot" type="system">
         <hardware>
             <plugin>mecanum_pico/MecanumPicoHardware</plugin>
-            <!-- <param name="front_left_wheel_name">front_left_wheel_joint</param> -->
-            <!-- <param name="front_right_wheel_name">front_right_wheel_joint</param> -->
-            <!-- <param name="rear_left_wheel_name">rear_left_wheel_joint</param> -->
-            <!-- <param name="rear_right_wheel_name">rear_right_wheel_joint</param> -->
             <param name="front_left_wheel_name">fl_wheel_joint</param>
             <param name="front_right_wheel_name">fr_wheel_joint</param>
             <param name="rear_left_wheel_name">rl_wheel_joint</param>
             <param name="rear_right_wheel_name">rr_wheel_joint</param>
-            <param name="loop_rate">30</param>
-            <param name="device">/dev/serial/by-id/usb-Raspberry_Pi_Pico_50443405786ACA1C-if00</param>
-            <param name="baud_rate">115200</param>
-            <param name="timeout_ms">1000</param>
-            <param name="enc_counts_per_rev">3436</param>
+            <param name="loop_rate">$(arg drive_loop_rate)</param>
+            <param name="device">$(arg drive_device)</param>
+            <param name="baud_rate">$(arg drive_baud_rate)</param>
+            <param name="timeout_ms">$(arg drive_timeout_ms)</param>
+            <param name="enc_counts_per_rev">$(arg enc_counts_per_rev)</param>
         </hardware>
-        <joint name="fl_wheel_joint">
-            <command_interface name="velocity">
-                <param name="min">-10</param>
-                <param name="max">10</param>
-            </command_interface>
-            <state_interface name="position"/>
-            <state_interface name="velocity"/>
-        </joint>
-        <joint name="fr_wheel_joint">
-            <command_interface name="velocity">
-                <param name="min">-10</param>
-                <param name="max">10</param>
-            </command_interface>
-            <state_interface name="position"/>
-            <state_interface name="velocity"/>
-        </joint>
-        <joint name="rl_wheel_joint">
-            <command_interface name="velocity">
-                <param name="min">-10</param>
-                <param name="max">10</param>
-            </command_interface>
-            <state_interface name="position"/>
-            <state_interface name="velocity"/>
-        </joint>
-        <joint name="rr_wheel_joint">
-            <command_interface name="velocity">
-                <param name="min">-10</param>
-                <param name="max">10</param>
-            </command_interface>
-            <state_interface name="position"/>
-            <state_interface name="velocity"/>
-        </joint>
-        <sensor name="imu_sensor">
-            <state_interface name="linear_acceleration.x"/>
-            <state_interface name="linear_acceleration.y"/>
-            <state_interface name="linear_acceleration.z"/>
-            <state_interface name="angular_velocity.x"/>
-            <state_interface name="angular_velocity.y"/>
-            <state_interface name="angular_velocity.z"/>
-            <state_interface name="orientation.x"/>
-            <state_interface name="orientation.y"/>
-            <state_interface name="orientation.z"/>
-            <state_interface name="orientation.w"/>
-        </sensor>
+        <xacro:ros2_control_wheel_joint name="fl_wheel_joint" sim="false"/>
+        <xacro:ros2_control_wheel_joint name="fr_wheel_joint" sim="false"/>
+        <xacro:ros2_control_wheel_joint name="rl_wheel_joint" sim="false"/>
+        <xacro:ros2_control_wheel_joint name="rr_wheel_joint" sim="false"/>
+        <xacro:ros2_control_imu_sensor/>
     </ros2_control>
     <xacro:if value="$(arg use_nerf_hardware)">
         <!-- Einzige Quelle der Wahrheit für den NerfSystem-Block: Macro aus
              nerf_launch_system statt lokal dupliziert (vermeidet Drift). -->
-        <xacro:nerf_ros2_control_hardware port="$(arg nerf_port)" tilt_min="-0.52" tilt_max="0.52"/>
+        <xacro:nerf_ros2_control_hardware port="$(arg nerf_port)" tilt_min="$(arg nerf_tilt_min)" tilt_max="$(arg nerf_tilt_max)"/>
     </xacro:if>
 </robot>
