Commit message: refactor(description): modulare xacros + shared dimensions yaml + urdf tests
Co-Authored-By: Claude Fable 5 <noreply@anthropic.com>

File: src/gubot_description/urdf/sensor_camera.xacro (robot description, xacro)
@@ -6,4 +6,6 @@
         <origin xyz="0.276 0 0.181" rpy="0 0.18 0"/>
     </joint>
+    <!-- camera_link bewusst ohne inertial/collision: der fixe Joint wird von
+         Gazebo in body_link gelumpt (fixed joint lumping). -->
     <link name="camera_link">
         <visual>
@@ -49,9 +51,5 @@
                 </clip>
             </camera>
-            <!-- <xacro:if value="$(arg use_gazebo_classic)"> -->
-            <!--     <plugin name="camera_controller" filename="libgazebo_ros_camera.so"> -->
-            <!--         <frame_name>camera_link_optical</frame_name> -->
-            <!--     </plugin> -->
-            <!-- NEU: Expliziter Frame-ID damit Ignition nicht den auto-generierten
+            <!-- Expliziter Frame-ID damit Ignition nicht den auto-generierten
                  Pfad 'gubot_one/base_link/camera' verwendet, sondern den TF-Frame
                  'camera_link_optical' der von robot_state_publisher veroeffentlicht wird -->

File: src/gubot_description/urdf/sensor_depth_camera.xacro (robot description, xacro)
@@ -1,10 +1,13 @@
 <?xml version="1.0"?>
 <robot xmlns:xacro="http://www.ros.org/wiki/xacro" >
-    <joint name="camera_joint" type="fixed">
+    <!-- Optionale Tiefenkamera (use_depth_camera:=true, Standard aus).
+         Eigene Frame-Namen (depth_camera_*), kollidiert nicht mit
+         sensor_camera.xacro. Sensor: Ignition Fortress depth_camera. -->
+    <joint name="depth_camera_joint" type="fixed">
         <parent link="body_link"/>
-        <child link="camera_link"/>
+        <child link="depth_camera_link"/>
         <origin xyz="0.305 0 0.08" rpy="0 0 0"/>
     </joint>
-    <link name="camera_link">
+    <link name="depth_camera_link">
         <visual>
             <geometry>
@@ -14,20 +17,20 @@
         </visual>
     </link>
-    <joint name="camera_optical_joint" type="fixed">
-        <parent link="camera_link"/>
-        <child link="camera_link_optical"/>
+    <joint name="depth_camera_optical_joint" type="fixed">
+        <parent link="depth_camera_link"/>
+        <child link="depth_camera_link_optical"/>
         <origin xyz="0 0 0" rpy="${-pi/2} 0 ${-pi/2}"/>
     </joint>
-    <link name="camera_link_optical"></link>
-    <gazebo reference="camera_link">
+    <link name="depth_camera_link_optical"></link>
+    <gazebo reference="depth_camera_link">
         <material>Gazebo/Red</material>
-        <sensor name="camera" type="depth">
+        <sensor name="depth_camera" type="depth_camera">
             <pose> 0 0 0 0 0 0 </pose>
-            <visualize>true</visualize>
+            <visualize>false</visualize>
             <update_rate>10</update_rate>
             <camera>
                 <horizontal_fov>1.089</horizontal_fov>
                 <image>
-                    <format>B8G8R8</format>
+                    <format>R_FLOAT32</format>
                     <width>640</width>
                     <height>480</height>
@@ -38,9 +41,6 @@
                 </clip>
             </camera>
-            <plugin name="camera_controller" filename="libgazebo_ros_camera.so">
-                <frame_name>camera_link_optical</frame_name>
-                <min_depth>0.1</min_depth>
-                <max_depth>100.0</max_depth>
-            </plugin>
+            <topic>camera/depth</topic>
+            <ignition_frame_id>depth_camera_link_optical</ignition_frame_id>
         </sensor>
     </gazebo>
